File: Mainboard/LattePanda Module.kicad_sch (KiCad schematic)
At the start: 21 parts, among them J1 Conn_01x03_Pin, U18 W25Q128JVS

Commit message: Added HDMI > LDVS screens
Parts:
- removed R76: 100K/1%, A_DFRobot:R_0402, symbol Device:R
- added J2, J6: BM14B-NSHSS-TBT_LF__SN_, BM14BNSHSSTBTLFSN, symbol BM14B-NSHSS-TBT_LF__SN_:BM14B-NSHSS-TBT_LF__SN_
Connections:
- net TCP_0_DDC_SDA: now reaches A1.177 (DDC_0_SDA)
- net TCP_0_DDC_SCL: now reaches A1.179 (DDC_0_SCL)
- net TCP_0_HPD: now reaches A1.187 (HPD_0)
- net TCP_0_TX3-: now reaches A1.227 (TCP_0_TXRX1-)
- net TCP_0_TX3+: now reaches A1.229 (TCP_0_TXRX1+)
- net TCP_0_TX2-: now reaches A1.233 (TCP_0_TX1-)
- net TCP_0_TX2+: now reaches A1.235 (TCP_0_TX1+)
- net TCP_0_TX1-: now reaches A1.239 (TCP_0_TXRX0-)
- net TCP_0_TX1+: now reaches A1.241 (TCP_0_TXRX0+)
- net TCP_0_TX0-: now reaches A1.245 (TCP_0_TX0-)
- net TCP_0_TX0+: now reaches A1.247 (TCP_0_TX0+)
- net REFCLK0+: no longer names the net of A1.85 (REFCLK0+)
- net REFCLK0-: no longer names the net of A1.87 (REFCLK0-)
- net REFCLK2+: no longer names the net of A1.97 (REFCLK2+)
- net REFCLK2-: no longer names the net of A1.99 (REFCLK2-)
- net REFCLK3+: no longer names the net of A1.88 (REFCLK3+)
- net REFCLK3-: no longer names the net of A1.90 (REFCLK3-)
- net REFCLK4+: no longer names the net of A1.94 (REFCLK4+)
- net REFCLK4-: no longer names the net of A1.96 (REFCLK4-)
- net SOC_UART0_RX: no longer names the net of A1.137 (SOC_UART0_RXD)
- net SOC_UART0_TX: no longer names the net of A1.139 (SOC_UART0_TXD)
- net SOC_UART1_RX: no longer names the net of A1.141 (SOC_UART1_RXD)
- net SOC_UART1_TX: no longer names the net of A1.143 (SOC_UART1_TXD)
- net SOC_UART2_RX: no longer names the net of A1.140 (SOC_UART2_RXD)
- net SOC_UART2_TX: no longer names the net of A1.138 (SOC_UART2_TXD)
- net ~{CLKREQ3}: no longer names the net of A1.100 (~{PCIeCLK_REQ3})
- net ~{CLKREQ4}: no longer names the net of A1.102 (~{PCIeCLK_REQ4})
- net ~{PEWAKE}: no longer names the net of A1.103 (~{PCIe_WAKE})
- net ~{PLT_RST}: no longer names the net of A1.105 (~{BUF_PLT_RST})
- no-connect marks 73 -> 72

Commit message: More work on the Screens
Connections:
- net HSIO_6_RX+: no longer names the net of A1.64 (HSIO6_RXP)
- net HSIO_6_RX-: no longer names the net of A1.66 (HSIO6_RXN)
- net HSIO_6_TX+: no longer names the net of A1.61 (HSIO6_TXP)
- net HSIO_6_TX-: no longer names the net of A1.63 (HSIO6_TXN)
- no-connect marks 72 -> 76
Changed lines of the file:
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@@
-		)
-	)
-	(text_box "HSIO_6 used for GbE(PCIe x1)\n"
-		(exclude_from_sim no)
-		(at 175.26 163.83 0)
-		(size 39.37 10.16)
-		(margins 1.905 1.905 1.905 1.905)
-		(stroke
-			(width 0)
-			(type default)
-		)
-		(fill
-			(type none)
-		)
-		(effects
-			(font
-				(size 2.54 2.54)
-				(thickness 0.508)
-				(bold yes)
-			)
-			(justify left top)
 		)
 	)
@@
 	)
 	(no_connect
+		(at 267.97 165.1)
+	)
+	(no_connect
 		(at 267.97 299.72)
 	)
@@
 	)
 	(no_connect
+		(at 267.97 172.72)
+	)
+	(no_connect
 		(at 354.33 71.12)
 	)
@@
 	)
 	(no_connect
+		(at 267.97 167.64)
+	)
+	(no_connect
 		(at 354.33 320.04)
 	)
@@
 	)
 	(no_connect
+		(at 267.97 170.18)
+	)
+	(no_connect
 		(at 267.97 317.5)
 	)
@@
 	(wire
 		(pts
-			(xy 236.22 172.72) (xy 267.97 172.72)
-		)
-		(stroke
-			(width 0)
-			(type default)
-		)
-	)
-	(wire
-		(pts
 			(xy 309.88 53.34) (xy 312.42 53.34)
 		)
@@
 	(wire
 		(pts
-			(xy 236.22 165.1) (xy 267.97 165.1)
-		)
-		(stroke
-			(width 0)
-			(type default)
-		)
-	)
-	(wire
-		(pts
 			(xy 394.97 226.06) (xy 406.4 226.06)
 		)
@@
 	(wire
 		(pts
-			(xy 236.22 167.64) (xy 267.97 167.64)
-		)
-		(stroke
-			(width 0)
-			(type default)
-		)
-	)
-	(wire
-		(pts
 			(xy 394.97 226.06) (xy 394.97 236.22)
 		)
@@
 		(pts
 			(xy 236.22 177.8) (xy 267.97 177.8)
-		)
-		(stroke
-			(width 0)
-			(type default)
-		)
-	)
-	(wire
-		(pts
-			(xy 236.22 170.18) (xy 267.97 170.18)
 		)
 		(stroke
@@
 		)
 	)
-	(hierarchical_label "HSIO_6_RX-"
-		(shape input)
-		(at 236.22 172.72 180)
-		(effects
-			(font
-				(size 1.27 1.27)
-			)
-			(justify right)
-		)
-	)
 	(hierarchical_label "I2C4_SCL"
 		(shape output)
@@
 		)
 	)
-	(hierarchical_label "HSIO_6_RX+"
-		(shape input)
-		(at 236.22 170.18 180)
-		(effects
-			(font
-				(size 1.27 1.27)
-			)
-			(justify right)
-		)
-	)
 	(hierarchical_label "DDI_B_TX2+"
 		(shape output)
@@
 		(effects
 			(font
-				(size 1.27 1.27)
-			)
-			(justify right)
-		)
-	)
-	(hierarchical_label "HSIO_6_TX-"
-		(shape output)
-		(at 236.22 167.64 180)
-		(effects
-			(font
-				(size 1.27 1.27)
-			)
-			(justify right)
-		)
-	)
-	(hierarchical_label "HSIO_6_TX+"
-		(shape output)
-		(at 236.22 165.1 180)
-		(effects
-			(font
