File: Mainboard.COOKED/HDMI.kicad_sch (KiCad schematic)
At the start: 51 parts, among them Q10 2SK3018, Q17 2SK3018, Q18 2SK3018, Q9 2N7002, U20 ADV7613WBBCZ, U7 TPAZ1023-04F, U8 TPAZ1023-04F, Y2 SiT8008xx-1x-xxE

Commit message: "Scrapped" the current Mainboard, seems to be very broken for no reason.
It is being kept for now so that work done for the displays can be copied over later.
Parts:
- C25, C33, C34, C35, C36, C37, C38, C39: value 100nF/16V -> 10uF/10V; DF_Comment 贴片电容0402-100nF-16V-X7R(0402) -> 贴片电容0402-10UF-10V-X5R_GRM155R61A106ME44D; SCH_Show_Footprint C0402 -> -- mixed values --
- D34, D35, D36: value 0402ESDA-05N -> Barrel_Jack_Switch; footprint A_HDJ_Library:D_0402_1005Metric -> A_HDJ_Library:DC_Jack_DC007B_30V_10A; Buy_Link (none) -> https://item.szlcsc.com/19360929.html; DF_Comment 5.0V双向静电保护管_0402ESDA-05N -> DC2.5电源母座_12V/10A_XDJK-060B-055; SCH_Show_Footprint D0402 -> (none)
- D37: value 1N5819WS -> 1K/1%; footprint A_DFRobot:D_SOD-323 -> A_HDJ_Library:R_0402_1005Metric; DF_Comment 二极管-1N5819W-SOD323备选型号:B5819WS、JSPD140A -> 贴片电阻0402-1K-1%; SCH_Show_Footprint SOD-323 -> (none)
- Q10, Q17, Q18: value 2SK3018 -> HM7533HBPR; footprint Package_TO_SOT_SMD:SOT-23 -> Package_TO_SOT_SMD:SOT-89-3; Buy_Link https://item.szlcsc.com/774253.html -> (none); DF_Comment NMOS_2SK3018_SOT-23 -> 高压LDO_HM7533HBPR_SOT89
- Q9: value 2N7002 -> AO3407; DF_Comment 2N7002-N沟道MOS管-SOT-23[备选型号:JMTL2N7002K] -> PMOS管AO3407-SOT23-3
- R104, R114, R117, R118, R28: value 2.2K/1% -> 21.5K/1%; footprint A_DFRobot:R_0402 -> A_HDJ_Library:R_0402_1005Metric; DF_Comment 贴片电阻0402-2.2K-1% -> 贴片电阻0402-21.5K-1%
- R105: value 21.5K/1% -> 0R/1%; footprint A_DFRobot:R_0402 -> A_HDJ_Library:R_0402_1005Metric; DF_Comment 贴片电阻0402-21.5K-1% -> 贴片电阻0402-0R-1%
- R106, R107, R108, R109, R112, R113, R115, R116: value 470R/1% -> 56K/1%; footprint A_DFRobot:R_0402 -> A_HDJ_Library:R_0402_1005Metric; DF_Comment 贴片电阻0402-470R-1% -> 贴片电阻0402-56K-1%(0402)
- R110: value 1K/1% -> 2.2K/1%; footprint A_DFRobot:R_0402 -> A_HDJ_Library:R_0402_1005Metric; DF_Comment 贴片电阻0402-1K-1% -> 贴片电阻0402-2.2K-1%
- R76: value 1M/1% -> 470R/1%; footprint A_DFRobot:R_0402 -> A_HDJ_Library:R_0402_1005Metric; DF_Comment 贴片电阻0402-1M-1% -> 贴片电阻0402-470R-1%
- U20: value ADV7613WBBCZ -> (none); footprint BC_100_4_ADI -> Connector_PinHeader_2.54mm:PinHeader_2x03_P2.54mm_Vertical; DF_Comment (none) -> 2.54黑色3x2P排针
- U7, U8: value TPAZ1023-04F -> CH224K; footprint A_HDJ_Library:Diodes_UDFN-10_1.0x2.5mm_P0.5mm -> A_HDJ_Library:ESSOP-10-1EP_3.9x5mm_P1.0mm_EP3.2x2.3; Buy_Link https://item.szlcsc.com/2973358.html -> (none); DF_Comment ESD静电保护IC-TPAZ1023-04F-DFN2510-10L -> USB PD等快充协议受电芯片-CH224K-ESSOP10
- Y2: value SiT8008xx-1x-xxE -> 2N7002; footprint Oscillator:Oscillator_SMD_SiT_PQFN-4Pin_2.5x2.0mm -> Package_TO_SOT_SMD:SOT-23; DF_Comment (none) -> 2N7002-N沟道MOS管-SOT-23[备选型号:JMTL2N7002K]
