File: Mainboard.COOKED/LattePanda Module.kicad_sch (KiCad schematic)
At the start: 22 parts, among them J1 Conn_01x03_Pin, J2 BM14B-NSHSS-TBT_LF__SN_, J6 BM14B-NSHSS-TBT_LF__SN_, U18 W25Q128JVS

Commit message: "Scrapped" the current Mainboard, seems to be very broken for no reason.
It is being kept for now so that work done for the displays can be copied over later.
Parts:
- A1: value LattePanda_Module_Gen1 -> ULC0524P; footprint A_HDJ_Library:DDR4_SODIMM_260P_8.0H_STD -> A_HDJ_Library:Diodes_UDFN-10_1.0x2.5mm_P0.5mm; Buy_Link https://item.szlcsc.com/5812308.html -> (none); DF_Comment 连接器_DDR4-SODIMM-260P-8H_TE_2309411-1 -> ESD静电保护IC-BV-ULC0524P-DFN2510-10L
- BT1: value Battery_Cell -> 220nF/16V; footprint A_HDJ_Library:Battery_Holder_CR1220_S8411-45R -> A_HDJ_Library:C_0402_1005Metric; Buy_Link https://item.szlcsc.com/1049689.html -> https://item.szlcsc.com/137804.html; DF_Comment CR1220电池座贴片塑料 -> 贴片电容0402-220nF-16V-X7R; SCH_Show_Footprint (none) -> C0402
- H5, H6: value MountingHole_Pad -> Bus_M.2_Socket_M; footprint A_HDJ_Library:MountingHole_3mm_M2_Pad_TopOnly -> A_HDJ_Library:PCIe_M.2_Connectors_P=0.5mm_H=4.2mm_KeyM; Buy_Link https://item.taobao.com/item.htm?abbucket=8&id=655855111684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 -> https://item.szlcsc.com/8568582.html; DF_Comment 贴片螺母柱M2XC4X5.5+C3X1.5（无铅铜） -> M.2连接器KEY-M_H4.2mm-67P_APCI0107-P001A
- J1: DF_Comment 2.54黑色单排排针-3P -> 2.54蓝色单排排针-3P
- J2, J6: value BM14B-NSHSS-TBT_LF__SN_ -> 22uF/25V; footprint BM14BNSHSSTBTLFSN -> Capacitor_SMD:C_0805_2012Metric; DF_Comment (none) -> 贴片电容0805-22uF-25V-X5R; Height 6 -> (none); Manufacturer_Name JST (JAPAN SOLDERLESS TERMINALS) -> (none); Manufacturer_Part_Number BM14B-NSHSS-TBT(LF)(SN) -> (none); SCH_Show_Footprint (none) -> C603
- R1: value 1K/1% -> 2.2K/1%; footprint A_DFRobot:R_0402 -> A_HDJ_Library:R_0402_1005Metric; DF_Comment 贴片电阻0402-1K-1% -> 贴片电阻0402-2.2K-1%
- R2: value 10K/1% -> 1M/1%; footprint A_DFRobot:R_0402 -> A_HDJ_Library:R_0402_1005Metric; DF_Comment 贴片电阻0402-10K-1% -> 贴片电阻0402-1M-1%
- R77: value 100K/1% -> 75K/1%; footprint A_DFRobot:R_0402 -> A_HDJ_Library:R_0402_1005Metric; DF_Comment 贴片电阻0402-100K-1% -> 贴片电阻0402-75K-1%
Changed lines of the file:
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@@
 			)
 		)
-		(property "Value" "LattePanda_Module_Gen1"
+		(property "Value" "ULC0524P"
 			(at 313.3441 327.66 0)
 			(show_name no)
@@
 			)
 		)
-		(property "Footprint" "A_HDJ_Library:DDR4_SODIMM_260P_8.0H_STD"
+		(property "Footprint" "A_HDJ_Library:Diodes_UDFN-10_1.0x2.5mm_P0.5mm"
 			(at 311.15 190.5 0)
 			(hide yes)
@@
 			)
 		)
-		(property "Datasheet" ""
+		(property "Datasheet" "https://www.diodes.com/assets/Datasheets/D3V3XA4B10LP.pdf"
 			(at 311.15 190.5 0)
 			(hide yes)
@@
 			)
 		)
-		(property "Description" "Intel Processor N100 up to 3.4 GHz quad core, 8GB RAM, 64GB eMMC, SoM computer"
+		(property "Description" ""
 			(at 311.15 190.5 0)
 			(hide yes)
@@
 			)
 		)
-		(property "Buy_Link" "https://item.szlcsc.com/5812308.html"
+		(property "Buy_Link" ""
 			(at 311.15 190.5 0)
 			(hide yes)
@@
 			)
 		)
-		(property "DF_Comment" "连接器_DDR4-SODIMM-260P-8H_TE_2309411-1"
+		(property "DF_Comment" "ESD静电保护IC-BV-ULC0524P-DFN2510-10L"
 			(at 311.15 190.5 0)
 			(hide yes)
@@
 			)
 		)
-		(property "Value" "1K/1%"
+		(property "Value" "2.2K/1%"
 			(at 337.82 50.8 90)
 			(show_name no)
@@
 			)
 		)
-		(property "Footprint" "A_DFRobot:R_0402"
+		(property "Footprint" "A_HDJ_Library:R_0402_1005Metric"
 			(at 339.09 55.118 90)
 			(hide yes)
@@
 			)
 		)
-		(property "DF_Comment" "贴片电阻0402-1K-1%"
+		(property "DF_Comment" "贴片电阻0402-2.2K-1%"
 			(at 339.09 53.34 0)
 			(hide yes)
@@
 			)
 		)
-		(property "Value" "100K/1%"
+		(property "Value" "75K/1%"
 			(at 255.778 287.02 90)
 			(show_name no)
@@
 			)
 		)
-		(property "Footprint" "A_DFRobot:R_0402"
+		(property "Footprint" "A_HDJ_Library:R_0402_1005Metric"
 			(at 255.27 282.702 90)
 			(hide yes)
@@
 			)
 		)
-		(property "DF_Comment" "贴片电阻0402-100K-1%"
+		(property "DF_Comment" "贴片电阻0402-75K-1%"
 			(at 255.27 284.48 0)
 			(hide yes)
@@
 			)
 		)
-		(property "DF_Comment" "2.54黑色单排排针-3P"
+		(property "DF_Comment" "2.54蓝色单排排针-3P"
 			(at 223.52 73.66 0)
 			(hide yes)
@@
 			)
 		)
-		(property "Value" "Battery_Cell"
+		(property "Value" "220nF/16V"
 			(at 354.33 46.99 90)
 			(show_name no)
@@
 			)
 		)
-		(property "Footprint" "A_HDJ_Library:Battery_Holder_CR1220_S8411-45R"
+		(property "Footprint" "A_HDJ_Library:C_0402_1005Metric"
 			(at 347.726 53.34 90)
 			(hide yes)
@@
 			)
 		)
-		(property "Buy_Link" "https://item.szlcsc.com/1049689.html"
+		(property "Buy_Link" "https://item.szlcsc.com/137804.html"
 			(at 349.25 53.34 0)
 			(hide yes)
@@
 			)
 		)
-		(property "DF_Comment" "CR1220电池座贴片塑料"
+		(property "DF_Comment" "贴片电容0402-220nF-16V-X7R"
 			(at 349.25 53.34 0)
 			(hide yes)
@@
 			)
 		)
-		(property "SCH_Show_Footprint" ""
+		(property "SCH_Show_Footprint" "C0402"
 			(at 349.25 53.34 0)
 			(hide yes)
@@
 			)
 		)
-		(property "Value" "MountingHole_Pad"
+		(property "Value" "Bus_M.2_Socket_M"
 			(at 416.56 299.72 0)
 			(show_name no)
@@
 			)
 		)
-		(property "Footprint" "A_HDJ_Library:MountingHole_3mm_M2_Pad_TopOnly"
+		(property "Footprint" "A_HDJ_Library:PCIe_M.2_Connectors_P=0.5mm_H=4.2mm_KeyM"
 			(at 414.02 299.72 0)
 			(hide yes)
@@
 			)
 		)
-		(property "Datasheet" ""
+		(property "Datasheet" "http://read.pudn.com/downloads794/doc/project/3133918/PCIe_M.2_Electromechanical_Spec_Rev1.0_Final_11012013_RS_Clean.pdf#page=155"
 			(at 414.02 299.72 0)
 			(hide yes)
@@
 			)
 		)
-		(property "DF_Comment" "贴片螺母柱M2XC4X5.5+C3X1.5（无铅铜）"
+		(property "DF_Comment" "M.2连接器KEY-M_H4.2mm-67P_APCI0107-P001A"
 			(at 414.02 299.72 0)
 			(hide yes)
@@
 			)
 		)
-		(property "Buy_Link" "https://item.taobao.com/item.htm?abbucket=8&id=655855111684&ns=1&skuId=4725777108077&spm=a21n57.1.0.0.5263523chYMn0X"
+		(property "Buy_Link" "https://item.szlcsc.com/8568582.html"
 			(at 414.02 299.72 0)
 			(hide yes)
@@
 			)
 		)
-		(property "Value" "BM14B-NSHSS-TBT_LF__SN_"
+		(property "Value" "22uF/25V"
 			(at 454.66 161.29 0)
 			(show_name no)
@@
 			)
 		)
-		(property "Footprint" "BM14BNSHSSTBTLFSN"
+		(property "Footprint" "Capacitor_SMD:C_0805_2012Metric"
 			(at 445.77 104.47 0)
 			(hide yes)
@@
 			)
 		)
-		(property "Datasheet" "https://www.jst-mfg.com/product/pdf/eng/eNSH.pdf"
+		(property "Datasheet" ""
 			(at 445.77 4.47 0)
 			(hide yes)
@@
 			)
 		)
-		(property "Description" "Connector Header Surface Mount 14 position 0.039\" (1.00mm), 1A, 50V, -25C ~ 85C"
+		(property "Description" ""
 			(at 467.36 199.39 0)
 			(hide yes)
@@
 			)
 		)
-		(property "Height" "6"
+		(property "Height" ""
 			(at 445.77 -195.53 0)
 			(hide yes)
@@
 			)
 		)
-		(property "Manufacturer_Name" "JST (JAPAN SOLDERLESS TERMINALS)"
+		(property "Manufacturer_Name" ""
 			(at 445.77 -495.53 0)
 			(hide yes)
@@
 			)
 		)
-		(property "Manufacturer_Part_Number" "BM14B-NSHSS-TBT(LF)(SN)"
+		(property "Manufacturer_Part_Number" ""
 			(at 445.77 -595.53 0)
 			(hide yes)
@@
 			)
 		)
+		(property "DF_Comment" "贴片电容0805-22uF-25V-X5R"
+			(at 467.36 199.39 0)
+			(hide yes)
+			(show_name no)
+			(do_not_autoplace no)
+			(effects
+				(font
+					(size 1.27 1.27)
+				)
+			)
+		)
+		(property "SCH_Show_Footprint" "C603"
+			(at 467.36 199.39 0)
+			(hide yes)
+			(show_name no)
+			(do_not_autoplace no)
+			(effects
+				(font
+					(size 1.27 1.27)
+				)
+			)
+		)
 		(pin "5"
 		)
@@
 			)
 		)
-		(property "Value" "BM14B-NSHSS-TBT_LF__SN_"
+		(property "Value" "22uF/25V"
 			(at 454.66 115.57 0)
 			(show_name no)
@@
 			)
 		)
-		(property "Footprint" "BM14BNSHSSTBTLFSN"
+		(property "Footprint" "Capacitor_SMD:C_0805_2012Metric"
 			(at 445.77 58.75 0)
 			(hide yes)
@@
 			)
 		)
-		(property "Datasheet" "https://www.jst-mfg.com/product/pdf/eng/eNSH.pdf"
+		(property "Datasheet" ""
 			(at 445.77 -41.25 0)
 			(hide yes)
@@
 			)
 		)
-		(property "Description" "Connector Header Surface Mount 14 position 0.039\" (1.00mm), 1A, 50V, -25C ~ 85C"
+		(property "Description" ""
 			(at 467.36 153.67 0)
 			(hide yes)
@@
 			)
 		)
-		(property "Height" "6"
+		(property "Height" ""
 			(at 445.77 -241.25 0)
 			(hide yes)
@@
 			)
 		)
-		(property "Manufacturer_Name" "JST (JAPAN SOLDERLESS TERMINALS)"
+		(property "Manufacturer_Name" ""
 			(at 445.77 -541.25 0)
 			(hide yes)
@@
 			)
 		)
-		(property "Manufacturer_Part_Number" "BM14B-NSHSS-TBT(LF)(SN)"
+		(property "Manufacturer_Part_Number" ""
 			(at 445.77 -641.25 0)
 			(hide yes)
@@
 			)
 		)
+		(property "DF_Comment" "贴片电容0805-22uF-25V-X5R"
+			(at 467.36 153.67 0)
+			(hide yes)
+			(show_name no)
+			(do_not_autoplace no)
+			(effects
+				(font
+					(size 1.27 1.27)
+				)
+			)
+		)
+		(property "SCH_Show_Footprint" "C603"
+			(at 467.36 153.67 0)
+			(hide yes)
+			(show_name no)
+			(do_not_autoplace no)
+			(effects
+				(font
+					(size 1.27 1.27)
+				)
+			)
+		)
 		(pin "5"
 		)
@@
 			)
 		)
-		(property "Value" "10K/1%"
+		(property "Value" "1M/1%"
 			(at 380.238 260.858 90)
 			(show_name no)
@@
 			)
 		)
-		(property "Footprint" "A_DFRobot:R_0402"
+		(property "Footprint" "A_HDJ_Library:R_0402_1005Metric"
 			(at 376.936 258.318 90)
 			(hide yes)
@@
 			)
 		)
-		(property "DF_Comment" "贴片电阻0402-10K-1%"
+		(property "DF_Comment" "贴片电阻0402-1M-1%"
 			(at 376.936 256.54 0)
 			(hide yes)
@@
 			)
 		)
-		(property "Value" "MountingHole_Pad"
+		(property "Value" "Bus_M.2_Socket_M"
 			(at 441.96 299.72 0)
 			(show_name no)
@@
 			)
 		)
-		(property "Footprint" "A_HDJ_Library:MountingHole_3mm_M2_Pad_TopOnly"
+		(property "Footprint" "A_HDJ_Library:PCIe_M.2_Connectors_P=0.5mm_H=4.2mm_KeyM"
 			(at 439.42 299.72 0)
 			(hide yes)
@@
 			)
 		)
-		(property "Datasheet" ""
+		(property "Datasheet" "http://read.pudn.com/downloads794/doc/project/3133918/PCIe_M.2_Electromechanical_Spec_Rev1.0_Final_11012013_RS_Clean.pdf#page=155"
 			(at 439.42 299.72 0)
 			(hide yes)
@@
 			)
 		)
-		(property "DF_Comment" "贴片螺母柱M2XC4X5.5+C3X1.5（无铅铜）"
+		(property "DF_Comment" "M.2连接器KEY-M_H4.2mm-67P_APCI0107-P001A"
 			(at 439.42 299.72 0)
 			(hide yes)
@@
 			)
 		)
-		(property "Buy_Link" "https://item.taobao.com/item.htm?abbucket=8&id=655855111684&ns=1&skuId=4725777108077&spm=a21n57.1.0.0.5263523chYMn0X"
+		(property "Buy_Link" "https://item.szlcsc.com/8568582.html"
 			(at 439.42 299.72 0)
 			(hide yes)
