File: Mainboard.COOKED/USB2.0&USB3.0.kicad_sch (KiCad schematic)
At the start: 20 parts, among them J4 USB3_A_Stacked, J5 USB_A_Stacked, U3 ULC0524P, U4 ULC0524P, U5 ULC0524P

Commit message: "Scrapped" the current Mainboard, seems to be very broken for no reason.
It is being kept for now so that work done for the displays can be copied over later.
Parts:
- C26, C27, C28, C29: value 100nF/16V -> 10uF/10V; DF_Comment 贴片电容0402-100nF-16V-X7R(0402) -> 贴片电容0402-10UF-10V-X5R_GRM155R61A106ME44D; SCH_Show_Footprint C0402 -> -- mixed values --
- C30, C31, C32: value 22uF/10V -> 4.7uF
- D5, D6, D7, D8: value 0402ESDA-05N -> Barrel_Jack_Switch; footprint A_HDJ_Library:D_0402_1005Metric -> A_HDJ_Library:DC_Jack_DC007B_30V_10A; Buy_Link (none) -> https://item.szlcsc.com/19360929.html; DF_Comment 5.0V双向静电保护管_0402ESDA-05N -> DC2.5电源母座_12V/10A_XDJK-060B-055; SCH_Show_Footprint D0402 -> (none)
- F2, F3: value 6V/1A -> 2.2uH/4.3A; footprint A_HDJ_Library:Fuse_0805_2012Metric -> A_HDJ_Library:L_Sunlord_SWPA4020S; Buy_Link https://item.szlcsc.com/947770.html -> (none); DF_Comment 0805贴片自恢复保险丝1A-6V_BSMD0805-100-6V -> WPN4020H2R2MT 2.2UH 20% 额定电流4.3A 顺络; SCH_Show_Footprint R0603 -> (none)
- F4, F5: value 6V/2A -> SiT8008xx-1x-xxE; footprint Fuse:Fuse_0805_2012Metric -> Oscillator:Oscillator_SMD_SiT_PQFN-4Pin_2.5x2.0mm; Buy_Link https://item.szlcsc.com/947787.html -> (none); DF_Comment 0805贴片自恢复保险丝2A-6V_BSMD0805L-200 -> (none); SCH_Show_Footprint R0805 -> (none)
- J4: value USB3_A_Stacked -> USB_C_Receptacle_USB2.0; footprint A_HDJ_Library:USB3_A_Molex_48406-0001_Horizontal_Stacked -> A_HDJ_Library:USB_C_Receptacle_G-Switch_GT-USB-7010ASV; Buy_Link https://item.szlcsc.com/3132965.html -> (none); DF_Comment 双层USB3.0_A母座_USB-303WSD-BRY -> USB Type-C母座-U263-163N-4BS1735 5A
- J5: value USB_A_Stacked -> BM14B-NSHSS-TBT_LF__SN_; footprint A_HDJ_Library:USB_A_CUI_UJ2-ADH-TH_Horizontal_Stacked -> BM14BNSHSSTBTLFSN; DF_Comment USB2.0-A型双层白胶母座 -> (none); Height (none) -> 6; Manufacturer_Name (none) -> JST (JAPAN SOLDERLESS TERMINALS); Manufacturer_Part_Number (none) -> BM14B-NSHSS-TBT(LF)(SN)
- U3, U4, U5: value ULC0524P -> 6V/1A; footprint A_HDJ_Library:Diodes_UDFN-10_1.0x2.5mm_P0.5mm -> A_HDJ_Library:Fuse_0805_2012Metric; Buy_Link (none) -> https://item.szlcsc.com/947770.html; DF_Comment ESD静电保护IC-BV-ULC0524P-DFN2510-10L -> 0805贴片自恢复保险丝1A-6V_BSMD0805-100-6V; SCH_Show_Footprint (none) -> R0603
