File: Mainboard.COOKED/[DFR1142]Lite Carrier for LattePanda Mu(V2).kicad_sch (KiCad schematic)
At the start: 16 parts, among them J20 200485-0710, J3 2004850740, U21 TPS61165DBV

Commit message: "Scrapped" the current Mainboard, seems to be very broken for no reason.
It is being kept for now so that work done for the displays can be copied over later.
Parts:
- C40: value 1uF -> 220nF
- C41: value 4.7uF -> 0402ESDA-05N; footprint A_HDJ_Library:C_0603_1608Metric -> A_HDJ_Library:D_0402_1005Metric; DF_Comment 贴片电容0603-22uF-10V-X5R(0603) -> 5.0V双向静电保护管_0402ESDA-05N; SCH_Show_Footprint C603 -> D0402
- C42: value 220nF -> PESD24VS1UL-N; footprint A_HDJ_Library:C_0603_1608Metric -> A_HDJ_Library:D_0402_1005Metric; Buy_Link (none) -> https://item.szlcsc.com/393990.html; DF_Comment 贴片电容0603-22uF-10V-X5R(0603) -> 单向静电保护二极管_PESD24VS1UL-N_DFN1006; SCH_Show_Footprint C603 -> D0402
- D38: value D -> 0.57Ohm; footprint Diode_SMD:D_01005_0402Metric -> Inductor_SMD:L_01005_0402Metric
- J20: value 200485-0710 -> 2.2uF/50V; footprint 200485-0710:2004850710 -> A_HDJ_Library:C_0603_1608Metric; DF_Comment (none) -> 贴片电容0603-2.2uF-50V-X5R; Height 5.7 -> (none); Manufacturer_Name Molex -> (none); Manufacturer_Part_Number 200485-0710 -> (none); Mouser Part Number 538-200485-0710 -> (none); Mouser Price/Stock https://www.mouser.co.uk/ProductDetail/Molex/200485-0710?qs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 -> (none); SCH_Show_Footprint (none) -> -- mixed values --
- J3: value 2004850740 -> SS54; footprint 200485-0740:CON_2004850740 -> Diode_SMD:D_SMA; DF_Comment (none) -> 二极管-SS54-SMA(SMA); SCH_Show_Footprint (none) -> SMA
- R133: value 0.57Ohm -> TPS61165DBV; footprint Inductor_SMD:L_01005_0402Metric -> Package_SON:WSON-6-1EP_2x2mm_P0.65mm_EP1x1.6mm
- U21: value TPS61165DBV -> 2SK3018; footprint Package_SON:WSON-6-1EP_2x2mm_P0.65mm_EP1x1.6mm -> Package_TO_SOT_SMD:SOT-23; Buy_Link (none) -> https://item.szlcsc.com/774253.html; DF_Comment (none) -> NMOS_2SK3018_SOT-23
Changed lines of the file:
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@@
 			)
 		)
-		(property "Value" "TPS61165DBV"
+		(property "Value" "2SK3018"
 			(at 504.19 127 0)
 			(show_name no)
@@
 			)
 		)
-		(property "Footprint" "Package_SON:WSON-6-1EP_2x2mm_P0.65mm_EP1x1.6mm"
+		(property "Footprint" "Package_TO_SOT_SMD:SOT-23"
 			(at 504.19 162.306 0)
 			(hide yes)
@@
 			)
 		)
-		(property "Datasheet" "https://www.ti.com/lit/ds/symlink/tps61165.pdf"
+		(property "Datasheet" "https://www.onsemi.com/pub/Collateral/NDS7002A-D.PDF"
 			(at 504.19 160.02 0)
 			(hide yes)
@@
 			)
 		)
-		(property "Description" "High-Brightness, White LED Driver, 3V to 18V input voltage range, internal switch, constant current, up to 38V/1.2A output, SOT-23-6"
+		(property "Description" ""
 			(at 504.19 157.734 0)
+			(hide yes)
+			(show_name no)
+			(do_not_autoplace no)
+			(effects
+				(font
+					(size 1.27 1.27)
+				)
+			)
+		)
+		(property "Buy_Link" "https://item.szlcsc.com/774253.html"
+			(at 504.19 137.16 0)
+			(hide yes)
+			(show_name no)
+			(do_not_autoplace no)
+			(effects
+				(font
+					(size 1.27 1.27)
+				)
+			)
+		)
+		(property "DF_Comment" "NMOS_2SK3018_SOT-23"
+			(at 504.19 137.16 0)
 			(hide yes)
 			(show_name no)
@@
 			)
 		)
-		(property "Value" "D"
+		(property "Value" "0.57Ohm"
 			(at 514.35 115.5699 90)
 			(show_name no)
@@
 			)
 		)
-		(property "Footprint" "Diode_SMD:D_01005_0402Metric"
+		(property "Footprint" "Inductor_SMD:L_01005_0402Metric"
 			(at 511.81 114.3 0)
 			(hide yes)
@@
 			)
 		)
-		(property "Description" "Diode"
+		(property "Description" "Resistor"
 			(at 511.81 114.3 0)
 			(hide yes)
@@
 			)
 		)
-		(property "Sim.Device" "D"
+		(property "Sim.Device" ""
 			(at 511.81 114.3 0)
 			(hide yes)
@@
 			)
 		)
-		(property "Sim.Pins" "1=K 2=A"
+		(property "Sim.Pins" ""
 			(at 511.81 114.3 0)
 			(hide yes)
@@
 			)
 		)
-		(property "Value" "1uF"
+		(property "Value" "220nF"
 			(at 508 102.87 90)
 			(show_name no)
@@
 			)
 		)
-		(property "Value" "220nF"
+		(property "Value" "PESD24VS1UL-N"
 			(at 488.188 142.24 0)
 			(show_name no)
@@
 			)
 		)
-		(property "Footprint" "A_HDJ_Library:C_0603_1608Metric"
+		(property "Footprint" "A_HDJ_Library:D_0402_1005Metric"
 			(at 493.0648 137.16 0)
 			(hide yes)
@@
 			)
 		)
-		(property "Buy_Link" ""
+		(property "Buy_Link" "https://item.szlcsc.com/393990.html"
 			(at 494.03 140.97 0)
 			(hide yes)
@@
 			)
 		)
-		(property "DF_Comment" "贴片电容0603-22uF-10V-X5R(0603)"
+		(property "DF_Comment" "单向静电保护二极管_PESD24VS1UL-N_DFN1006"
 			(at 494.03 140.97 0)
 			(hide yes)
@@
 			)
 		)
-		(property "SCH_Show_Footprint" "C603"
+		(property "SCH_Show_Footprint" "D0402"
 			(at 494.03 140.97 0)
 			(hide yes)
@@
 			)
 		)
-		(property "Value" "0.57Ohm"
+		(property "Value" "TPS61165DBV"
 			(at 515.62 136.906 90)
 			(show_name no)
@@
 			)
 		)
-		(property "Footprint" "Inductor_SMD:L_01005_0402Metric"
+		(property "Footprint" "Package_SON:WSON-6-1EP_2x2mm_P0.65mm_EP1x1.6mm"
 			(at 515.62 136.398 90)
 			(hide yes)
@@
 			)
 		)
-		(property "Datasheet" ""
+		(property "Datasheet" "https://www.ti.com/lit/ds/symlink/tps61165.pdf"
 			(at 515.62 134.62 0)
 			(hide yes)
@@
 			)
 		)
-		(property "Description" "Resistor"
+		(property "Description" "High-Brightness, White LED Driver, 3V to 18V input voltage range, internal switch, constant current, up to 38V/1.2A output, SOT-23-6"
 			(at 515.62 134.62 0)
 			(hide yes)
@@
 			)
 		)
-		(property "Value" "2004850740"
+		(property "Value" "SS54"
 			(at 466.09 101.5999 0)
 			(show_name no)
@@
 			)
 		)
-		(property "Footprint" "200485-0740:CON_2004850740"
+		(property "Footprint" "Diode_SMD:D_SMA"
 			(at 452.12 43.18 0)
 			(hide yes)
@@
 			)
 		)
-		(property "Datasheet" "https://www.molex.com/en-us/products/part-detail-pdf/2004850740?display=pdf"
+		(property "Datasheet" ""
 			(at 452.12 43.18 0)
 			(hide yes)
@@
 		)
 		(property "Description" ""
+			(at 452.12 43.18 0)
+			(hide yes)
+			(show_name no)
+			(do_not_autoplace no)
+			(effects
+				(font
+					(size 1.27 1.27)
+				)
+			)
+		)
+		(property "DF_Comment" "二极管-SS54-SMA(SMA)"
+			(at 452.12 43.18 0)
+			(hide yes)
+			(show_name no)
+			(do_not_autoplace no)
+			(effects
+				(font
+					(size 1.27 1.27)
+				)
+			)
+		)
+		(property "SCH_Show_Footprint" "SMA"
 			(at 452.12 43.18 0)
 			(hide yes)
@@
 			)
 		)
-		(property "Value" "200485-0710"
+		(property "Value" "2.2uF/50V"
 			(at 368.3 85.09 0)
 			(show_name no)
@@
 			)
 		)
-		(property "Footprint" "200485-0710:2004850710"
+		(property "Footprint" "A_HDJ_Library:C_0603_1608Metric"
 			(at 296.24 76.2 0)
 			(hide yes)
@@
 			)
 		)
-		(property "Datasheet" "https://www.molex.com/pdm_docs/sd/2004850710_sd.pdf"
+		(property "Datasheet" ""
 			(at 196.24 76.2 0)
 			(hide yes)
@@
 			)
 		)
-		(property "Description" "FFC & FPC Connectors .50mm Easy-On One TouchST 10Ckt GND"
+		(property "Description" ""
 			(at 391.16 97.79 0)
 			(hide yes)
@@
 			)
 		)
-		(property "Height" "5.7"
+		(property "Height" ""
 			(at -3.76 76.2 0)
 			(hide yes)
@@
 			)
 		)
-		(property "Mouser Part Number" "538-200485-0710"
+		(property "Mouser Part Number" ""
 			(at -103.76 76.2 0)
 			(hide yes)
@@
 			)
 		)
-		(property "Mouser Price/Stock" "https://www.mouser.co.uk/ProductDetail/Molex/200485-0710?qs=81r%252BiQLm7BTVhoZMpMfD8A%3D%3D"
+		(property "Mouser Price/Stock" ""
 			(at -203.76 76.2 0)
 			(hide yes)
@@
 			)
 		)
-		(property "Manufacturer_Name" "Molex"
+		(property "Manufacturer_Name" ""
 			(at -303.76 76.2 0)
 			(hide yes)
@@
 			)
 		)
-		(property "Manufacturer_Part_Number" "200485-0710"
+		(property "Manufacturer_Part_Number" ""
 			(at -403.76 76.2 0)
 			(hide yes)
@@
 				)
 				(justify left top)
+			)
+		)
+		(property "DF_Comment" "贴片电容0603-2.2uF-50V-X5R"
+			(at 391.16 97.79 0)
+			(hide yes)
+			(show_name no)
+			(do_not_autoplace no)
+			(effects
+				(font
+					(size 1.27 1.27)
+				)
+			)
+		)
+		(property "SCH_Show_Footprint" "-- mixed values --"
+			(at 391.16 97.79 0)
+			(hide yes)
+			(show_name no)
+			(do_not_autoplace no)
+			(effects
+				(font
+					(size 1.27 1.27)
+				)
 			)
 		)
@@
 			)
 		)
-		(property "Value" "4.7uF"
+		(property "Value" "0402ESDA-05N"
 			(at 492.76 123.19 90)
 			(show_name no)
@@
 			)
 		)
-		(property "Footprint" "A_HDJ_Library:C_0603_1608Metric"
+		(property "Footprint" "A_HDJ_Library:D_0402_1005Metric"
 			(at 496.57 126.0348 0)
 			(hide yes)
@@
 			)
 		)
-		(property "Datasheet" ""
+		(property "Datasheet" "https://www.onsemi.com/pub/Collateral/ESD9B-D.PDF"
 			(at 492.76 127 0)
 			(hide yes)
@@
 			)
 		)
-		(property "DF_Comment" "贴片电容0603-22uF-10V-X5R(0603)"
+		(property "DF_Comment" "5.0V双向静电保护管_0402ESDA-05N"
 			(at 492.76 127 0)
 			(hide yes)
@@
 			)
 		)
-		(property "SCH_Show_Footprint" "C603"
+		(property "SCH_Show_Footprint" "D0402"
 			(at 492.76 127 0)
 			(hide yes)
