File: LattePanda-Mu-main-idkwhatimdoing-help/Electricals/Examples/[DFR1142]Lite Carrier for LattePanda Mu(V2)/M.2 E&M Key.kicad_sch (KiCad schematic)
At the start: 28 parts, among them J15 Bus_M.2_Socket_M, J16 Bus_M.2_Socket_E

Commit message: Updated M key to be strictly SSD (no SATA)
Parts:
- removed R28: 0R/1%, A_HDJ_Library:R_0402_1005Metric, symbol Device:R
- removed TP2: TestPoint, A_HDJ_Library:TestPoint_Pad_D1.5mm, symbol Connector:TestPoint
Connections:
- no-connect marks 50 -> 52
