File: LattePanda-Mu-main-idkwhatimdoing-help/Electricals/Examples/[DFR1142]Lite Carrier for LattePanda Mu(V2)/HDMI.kicad_sch (KiCad schematic)
At the start: 115 parts, among them J17 200485-0710, J19 SS54, J20 200485-0710, J3 SS54, Q10 HM7533HBPR, Q17 HM7533HBPR, Q18 HM7533HBPR, Q19 AO3407, Q20 HM7533HBPR, Q21 HM7533HBPR, Q22 HM7533HBPR, Q9 AO3407, U13 CH224K, U19 CH224K, U21 CH224K, U22 CH224K, U24 2SK3018, Y2 2N7002, Y3 2N7002

Commit message: Gave each screen a seperate backlight controller (different nit brightness)
Parts:
- added C107: 0402ESDA-05N, A_HDJ_Library:D_0402_1005Metric, symbol Device:C
- added C108: PESD24VS1UL-N, A_HDJ_Library:D_0402_1005Metric, symbol Device:C
- added C109: 220nF, A_HDJ_Library:C_0603_1608Metric, symbol Device:C
- added D43: 0.57Ohm, Inductor_SMD:L_01005_0402Metric, symbol Device:D
- added L4: A915_Y-100M, symbol Device:L
- added R163: TPS61165DBV, Package_SON:WSON-6-1EP_2x2mm_P0.65mm_EP1x1.6mm, symbol Device:R
- added U25: 2SK3018, Package_TO_SOT_SMD:SOT-23, symbol Driver_LED:TPS61165DBV
Connections:
- net +5V: now also C107.2, L4.1, U25.1 (VIN)
- net GND: now also C107.1, C108.1, C109.1, U25.4 (GND)
- net SL_BRI: now also U25.2 (CTRL)
- net LED+ renamed LED_SCT+
- net LED_SCT+: no longer J3.39, J3.40
- net LED- renamed LED_SCT-
- net LED_SCT-: no longer J3.31, J3.32
- new net: D43.2 (A), L4.2, U25.3 (SW)
- new net: R163.1, U25.6 (FB)
- new net: C108.2, U25.5 (COMP)
- new net LED_SCB+: C109.2, D43.1 (K), J3.39, J3.40
- new net LED_SCB-: J3.31, J3.32, R163.2
Other:
- moved on the sheet: C104, C105, C106, D42, L3, R162, U24
