File: LattePanda-Mu-main-idkwhatimdoing-help/Electricals/Examples/[DFR1142]Lite Carrier for LattePanda Mu(V2)/PSU.kicad_sch (KiCad schematic)
At the start: 90 parts, among them J18 USB_C_Receptacle_USB2.0, Q11 2N7002, Q12 2N7002, Q13 2N7002, Q14 2N7002, Q15 2N7002, Q16 AO3407, Q8 2N7002, SW1 SW_Push, SW2 SW_Push, U14 CH224K, U15 SY8253ADC, U16 SY8253ADC, U17 HM7533HBPR

Commit message: Switched Template Carrier board due to issues with the Lattepanda-provided version.
I am not sure what the cause of these "A:DFRobot" missing library footprints are, however the carrier board designed by
youtuber "Ben Makes Everything" has no large changes to the schematic files that I cant handle, and dosen't have this annoying issue. For this reason I
will be using his design as a base. Although I am not using his design directly, I will still link his repository:
https://github.com/BenMakesEverything/Mu_Cyberdeck/tree/main
Thank you BenMakesEverything!
Parts:
- removed TP10: TestPoint, A_HDJ_Library:TestPoint_Pad_D1.5mm, symbol Connector:TestPoint
- added IC1: BQ25792RQMR, BQ25792RQMR, symbol BQ25792RQMR:BQ25792RQMR
- added J21, J22, J23, J24, J25: Conn_01x02_Socket, Connector_JST:JST_PH_B2B-PH-K_1x02_P2.00mm_Vertical, symbol Connector:Conn_01x02_Socket
Connections:
- net VDC: no longer D18.1 (K), D19.1 (K), D20.1 (K)
- new net: D18.1 (K), D19.1 (K), D20.1 (K), IC1.2 (VBUS_1), IC1.3 (VBUS_2)
- new net Connect to LED: IC1.1 (STAT_1)
Other:
- moved on the sheet: C64, C65, C66, C67, C68, C69, C70, C71, C72, C73, C74, C75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
