File: Mu_Cyberdeck_Carrier_KiCad/Mu_Cyberdeck_Carrier_KiCad/PCIe x4.kicad_sch (KiCad schematic)
At the start: 18 parts, among them J2 Bus_PCI_Express_x4

Commit message: Added BQ25798 Power IC
Parts:
- C10, C9: now not fitted
Changed lines of the file:
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@@
 		(on_board no)
 		(in_pos_files yes)
-		(dnp no)
+		(dnp yes)
 		(property "Reference" "C9"
 			(at 284.48 172.72 90)
@@
 		(on_board no)
 		(in_pos_files yes)
-		(dnp no)
+		(dnp yes)
 		(property "Reference" "C10"
 			(at 289.56 172.72 90)
