File: Mu_Cyberdeck_Carrier_KiCad/Mu_Cyberdeck_Carrier_KiCad/PSU.kicad_sch (KiCad schematic)
At the start: 88 parts, among them J18 USB_C_Receptacle_USB2.0, J78 Screw_Terminal_01x02, Q5 2N7002, Q6 2N7002, Q7 NCE30P28Q, Q8 2N7002, SW1 SW_Push, SW2 SW_Push, U13 TL431DBZ, U14 CH224K, U15 SY8253ADC, U16 SY8253ADC

Commit message: Added BQ25798 Power IC
Parts:
- removed C62, C63: 1uF/16V, A_HDJ_Library:C_0402_1005Metric, symbol Device:C
- removed D15, D16, D17: SS54, A_HDJ_Library:D_SMA, symbol Device:D_Schottky
- removed D23: LED_G, A_HDJ_Library:LED_0603_1608Metric, symbol Device:LED
- removed DC78: DC-042C-W-2.0, easyeda2kicad:DC-IN-TH_DC-042C-W-2.0, symbol easyeda2kicad:DC-042C-W-2.0
- removed J78: Screw_Terminal_01x02, TerminalBlock:TerminalBlock_bornier-2_P5.08mm, symbol Connector:Screw_Terminal_01x02
- removed Q5, Q6: 2N7002, A_HDJ_Library:SOT-23, symbol Transistor_FET:2N7002
- removed Q7: NCE30P28Q, A_HDJ_Library:MOSFET_PDFN8_3.3x3.3, symbol A_HDJ_Library:AON7262E
- removed R38, R40: 10K/1%, A_HDJ_Library:R_0402_1005Metric, symbol Device:R
- removed R39: 2.2K/1%, A_HDJ_Library:R_0402_1005Metric, symbol Device:R
- removed R41, R42, R54: 21.5K/1%, A_HDJ_Library:R_0402_1005Metric, symbol Device:R
- removed R44, R45: 100K/1%, A_HDJ_Library:R_0402_1005Metric, symbol Device:R
- removed TP3, TP4, TP8, TP9: TestPoint, A_HDJ_Library:TestPoint_Pad_D1.5mm, symbol Connector:TestPoint
- removed U13: TL431DBZ, A_HDJ_Library:SOT-23, symbol Reference_Voltage:TL431DBZ
- added C100, C88, C91, C99: 10uF/25V, A_HDJ_Library:C_0603_1608Metric, symbol Device:C
- added C87: 1nF/50V, A_HDJ_Library:C_0402_1005Metric, symbol Device:C
- added C92, C98: 0.1uF/25V, A_HDJ_Library:C_0603_1608Metric, symbol Device:C
- added C93, C97: 47nF/10V, A_HDJ_Library:C_0603_1608Metric, symbol Device:C
- added C94: 4.7uF/10V, A_HDJ_Library:C_0603_1608Metric, symbol Device:C
- added C95, C96: 10uF/10V, A_HDJ_Library:C_0603_1608Metric, symbol Device:C
- added J78, J81, J82, J83, J84: Conn_01x02_Socket, Connector_JST:JST_PH_B2B-PH-K_1x02_P2.00mm_Vertical, symbol Connector:Conn_01x02_Socket
- added Q78, Q79: CSD17303Q5, Package_TO_SOT_SMD:TDSON-8-1, symbol Transistor_FET:CSD17303Q5
- added R61, R62: 10K/1%, A_HDJ_Library:R_0402_1005Metric, symbol Device:R
- added R76: 0.1K/1%, A_HDJ_Library:R_0402_1005Metric, symbol Device:R
- added R77: 3K/1%, A_HDJ_Library:R_0402_1005Metric, symbol Device:R
- added TH78: 10k/1%, symbol Device:Thermistor_NTC
- added U79: BQ25798, Package_DFN_QFN:Texas_RQM0029A_VQFN-29_4x4mm_P0.4mm, symbol Battery_Management:BQ25798
- C61, D10, D11, D12, D13, D14, D18, D19, D20, J18, R36, R37, TP10, U14: now fitted; now in the parts list
- R43: value 56K/1% -> 24K/1%; now fitted; now in the parts list
Connections:
- net GND: now also C100.1, C87.1, C88.1, C91.1, C92.1, C94.2, C98.1, C99.1, R77.1, TH78.1, U79.13 (~{CE}), U79.27 (GND)
- net PWR_C_D+: now also U79.6 (D+)
- net PWR_C_D-: now also U79.7 (D-)
- net VDC: no longer D18.1 (K), D19.1 (K), D20.1 (K), TP10.1
- new net: TH78.2, U79.16 (TS)
- new net: R77.2, U79.20 (PROG)
- new net: C97.1, U79.26 (SW2)
- new net: C97.2, U79.19 (BTST2)
- new net: R62.1, U79.15 (SDA)
- new net: C88.2, C91.2, C92.2, Q78.5 (D), U79.2 (VBUS), U79.3 (VBUS)
- new net: C94.1, D18.1 (K), D19.1 (K), D20.1 (K), Q79.5 (D), TP10.1, U79.17 (ILIM_HIZ), U79.5 (REGN), U79.8 (VAC2), U79.9 (VAC1)
- new net: Q78.1 (S), Q78.2 (S), Q78.3 (S), Q79.1 (S), Q79.2 (S), Q79.3 (S)
- new net: Q78.4 (G), Q79.4 (G), U79.10 (ACDRV2), U79.11 (ACDRV1)
- new net: C100.2, C98.2, C99.2, U79.29 (PMID)
- new net: R76.2, U79.18 (BATP)
- new net: R61.1, U79.14 (SCL)
- new net: C95.2, C96.2, U79.22 (BAT), U79.23 (BAT)
- new net: C93.1, U79.4 (BTST1)
- new net: C93.2, U79.28 (SW1)
- new net: C87.2, U79.24 (SDRV)
- new net BAT+: C95.1, C96.1, J78.1 (Pin_1), J81.1 (Pin_1), J82.1 (Pin_1), J83.1 (Pin_1), J84.1 (Pin_1), R76.1
- new net BAT-: J78.2 (Pin_2), J81.2 (Pin_2), J82.2 (Pin_2), J83.2 (Pin_2), J84.2 (Pin_2)
- new net BAT_SCL: R61.2
- new net BAT_SDA: R62.2
- new net STAT_LED: U79.1 (STAT)
- no-connect marks 5 -> 7
Other:
- note added: "12V PD Input"
- note added: "CH224K get DC 9-20V (12V) power from USB-PD adapter"
- note removed: "12V DC Input(12V 6A-10A)"
- note removed: "15V PD Input"
- note removed: "CH224K get DC 15V power from USB-PD adapter"
- note removed: "PCIe Power Enable LED"
- note removed: "Power for PCIe x4 OVP@13.86V"
- note removed: "soft start"

Commit message: Added TPS61088 Voltage booster.
Parts:
- added C101, C102: 10uF, A_HDJ_Library:C_0603_1608Metric, symbol Device:C
- added C103, C131: 100nF, A_HDJ_Library:C_0603_1608Metric, symbol Device:C
- added C104, C132: 1uF, A_HDJ_Library:C_0603_1608Metric, symbol Device:C
- added C106, C107, C108: 22uF, A_HDJ_Library:C_0603_1608Metric, symbol Device:C
- added C109: 8.2nF, A_HDJ_Library:C_0603_1608Metric, symbol Device:C
- added L78: 1.5uH, symbol Device:L
- added R78: 255K/1%, A_HDJ_Library:R_0402_1005Metric, symbol Device:R
- added R79: 680K/1%, A_HDJ_Library:R_0402_1005Metric, symbol Device:R
- added R87, R88: 105K/1%, A_HDJ_Library:R_0402_1005Metric, symbol Device:R
- added U81: TPS61088RHLR, RHL0020A, symbol TPS61088:TPS61088RHLR
- R43: value 24K/1% -> 56K/1%
Connections:
- net BAT- is gone; now on net GND: J78.2 (Pin_2), J81.2 (Pin_2), J82.2 (Pin_2), J83.2 (Pin_2), J84.2 (Pin_2)
- net GND: now also C101.1, C102.1, C104.1, C106.1, C107.1, C108.1, C109.1, C131.1, C132.1, R87.1, R88.2, U81.13 (MODE), U81.20 (AGND), U81.21 (PGND)
- net VDC: now also C106.2, C107.2, C108.2, R79.2, U81.14 (VOUT), U81.15 (VOUT), U81.16 (VOUT)
- net at U79.25 (SYS): now also C101.2, C102.2, C131.2, L78.1, U81.9 (VIN)
- new net: R79.1, R87.2, U81.17 (FB)
- new net: C103.2, L78.2, R78.1, U81.4 (SW), U81.5 (SW), U81.6 (SW), U81.7 (SW)
- new net: R78.2, U81.3 (FSW)
- new net: C109.2, U81.10 (SS)
- new net: C103.1, U81.8 (BOOT)
- new net: R88.1, U81.19 (ILIM)
- new net: C104.2, C132.2, U81.1 (VCC), U81.2 (EN)
- new net: U81.11 (NC), U81.12 (NC)
- no-connect marks 7 -> 8
Other:
- moved on the sheet: C64, C65, C66, C67, C68, C69, C70, C71, C72, C73, C74, C75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

Commit message: PSU Complete!
Parts:
- removed J78, J81, J82, J83, J84: Conn_01x02_Socket, Connector_JST:JST_PH_B2B-PH-K_1x02_P2.00mm_Vertical, symbol Connector:Conn_01x02_Socket
- added J85: JST_XHP2_Battery1, Connector_JST:JST_XH_B2B-XH-A_1x02_P2.50mm_Vertical, symbol Connector:Conn_01x02_Socket
- added J86: JST_XHP2_Battery2, Connector_JST:JST_XH_B2B-XH-A_1x02_P2.50mm_Vertical, symbol Connector:Conn_01x02_Socket
- added J87: JST_XHP2_Battery3, Connector_JST:JST_XH_B2B-XH-A_1x02_P2.50mm_Vertical, symbol Connector:Conn_01x02_Socket
- added J88: JST_XHP2_Battery4, Connector_JST:JST_XH_B2B-XH-A_1x02_P2.50mm_Vertical, symbol Connector:Conn_01x02_Socket
- added J89: JST_XHP2_Battery5, Connector_JST:JST_XH_B2B-XH-A_1x02_P2.50mm_Vertical, symbol Connector:Conn_01x02_Socket
Connections:
- net BAT+: now also J85.1 (Pin_1), J86.1 (Pin_1), J87.1 (Pin_1), J88.1 (Pin_1), J89.1 (Pin_1)
- net GND: now also J85.2 (Pin_2), J86.2 (Pin_2), J87.2 (Pin_2), J88.2 (Pin_2), J89.2 (Pin_2)
