File: Mu_Cyberdeck_Carrier_KiCad/Mu_Cyberdeck_Carrier_KiCad/PSU.kicad_sch (KiCad schematic)
At the start: 105 parts, among them J18 USB_C_Receptacle_USB2.0, J85 JST_XHP2_Battery1, J86 JST_XHP2_Battery2, J87 JST_XHP2_Battery3, J88 JST_XHP2_Battery4, J89 JST_XHP2_Battery5, Q78 CSD17303Q5, Q79 CSD17303Q5, Q8 2N7002, SW1 SW_Push, SW2 SW_Push, U14 CH224K, U15 SY8253ADC, U16 SY8253ADC, U79 BQ25798, U81 TPS61088RHLR

Commit message: Added 'BQ27441DRZT-G1A' fuel guage IC.
Parts:
- removed C101: 10uF, A_HDJ_Library:C_0603_1608Metric, symbol Device:C
- added C136, C137: 1uF, A_HDJ_Library:C_0603_1608Metric, symbol Device:C
- added C138: 0.47uF, A_HDJ_Library:C_0603_1608Metric, symbol Device:C
- added R89, R90, R91, R92: 10K/1%, A_HDJ_Library:R_0402_1005Metric, symbol Device:R
- added R93: 10mO/1%, Resistor_SMD:R_2512_6332Metric, symbol Device:R
- added U82: BQ27441DRZT-G1A, Package_SON:Texas_S-PDSO-N12, symbol Battery_Management:BQ27441DRZT-G1A
- C102, C131: DF_Comment 贴片电容0603-10uF-10V-X5R(0603) -> 贴片电容0603-100nF-10V-X5R(0603)
- C103: DF_Comment 贴片电容0603-22uF-10V-X5R(0603) -> 贴片电容0603-100nF-10V-X5R(0603)
- C104: value 1uF -> 10uF; DF_Comment 贴片电容0603-10uF-10V-X5R(0603) -> 贴片电容0603-100nF-10V-X5R(0603)
- C106, C107, C108: DF_Comment 贴片电容0603-10uF-10V-X5R(0603) -> 贴片电容0603-22uF-10V-X5R(0603)
- C109: DF_Comment 贴片电容0603-10uF-10V-X5R(0603) -> 贴片电容0603-8.2nF-10V-X5R(0603)
- C132: DF_Comment 贴片电容0603-10uF-10V-X5R(0603) -> 贴片电容0603-1uF-10V-X5R(0603)
- C87: DF_Comment 贴片电容0402-10UF-10V-X5R_GRM155R61A106ME44D -> 贴片电容0402-1nF-50V-X5R
- R76: value 0.1K/1% -> 100R/1%; DF_Comment 贴片电阻0402-10K-1% -> 贴片电阻0402-0.1K-1%
- R78: DF_Comment 贴片电阻0402-10K-1% -> 贴片电阻0402-255K-1%
- R79: DF_Comment 贴片电阻0402-10K-1% -> 贴片电阻0402-680K-1%
- R87, R88: DF_Comment 贴片电阻0402-10K-1% -> 贴片电阻0402-105K-1%
Connections:
- net +3V3: now also R89.2, R90.1, R92.2
- net BAT+: now also C137.2, R93.2, U82.6 (BAT), U82.8 (SRP)
- net GND: now also C136.1, C137.1, C138.1, R91.1, R93.1, U82.3 (V_{SS}), U82.7 (SRN)
- net at C132.2, U81.1 (VCC), U81.2 (EN): now also C136.2; no longer C104.2
- net at C102.2, C131.2, L78.1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: now also C104.2
- new net: R91.2, U82.10 (BIN)
- new net: C138.2, U82.5 (V_{DD})
- new net RPI_BAT_GPO: R92.1, U82.12 (GPOUT)
- new net RPI_BAT_SCL: R89.1, U82.1 (SDA)
- new net RPI_BAT_SDA: R90.2, U82.2 (SCL)
Other:
- moved on the sheet: J85, J86, J87, J88, J89, JP79, R87
