File: Mu_Cyberdeck_Carrier_KiCad/Mu_Cyberdeck_Carrier_KiCad/_autosave-PSU.kicad_sch (KiCad schematic)
At the start: 105 parts, among them J18 USB_C_Receptacle_USB2.0, J85 JST_XHP2_Battery1, J86 JST_XHP2_Battery2, J87 JST_XHP2_Battery3, J88 JST_XHP2_Battery4, J89 JST_XHP2_Battery5, Q78 CSD17303Q5, Q79 CSD17303Q5, Q8 2N7002, SW1 SW_Push, SW2 SW_Push, U14 CH224K, U15 SY8253ADC, U16 SY8253ADC, U79 BQ25798, U81 TPS61088RHLR

Commit message: Updated every. component. to have accurate description.
Parts:
- removed C101: 10uF, A_HDJ_Library:C_0603_1608Metric, symbol Device:C
- added C136: 1uF, A_HDJ_Library:C_0603_1608Metric, symbol Device:C
- C102, C131: DF_Comment 贴片电容0603-10uF-10V-X5R(0603) -> 贴片电容0603-100nF-10V-X5R(0603)
- C103: DF_Comment 贴片电容0603-22uF-10V-X5R(0603) -> 贴片电容0603-100nF-10V-X5R(0603)
- C104: value 1uF -> 10uF; DF_Comment 贴片电容0603-10uF-10V-X5R(0603) -> 贴片电容0603-100nF-10V-X5R(0603)
- C106, C107, C108: DF_Comment 贴片电容0603-10uF-10V-X5R(0603) -> 贴片电容0603-22uF-10V-X5R(0603)
- C109: DF_Comment 贴片电容0603-10uF-10V-X5R(0603) -> 贴片电容0603-8.2nF-10V-X5R(0603)
- C132: DF_Comment 贴片电容0603-10uF-10V-X5R(0603) -> 贴片电容0603-1uF-10V-X5R(0603)
- C87: DF_Comment 贴片电容0402-10UF-10V-X5R_GRM155R61A106ME44D -> 贴片电容0402-1nF-50V-X5R
- R76: DF_Comment 贴片电阻0402-10K-1% -> 贴片电阻0402-0.1K-1%
- R78: DF_Comment 贴片电阻0402-10K-1% -> 贴片电阻0402-255K-1%
- R79: DF_Comment 贴片电阻0402-10K-1% -> 贴片电阻0402-680K-1%
- R87, R88: DF_Comment 贴片电阻0402-10K-1% -> 贴片电阻0402-105K-1%
Connections:
- net GND: now also C136.1
- net at C132.2, U81.1 (VCC), U81.2 (EN): now also C136.2; no longer C104.2
- net at C102.2, C131.2, L78.1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: now also C104.2
