File: Mu_Cyberdeck_Carrier_KiCad/Mu_Cyberdeck_Carrier_KiCad/LattePanda Module.kicad_sch (KiCad schematic)
At the start: 11 parts, among them J3 Conn_01x03_Pin

Commit message: Added BQ25798 Power IC
Connections:
- net BAT_SCL: now reaches A2.154 (I2C2_SCL)
- net BAT_SDA: now reaches A2.156 (I2C2_SDA)
- no-connect marks 110 -> 108
Changed lines of the file:
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@@
+		)
+	)
+	(text_box "TCP 0 used for HDMI\n"
+		(exclude_from_sim no)
+		(at 175.26 247.65 0)
+		(size 39.37 10.16)
+		(margins 1.905 1.905 1.905 1.905)
+		(stroke
+			(width 0)
+			(type default)
+		)
+		(fill
+			(type none)
+		)
+		(effects
+			(font
+				(size 2.54 2.54)
+				(thickness 0.508)
+				(bold yes)
+			)
+			(justify left top)
 		)
 	)
@@
 	)
 	(no_connect
-		(at 351.79 218.44)
-	)
-	(no_connect
 		(at 351.79 275.59)
 	)
@@
 	)
 	(no_connect
-		(at 351.79 215.9)
-	)
-	(no_connect
 		(at 351.79 71.12)
 	)
@@
 	(wire
 		(pts
+			(xy 383.54 218.44) (xy 351.79 218.44)
+		)
+		(stroke
+			(width 0)
+			(type default)
+		)
+	)
+	(wire
+		(pts
 			(xy 238.76 279.4) (xy 270.51 279.4)
 		)
@@
 		(pts
 			(xy 365.76 256.54) (xy 370.84 256.54)
+		)
+		(stroke
+			(width 0)
+			(type default)
+		)
+	)
+	(wire
+		(pts
+			(xy 383.54 215.9) (xy 351.79 215.9)
 		)
 		(stroke
@@
 		)
 	)
+	(hierarchical_label "BAT_SDA"
+		(shape bidirectional)
+		(at 383.54 215.9 0)
+		(effects
+			(font
+				(size 1.27 1.27)
+			)
+			(justify left)
+		)
+	)
 	(hierarchical_label "HSIO_0_RX+"
 		(shape input)
@@
 		)
 	)
+	(hierarchical_label "BAT_SCL"
+		(shape output)
+		(at 383.54 218.44 0)
+		(effects
+			(font
+				(size 1.27 1.27)
+			)
+			(justify left)
+		)
+	)

Commit message: Added 'BQ27441DRZT-G1A' fuel guage IC.
Parts:
- added J1: BM14B-NSHSS-TBT_LF__SN_, BM14B-NSHSS-TBT:BM14BNSHSSTBTLFSN, symbol BM14B-NSHSS-TBT_LF__SN_:BM14B-NSHSS-TBT_LF__SN_
- added U80: RP2350A, Package_DFN_QFN:QFN-60-1EP_7x7mm_P0.4mm_EP3.4x3.4mm, symbol MCU_RaspberryPi:RP2350A
Connections:
- net GND: now also J1.1, J1.15 (MP_1), J1.16 (MP_2), J1.2
- new net: U80.1 (IOVDD), U80.11 (IOVDD), U80.20 (IOVDD), U80.30 (IOVDD), U80.38 (IOVDD), U80.45 (IOVDD)
- new net: U80.23 (DVDD), U80.39 (DVDD), U80.6 (DVDD)
- new net +3V3: J1.14
- new net Col1: J1.12
- new net Col2: J1.13
- new net Row1: J1.7
- new net Row2: J1.8
- new net Row3: J1.9
- new net Row4: J1.10
- new net Row5: J1.11
- new net SL_BRI: J1.5
- new net SL_VOL: J1.6

Commit message: CTRL Z, R, PWR Cleanup! Changes Made:
CTRL PWR -> Added Ground Plane and Ground Vias. Moved it out of parent folder CTRL_R upto Root.
CTRL Z ->  Removed Unnecessary ZX pin. Added Ground Plane and Ground Vias.
CTRL R -> Cleaned up pin count, from 14 down to 10. Added Ground Plane and Ground Vias. Made some modifications to the board shape.
Parts:
- added J17: BM14B-NSHSS-TBT_LF__SN_, BM14BNSHSSTBTLFSN, symbol BM14B-NSHSS-TBT_LF__SN_:BM14B-NSHSS-TBT_LF__SN_
- added J19, J20: BM04B-NSHSS-TBT_LF__SN_, BM04B-NSHSS-TBT:BM04BNSHSSTBTLFSN, symbol BM04B-NSHSS-TBT_LF__SN_:BM04B-NSHSS-TBT_LF__SN_
Connections:
- net +3V3: now also J17.1
- net Col1: now also J19.4
- net Col2: now also J19.1
- net GND: now also J17.15 (MP_1), J17.16 (MP_2), J17.2, J17.5, J19.5 (MP1), J19.6 (MP2), J20.5 (MP1), J20.6 (MP2)
- net Row1: now also J19.3, J20.3; no longer J1.7
- net Row2: now also J17.8
- net Row3: now also J17.9
- net Row4: now also J17.10
- net Row5: now also J17.11
- net ADC_Y: now reaches J1.3
- net ADC_Y: now also J17.3
- net ADC_X: now reaches J1.4
- net ADC_X: now also J17.4
- new net Col3: J17.12, J20.4
- new net Col4: J17.13, J20.1
- no-connect marks 108 -> 114
