File: CTRL_L/CTRL_L_SLI/CTRL_L_SLI.kicad_pcb (KiCad board)
At the start: 2 copper layers, 44.2 x 23.2 mm, 4 parts, among them J1 BM04B-NSHSS-TBT_LF__SN_

Commit message: Quick Save
Routing:
- net GND: track 46.7 -> 5.20 mm
- removed copper zone on B.Cu, net GND
- removed copper zone on F.Cu, net GND
Changed lines of the file:
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@@
 		)
-	)
-	(segment
-		(start 165.425 86.025)
-		(end 165.425 94.775)
-		(width 0.2)
-		(layer "F.Cu")
-		(net "GND")
-	)
-	(segment
-		(start 165.425 94.775)
-		(end 164 96.2)
-		(width 0.2)
-		(layer "F.Cu")
-		(net "GND")
-	)
-	(segment
-		(start 164 84.6)
-		(end 165.425 86.025)
-		(width 0.2)
-		(layer "F.Cu")
-		(net "GND")
 	)
 	(via
@@
 	(segment
 		(start 152.5 80)
-		(end 152.5 84.7)
-		(width 0.2)
-		(layer "B.Cu")
-		(net "GND")
-	)
-	(segment
-		(start 162.55 83.35)
-		(end 156.6 83.35)
-		(width 0.2)
-		(layer "B.Cu")
-		(net "GND")
-	)
-	(segment
-		(start 163.8 84.6)
-		(end 162.55 83.35)
-		(width 0.2)
-		(layer "B.Cu")
-		(net "GND")
-	)
-	(segment
-		(start 152.5 80)
 		(end 157.7 80)
-		(width 0.2)
-		(layer "B.Cu")
-		(net "GND")
-	)
-	(segment
-		(start 152.5 84.7)
-		(end 164 96.2)
 		(width 0.2)
 		(layer "B.Cu")
@@
 		(net "SL_VOL")
 	)
-	(zone
-		(net "GND")
-		(layer "F.Cu")
-		(name "Ground Plane")
-		(hatch edge 0.5)
-		(connect_pads
-			(clearance 0.5)
-		)
-		(min_thickness 0.25)
-		(fill yes
-			(thermal_gap 0.5)
-			(thermal_bridge_width 0.5)
-			(island_removal_mode 0)
-		)
-		(polygon
-			(pts
-				(xy 151.003 77.598) (xy 195.202 77.597) (xy 195.201 100.772) (xy 151.003 100.775)
-			)
-		)
-	)
-	(zone
-		(net "GND")
-		(layer "B.Cu")
-		(name "Ground Plane")
-		(hatch edge 0.5)
-		(priority 1)
-		(connect_pads
-			(clearance 0.5)
-		)
-		(min_thickness 0.25)
-		(fill yes
-			(thermal_gap 0.5)
-			(thermal_bridge_width 0.5)
-			(island_removal_mode 0)
-		)
-		(polygon
-			(pts
-				(xy 195.202 77.597) (xy 151.003 77.596) (xy 151.004 100.771) (xy 195.202 100.774)
-			)
-		)
-	)
 	(embedded_fonts no)
