File: Motherboard/_autosave-Motherboard.kicad_pcb (KiCad board)
At the start: 4 copper layers, 130 x 85 mm, 342 parts, among them J1 BM09B-NSHSS-TBT_LF__SN_, J15 Bus_M.2_Socket_M, J16 Bus_M.2_Socket_E, J17 BM10B-NSHSS-TBT_LF__SN_, J19 BM04B-NSHSS-TBT_LF__SN_, J20 BM04B-NSHSS-TBT_LF__SN_, J24 200485-0710, J25 BM12B-NSHSS-TBT_LF__SN_, J4 USB3_A_Stacked, J78 Speaker_L, J79 Speaker_R, J80 USB_C_Receptacle_USB2.0_16P, J83 2004850740, J84 FFC2A33-08-T-R, J85 JST_XHP2_Battery1, J86 JST_XHP2_Battery2, J87 JST_XHP2_Battery3, J88 JST_XHP2_Battery4, J89 JST_XHP2_Battery5, J90 2004850740, J91 HDMI_A_1.4, M1 Fan_4pin, Q11 AO3407, Q12 HM7533HBPR, Q23 AO3407, Q24 HM7533HBPR, Q25 HM7533HBPR, Q26 HM7533HBPR, Q27 HM7533HBPR, Q28 HM7533HBPR, Q29 AO3407, Q30 HM7533HBPR, Q31 HM7533HBPR, Q32 HM7533HBPR, Q78 CSD17303Q5, Q79 CSD17303Q5, Q80 2N7002, Q81 2N7002, SW78 SW_Push, SW79 SW_Push, U14 CH224K, U15 SY8253ADC, U16 SY8253ADC, U3 ULC0524P, U78 RP2040, U79 BQ25798, U80 PCM5102A, U81 TPS61088RHLR, U82 BQ27441DRZT-G1A, U83 CP2615-xx-xM, U84 PAM8403D, U85 ADS1015IDGS, U86 TPS62131, U87 STLD40DPUR, U89 D3V3XA4B10LP, U9 ULC0524P, U90 D3V3XA4B10LP, U91 D3V3XA4B10LP, U92 D3V3XA4B10LP, U95 W25Q128JVS, U96 ADV7611, U97 D3V3XA4B10LP, U98 D3V3XA4B10LP, U99 ADV7611, Y81 Crystal_GND24, Y82 Crystal_GND24

Commit message: Switched Screens to use RGB interface, ADV7613 -> ADV7611. Changes WIP
Parts:
- moved Q25 67.0 mm to (170.0, 91.6)
- moved Q24 59.8 mm to (163.5, 89.5), turned to -90 degrees
- moved Q29 22.1 mm to (155.5, 45.1)
Connections:
- Q24 pad 3: Net-(Q24-D) -> /HDMI-LVDS/DDC_SCL
- R174 pad 2: Net-(Q24-D) -> /HDMI-LVDS/DDC_SCL
Routing:
- net +3V3: track 33.3 -> 35.6 mm, vias 4 -> 6
Changed lines of the file:
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@@
 			(layers "F.Cu" "F.Mask" "F.Paste")
 			(roundrect_rratio 0.25)
-			(net "Net-(Q24-D)")
+			(net "/HDMI-LVDS/DDC_SCL")
 			(pintype "passive")
 			(teardrops
@@
 	(footprint "Package_TO_SOT_SMD:SOT-89-3"
 		(layer "F.Cu")
-		(at 104.576001 106.111026)
+		(at 170.030001 91.643026)
 		(descr "SOT-89-3, http://ww1.microchip.com/downloads/en/DeviceDoc/3L_SOT-89_MB_C04-029C.pdf")
 		(tags "SOT-89-3")
@@
 	(footprint "Package_TO_SOT_SMD:SOT-89-3"
 		(layer "F.Cu")
-		(at 104.576001 99.986026)
+		(at 163.490001 89.515526 -90)
 		(descr "SOT-89-3, http://ww1.microchip.com/downloads/en/DeviceDoc/3L_SOT-89_MB_C04-029C.pdf")
 		(tags "SOT-89-3")
 		(property "Reference" "Q24"
-			(at 0 -3.5 0)
+			(at 0 -3.5 90)
 			(layer "F.SilkS")
 			(effects
@@
 		)
 		(property "Value" "HM7533HBPR"
-			(at 0 3.5 0)
+			(at 0 3.5 90)
 			(layer "F.Fab")
 			(effects
@@
 		)
 		(property "Datasheet" ""
-			(at 0 0 0)
+			(at 0 0 270)
 			(unlocked yes)
 			(layer "F.Fab")
@@
 		)
 		(property "Description" "高压LDO_HM7533HBPR_SOT89"
-			(at 0 0 0)
+			(at 0 0 270)
 			(unlocked yes)
 			(layer "F.Fab")
@@
 		)
 		(property "Buy_Link" ""
-			(at 0 0 0)
+			(at 0 0 270)
 			(unlocked yes)
 			(layer "F.Fab")
@@
 		)
 		(property "DF_Comment" "高压LDO_HM7533HBPR_SOT89"
-			(at 0 0 0)
+			(at 0 0 270)
 			(unlocked yes)
 			(layer "F.Fab")
@@
 		)
 		(property "SCH_Show_Footprint" ""
-			(at 0 0 0)
+			(at 0 0 270)
 			(unlocked yes)
 			(layer "F.Fab")
@@
 		)
 		(property "Field-1" ""
-			(at 0 0 0)
+			(at 0 0 270)
 			(unlocked yes)
 			(layer "F.Fab")
@@
 		(duplicate_pad_numbers_are_jumpers no)
 		(fp_line
-			(start -1.22 -2.36)
-			(end 1.36 -2.36)
+			(start 1.36 2.36)
+			(end -1.36 2.36)
 			(stroke
 				(width 0.12)
@@
 		)
 		(fp_line
-			(start 1.36 -1.38)
-			(end 1.36 -2.36)
+			(start 1.36 1.38)
+			(end 1.36 2.36)
 			(stroke
 				(width 0.12)
@@
 		)
 		(fp_line
-			(start 1.36 1.38)
-			(end 1.36 2.36)
+			(start 1.36 -1.38)
+			(end 1.36 -2.36)
 			(stroke
 				(width 0.12)
@@
 		)
 		(fp_line
-			(start 1.36 2.36)
-			(end -1.36 2.36)
+			(start -1.22 -2.36)
+			(end 1.36 -2.36)
 			(stroke
 				(width 0.12)
@@
 		(fp_line
 			(start -2.85 2.5)
-			(end -2.85 -2.5)
+			(end 2.25 2.5)
 			(stroke
 				(width 0.05)
@@
 		(fp_line
 			(start -2.85 2.5)
-			(end 2.25 2.5)
+			(end -2.85 -2.5)
 			(stroke
 				(width 0.05)
@@
 		(fp_line
 			(start 2.25 -2.5)
-			(end -2.85 -2.5)
+			(end 2.25 2.5)
 			(stroke
 				(width 0.05)
@@
 		(fp_line
 			(start 2.25 -2.5)
-			(end 2.25 2.5)
+			(end -2.85 -2.5)
 			(stroke
 				(width 0.05)
@@
 		)
 		(fp_line
-			(start -1.25 -1.25)
-			(end -0.25 -2.25)
+			(start -1.25 2.25)
+			(end -1.25 -1.25)
 			(stroke
 				(width 0.1)
@@
 		)
 		(fp_line
-			(start -1.25 2.25)
-			(end -1.25 -1.25)
+			(start 1.25 2.25)
+			(end -1.25 2.25)
 			(stroke
 				(width 0.1)
@@
 		)
 		(fp_line
-			(start -0.25 -2.25)
-			(end 1.25 -2.25)
+			(start -1.25 -1.25)
+			(end -0.25 -2.25)
 			(stroke
 				(width 0.1)
@@
 		)
 		(fp_line
-			(start 1.25 -2.25)
-			(end 1.25 2.25)
+			(start -0.25 -2.25)
+			(end 1.25 -2.25)
 			(stroke
 				(width 0.1)
@@
 		)
 		(fp_line
-			(start 1.25 2.25)
-			(end -1.25 2.25)
+			(start 1.25 -2.25)
+			(end 1.25 2.25)
 			(stroke
 				(width 0.1)
@@
 		)
 		(fp_text user "${REFERENCE}"
-			(at 0.2 0 90)
+			(at 0.2 0 0)
 			(layer "F.Fab")
 			(effects
@@
 		)
 		(pad "1" smd roundrect
-			(at -1.95 -1.5)
+			(at -1.95 -1.5 270)
 			(size 1.3 0.9)
 			(layers "F.Cu" "F.Mask" "F.Paste")
@@
 		)
 		(pad "2" smd custom
-			(at -1.8625 0)
+			(at -1.8625 0 270)
 			(size 1.475 0.9)
 			(layers "F.Cu" "F.Mask" "F.Paste")
@@
 		)
 		(pad "3" smd roundrect
-			(at -1.95 1.5)
+			(at -1.95 1.5 270)
 			(size 1.3 0.9)
 			(layers "F.Cu" "F.Mask" "F.Paste")
 			(roundrect_rratio 0.25)
-			(net "Net-(Q24-D)")
+			(net "/HDMI-LVDS/DDC_SCL")
 			(pinfunction "D_3")
 			(pintype "passive")
@@
 	(footprint "Package_TO_SOT_SMD:SOT-23"
 		(layer "F.Cu")
-		(at 135.835001 55.248026)
+		(at 155.460001 45.063026)
 		(descr "SOT, 3 Pin (JEDEC TO-236 Var AB https://www.jedec.org/document_search?search_api_views_fulltext=TO-236)")
 		(tags "SOT TO_SOT_SMD")
@@
 	)
 	(segment
+		(start 181.740001 76.693026)
+		(end 181.620001 76.813026)
+		(width 0.2)
+		(layer "F.Cu")
+		(net "+3V3")
+	)
+	(segment
 		(start 169.830001 79.780436)
 		(end 170.097591 80.048026)
@@
 	)
 	(segment
+		(start 178.000002 67.130025)
+		(end 178.000002 68.473027)
+		(width 0.2)
+		(layer "F.Cu")
+		(net "+3V3")
+	)
+	(segment
 		(start 159.590001 76.513026)
 		(end 163.300001 76.513026)
@@
 	)
 	(segment
+		(start 181.740001 76.083026)
+		(end 181.740001 76.693026)
+		(width 0.2)
+		(layer "F.Cu")
+		(net "+3V3")
+	)
+	(segment
 		(start 164.980001 85.473026)
 		(end 164.480001 85.473026)
@@
 	)
 	(segment
+		(start 178.000002 68.473027)
+		(end 178.150001 68.623026)
+		(width 0.2)
+		(layer "F.Cu")
+		(net "+3V3")
+	)
+	(segment
 		(start 161.115001 81.548026)
 		(end 161.130001 81.533026)
@@
 	)
 	(via
+		(at 178.150001 68.623026)
+		(size 0.4)
+		(drill 0.2)
+		(layers "F.Cu" "B.Cu")
+		(net "+3V3")
+	)
+	(via
 		(at 169.835001 81.538026)
 		(size 0.5)
@@
 	)
 	(via
+		(at 181.620001 76.813026)
+		(size 0.4)
+		(drill 0.2)
+		(layers "F.Cu" "B.Cu")
+		(net "+3V3")
+	)
+	(via
 		(at 164.480001 84.333026)
 		(size 0.4)
@@
 			)
 		)
+	)
+	(zone
+		(net "+3V3")
+		(layer "F.Cu")
+		(hatch none 0.1)
+		(priority 30000)
+		(attr
+			(teardrop
+				(type padvia)
+			)
+		)
+		(connect_pads yes
+			(clearance 0)
+		)
+		(min_thickness 0.0254)
+		(fill yes
+			(island_removal_mode 1)
+		)
+		(polygon
+			(pts
+				(xy 181.840001 76.673026) (xy 181.857918 76.593808) (xy 181.910281 76.497306) (xy 181.958704 76.412933)
+				(xy 182.009344 76.306602) (xy 181.740001 76.082026) (xy 181.470658 76.306602) (xy 181.552332 76.46794)
+				(xy 181.569721 76.497306) (xy 181.619935 76.588859) (xy 181.634673 76.630734) (xy 181.640001 76.673026)
+			)
+		)
