File: Motherboard/HDMI.kicad_sch (KiCad schematic)
At the start: 122 parts, among them J21 SS54, J22 200485-0710, J23 SS54, J24 200485-0710, Q11 AO3407, Q12 HM7533HBPR, Q23 AO3407, Q24 HM7533HBPR, Q25 HM7533HBPR, Q26 HM7533HBPR, Q27 HM7533HBPR, Q28 HM7533HBPR, U18 CH224K, U26 2SK3018, U27 CH224K, U28 CH224K, U30 2SK3018, U31 CH224K, Y4 2N7002, Y5 2N7002

Commit message: Added stereo Audio using CP2615 > PCM5102A > PAM8403D through USB (Mu has dysfunctional I2S)
Changed lines of the file:
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@@
 	)
 	(junction
+		(at 167.64 252.73)
+		(diameter 0)
+		(color 0 0 0 0)
+	)
+	(junction
 		(at 730.25 198.12)
 		(diameter 0)
@@
 	)
 	(junction
-		(at 167.64 252.73)
-		(diameter 0)
-		(color 0 0 0 0)
-	)
-	(junction
 		(at 730.25 167.64)
 		(diameter 0)
@@
 	(wire
 		(pts
+			(xy 165.1 252.73) (xy 167.64 252.73)
+		)
+		(stroke
+			(width 0)
+			(type default)
+		)
+	)
+	(wire
+		(pts
 			(xy 552.45 254) (xy 552.45 248.92)
 		)
@@
 	(symbol
 		(lib_id "power:+5V")
-		(at 167.64 252.73 90)
+		(at 165.1 252.73 90)
 		(unit 1)
 		(body_style 1)
@@
 		(fields_autoplaced yes)
 		(property "Reference" "#PWR0280"
-			(at 171.45 252.73 0)
+			(at 168.91 252.73 0)
 			(hide yes)
 			(show_name no)
@@
 		)
 		(property "Value" "+5V"
-			(at 163.83 252.7299 90)
+			(at 161.29 252.7299 90)
 			(show_name no)
 			(do_not_autoplace no)
@@
 		)
 		(property "Footprint" ""
-			(at 167.64 252.73 0)
+			(at 165.1 252.73 0)
 			(hide yes)
 			(show_name no)
@@
 		)
 		(property "Datasheet" ""
-			(at 167.64 252.73 0)
+			(at 165.1 252.73 0)
 			(hide yes)
 			(show_name no)
@@
 		)
 		(property "Description" "Power symbol creates a global label with name \"+5V\""
-			(at 167.64 252.73 0)
+			(at 165.1 252.73 0)
 			(hide yes)
 			(show_name no)

Commit message: Motherboard Complete (aside from parts-BOM associations)
Parts:
- removed Y4, Y5: 2N7002, Package_TO_SOT_SMD:SOT-23, symbol Oscillator:SiT8008xx-1x-xxE
- added Y79, Y80: SiT8008xx-1x-xxE, Oscillator:Oscillator_SMD_SiT_PQFN-4Pin_2.5x2.0mm, symbol Oscillator:SiT8008xx-1x-xxE
Connections:
- net +3V3: now also U29.F3 (TVDD), U32.F3 (TVDD), Y79.1 (OE), Y79.4 (Vdd), Y80.1 (OE), Y80.4 (Vdd)
- net GND: now also Y79.2 (GND), Y80.2 (GND)
- net at U29.A5 (XTALP): now also Y79.3 (OUT)
- net at U32.A5 (XTALP): now also Y80.3 (OUT)

Commit message: Quick Save
Parts:
- removed C128: 0402ESDA-05N, A_HDJ_Library:D_0402_1005Metric, symbol Device:C
- removed C129: PESD24VS1UL-N, A_HDJ_Library:D_0402_1005Metric, symbol Device:C
- removed C130: 220nF, A_HDJ_Library:C_0603_1608Metric, symbol Device:C
- removed D53: 0.57Ohm, Inductor_SMD:L_01005_0402Metric, symbol Device:D
- removed J21, J23: SS54, Diode_SMD:D_SMA, symbol 200485-0740:2004850740
- removed J22: 200485-0710, 2004850710, symbol 200485-0710:200485-0710
- removed L6: A915_Y-100M, symbol Device:L
- removed R179, R209: TPS61165DBV, Package_SON:WSON-6-1EP_2x2mm_P0.65mm_EP1x1.6mm, symbol Device:R
- removed R180, R181, R182, R183, R184, R185, R186, R187, R188, R189, R190, R191, R192, R193, R210, R211, R212, R213, R214, R215, R216, R217, R218, R219, R220, R221, R222, R223: 1k, symbol Device:R
- removed R82, R84: 10k, symbol Device:R
- removed U18, U27, U28, U31: CH224K, A_HDJ_Library:ESSOP-10-1EP_3.9x5mm_P1.0mm_EP3.2x2.3, symbol Power_Protection:D3V3XA4B10LP
- removed U26, U30: 2SK3018, Package_TO_SOT_SMD:SOT-23, symbol Driver_LED:TPS61165DBV
- removed U29, U32: (no value), Connector_PinHeader_2.54mm:PinHeader_2x03_P2.54mm_Vertical, symbol ADV7613WBBCZ:ADV7613WBBCZ
- added C164: 4.7uF, A_HDJ_Library:D_0402_1005Metric, symbol Device:C
- added C165: 220nF, A_HDJ_Library:D_0402_1005Metric, symbol Device:C
- added C166: 220nF, A_HDJ_Library:C_0603_1608Metric, symbol Device:C
- added D54: 0.57Ohm, Inductor_SMD:L_01005_0402Metric, symbol Device:D
- added J82: 2004850740, CON_2004850740, symbol 200485-0740:2004850740
- added J83: 2004850740, 200485-0740:CON_2004850740, symbol 200485-0740:2004850740
- added J84: FFC2A33-08-T-R, FFC2A33-08-T-R:FFC2A3308TR, symbol FFC2A33-08-T-R:FFC2A33-08-T-R
- added L7: A915_Y-100M, symbol Device:L
- added R100, R101: 0.57R/1%, A_HDJ_Library:R_0402_1005Metric, symbol Device:R
- added R102, R103: 10K/1%, A_HDJ_Library:R_0402_1005Metric, symbol Device:R
- added R104, R105, R106, R107, R108, R109, R110, R111, R112, R113, R114, R115, R116, R117, R118, R119, R120, R121, R122, R123, R124, R125, R126, R127, R128, R129, R130, R131: 1K/1%, A_HDJ_Library:R_0402_1005Metric, symbol Device:R
- added U87, U88: ADV7613WBBCZ, ADV7613:BC_100_4_ADI, symbol ADV7613WBBCZ:ADV7613WBBCZ
- added U89, U90, U91, U92: D3V3XA4B10LP, Package_DFN_QFN:Diodes_UDFN-10_1x2.5mm_P0.5mm, symbol Power_Protection:D3V3XA4B10LP
- added U93, U94: TPS61165DBV, Package_TO_SOT_SMD:SOT-23-6, symbol Driver_LED:TPS61165DBV
- C118: value 0402ESDA-05N -> 4.7uF
- C119: value PESD24VS1UL-N -> 220nF
- C120: DF_Comment 贴片电容0603-22uF-10V-X5R(0603) -> 贴片电容0603-220nF-10V-X5R(0603)
- D44, D45, D46, D49, D50, D51: now not fitted; now left out of the parts list
Connections:
- net +1V8: now also U87.A6 (PVDD), U87.B7 (INT), U87.C3 (CVDD), U87.C6 (DVDD), U87.D3 (CVDD), U87.D6 (DVDD), U87.E3 (CVDD), U87.E6 (DVDD), U87.E7 (DVDD), U87.G1 (CVDD), U87.G2 (CVDD), U87.H2 (LTX_VDD), U87.H3 (LTX_VDD), U87.H6 (LTX_VDD), U87.H7 (LTX_VDD), U88.A6 (PVDD), U88.B7 (INT), U88.C3 (CVDD), U88.C6 (DVDD), U88.D3 (CVDD), U88.D6 (DVDD), U88.E3 (CVDD), U88.E6 (DVDD), U88.E7 (DVDD), U88.G1 (CVDD), U88.G2 (CVDD), U88.H2 (LTX_VDD), U88.H3 (LTX_VDD), U88.H6 (LTX_VDD), U88.H7 (LTX_VDD)
- net +3V3: now also J82.2, J82.3, J82.33, J82.34, J82.5, J82.6, J83.2, J83.3, J83.33, J83.34, J83.5, J83.6, J84.3, R102.1, R103.2, U87.F3 (TVDD), U87.F7 (DVDDIO), U87.G3 (TVDD), U87.G7 (DVDDIO), U88.F3 (TVDD), U88.F7 (DVDDIO), U88.G3 (TVDD), U88.G7 (DVDDIO)
- net +5V: now also C164.2, L7.1, U87.B1 (RXA_5V), U88.B1 (RXA_5V), U93.1 (VIN), U94.1 (VIN)
- net DDC_SCL: now also U87.A3 (DDCA_SCL), U88.A3 (DDCA_SCL)
- net DDC_SDA: now also U87.A2 (DDCA_SDA), U88.A2 (DDCA_SDA)
- net DDIB_SCL: now also U88.A8 (SCL)
- net DDIB_SDA: now also U88.B8 (SDA)
- net GND: now also C164.1, C165.1, C166.1, J82.10, J82.13, J82.16, J82.19, J82.22, J82.25, J82.30, J82.7, J82.G1, J82.G2, J82.P1, J82.P2, J82.P3, J82.P4, J83.10, J83.13, J83.16, J83.19, J83.22, J83.25, J83.30, J83.7, J83.G1, J83.G2, J83.P1, J83.P2, J83.P3, J83.P4, J84.1, J84.8, J84.MP1, J84.MP2, R100.2, R101.2, R104.1, R105.1, R106.1, R107.1, R108.1, R109.1, R110.1, R111.1, R112.1, R113.1, R114.1, R115.1, R116.1, R117.1, R118.1, R119.1, R120.1, R121.1, R122.1, R123.1, R124.1, R125.1, R126.1, R127.1, R128.1, R129.1, R130.1, R131.1, U87.A1 (GND), U87.A10 (GND), U87.A4 (GND), U87.A7 (RESET*), U87.B4 (GND), U87.B6 (CS*), U87.C4 (GND), U87.C5 (GND), U87.D4 (GND), U87.D5 (GND), U87.E4 (GND), U87.E5 (GND), U87.F4 (GND), U87.F5 (GND), U87.F6 (GND), U87.G4 (GND), U87.G5 (GND), U87.G6 (GND), U87.H4 (GND), U87.H5 (GND), U87.K1 (GND), U87.K10 (GND), U88.A1 (GND), U88.A10 (GND), U88.A4 (GND), U88.A7 (RESET*), U88.B4 (GND), U88.B6 (CS*), U88.C4 (GND), U88.C5 (GND), U88.D4 (GND), U88.D5 (GND), U88.E4 (GND), U88.E5 (GND), U88.F4 (GND), U88.F5 (GND), U88.F6 (GND), U88.G4 (GND), U88.G5 (GND), U88.G6 (GND), U88.H4 (GND), U88.H5 (GND), U88.K1 (GND), U88.K10 (GND), U89.3 (VSS), U89.8 (VSS), U90.3 (VSS), U90.8 (VSS), U91.3 (VSS), U91.8 (VSS), U92.3 (VSS), U92.8 (VSS), U93.4 (GND), U94.4 (GND)
- net HPD: now also U87.B2 (HPA_A), U88.B2 (HPA_A)
- net LED_SCB+: now also C166.2, D54.1 (K), J83.39, J83.40
- net LED_SCB-: now also J83.31, J83.32, R101.1, U94.6 (FB)
- net LED_SCT+: now also J82.39, J82.40
- net LED_SCT-: now also J82.31, J82.32, R100.1, U93.6 (FB)
- net SL_BRI: now also U93.2 (CTRL), U94.2 (CTRL)
- net TCP0_SCL: now also J84.4, U87.A8 (SCL)
- net TCP0_SDA: now also J84.5, U87.B8 (SDA)
- net TMDS_CK+: now also U87.C1 (RXA_C+), U88.C1 (RXA_C+), U90.4, U90.7 (NC), U92.4, U92.7 (NC)
- net TMDS_CK-: now also U87.C2 (RXA_C-), U88.C2 (RXA_C-), U90.5, U90.6 (NC), U92.5, U92.6 (NC)
- net TMDS_D0+: now also U87.D1 (RXA_0+), U88.D1 (RXA_0+), U90.1, U90.10 (NC), U92.1, U92.10 (NC)
- net TMDS_D0-: now also U87.D2 (RXA_0-), U88.D2 (RXA_0-), U90.2, U90.9 (NC), U92.2, U92.9 (NC)
- net TMDS_D1+: now also U87.E1 (RXA_1+), U88.E1 (RXA_1+), U89.4, U89.7 (NC), U91.4, U91.7 (NC)
- net TMDS_D1-: now also U87.E2 (RXA_1-), U88.E2 (RXA_1-), U89.5, U89.6 (NC), U91.5, U91.6 (NC)
- net TMDS_D2+: now also U87.F1 (RXA_2+), U88.F1 (RXA_2+), U89.1, U89.10 (NC), U91.1, U91.10 (NC)
- net TMDS_D2-: now also U87.F2 (RXA_2-), U88.F2 (RXA_2-), U89.2, U89.9 (NC), U91.2, U91.9 (NC)
- net at J24.7: now also R103.1
- net at D48.2 (A), L5.2: now also U93.3 (SW)
- net at C119.2: now also U93.5 (COMP)
- net at Y80.3 (OUT): now also U88.A5 (XTALP)
- net at Y79.3 (OUT): now also U87.A5 (XTALP)
- new net: R112.2, U87.E9 (TEST5)
- new net: R121.2, U88.G9 (TEST10)
- new net: R115.2, U87.D7 (TEST2)
- new net: D54.2 (A), L7.2, U94.3 (SW)
- new net: C165.2, U94.5 (COMP)
- new net: R108.2, U87.G8 (TEST9)
- new net: R122.2, U88.G8 (TEST9)
- new net: J84.7, R102.2
- new net: R126.2, U88.E9 (TEST5)
- new net: R130.2, U88.C8 (TEST1)
- new net: R127.2, U88.E8 (TEST4)
- new net: R118.2, U88.H9 (TEST13)
- new net: R123.2, U88.F10 (TEST8)
- new net: R117.2, U87.C7 (TEST0)
- new net: R104.2, U87.H9 (TEST13)
- new net: R128.2, U88.D8 (TEST3)
- new net: R125.2, U88.F8 (TEST6)
- new net: R131.2, U88.C7 (TEST0)
- new net: R129.2, U88.D7 (TEST2)
- new net: R124.2, U88.F9 (TEST7)
- new net: R120.2, U88.G10 (TEST11)
- new net: J83.8, U88.H10 (LTX1_0-)
- new net: R119.2, U88.H8 (TEST12)
- new net: J83.9, U88.J10 (LTX1_0+)
- new net: J83.20, U88.J6 (LTX1_3-)
- new net: J83.17, U88.J7 (LTX1_C-)
- new net: J83.14, U88.J8 (LTX1_2-)
- new net: J83.11, U88.J9 (LTX1_1-)
- new net: J83.21, U88.K6 (LTX1_3+)
- new net: J83.18, U88.K7 (LTX1_C+)
- new net: J83.15, U88.K8 (LTX1_2+)
- new net: J83.12, U88.K9 (LTX1_1+)
- new net: R105.2, U87.H8 (TEST12)
- new net: R116.2, U87.C8 (TEST1)
- new net: R114.2, U87.D8 (TEST3)
- new net: R113.2, U87.E8 (TEST4)
- new net: R109.2, U87.F10 (TEST8)
- new net: R111.2, U87.F8 (TEST6)
- new net: R110.2, U87.F9 (TEST7)
- new net: R106.2, U87.G10 (TEST11)
- new net: R107.2, U87.G9 (TEST10)
- new net TCP0_0+: J82.9, U87.J10 (LTX1_0+)
- new net TCP0_0-: J82.8, U87.H10 (LTX1_0-)
- new net TCP0_1+: J82.12, U87.K9 (LTX1_1+)
- new net TCP0_1-: J82.11, U87.J9 (LTX1_1-)
- new net TCP0_2+: J82.15, U87.K8 (LTX1_2+)
- new net TCP0_2-: J82.14, U87.J8 (LTX1_2-)
- new net TCP0_3+: J82.21, U87.K6 (LTX1_3+)
- new net TCP0_3-: J82.20, U87.J6 (LTX1_3-)
- new net TCP0_C+: J82.18, U87.K7 (LTX1_C+)
- new net TCP0_C-: J82.17, U87.J7 (LTX1_C-)
- no-connect marks 70 -> 68
Other:
- note added: "ADV7613 OBSOLETE TO BE REPLACED"

Commit message: Switched Screens to use RGB interface, ADV7613 -> ADV7611. Changes WIP
Parts:
- removed C118, C164: 4.7uF, A_HDJ_Library:D_0402_1005Metric, symbol Device:C
- removed C119, C165: 220nF, A_HDJ_Library:D_0402_1005Metric, symbol Device:C
- removed C120, C166: 220nF, A_HDJ_Library:C_0603_1608Metric, symbol Device:C
- removed D48, D54: 0.57Ohm, Inductor_SMD:L_01005_0402Metric, symbol Device:D
- removed J82: 2004850740, CON_2004850740, symbol 200485-0740:2004850740
- removed L5, L7: A915_Y-100M, symbol Device:L
- removed R100, R101: 0.57R/1%, A_HDJ_Library:R_0402_1005Metric, symbol Device:R
- removed R105, R106, R107, R108, R109, R110, R111, R112, R113, R114, R115, R116, R117, R118, R119, R120, R121, R122, R123, R124, R125, R126, R127, R128, R129, R130, R131: 1K/1%, A_HDJ_Library:R_0402_1005Metric, symbol Device:R
- removed U87, U88: ADV7613WBBCZ, ADV7613:BC_100_4_ADI, symbol ADV7613WBBCZ:ADV7613WBBCZ
- removed U93, U94: TPS61165DBV, Package_TO_SOT_SMD:SOT-23-6, symbol Driver_LED:TPS61165DBV
- removed Y79, Y80: SiT8008xx-1x-xxE, Oscillator:Oscillator_SMD_SiT_PQFN-4Pin_2.5x2.0mm, symbol Oscillator:SiT8008xx-1x-xxE
- added C101: 4.7uF/35V, A_HDJ_Library:C_0402_1005Metric, symbol Device:C
- added C128, C129, C130, C140, C141, C142, C144, C145: 10uF/10V, A_HDJ_Library:C_0402_1005Metric, symbol Device:C
- added C99: 2.2uF/10V, A_HDJ_Library:C_0402_1005Metric, symbol Device:C
- added D1: 1N5819WS, A_HDJ_Library:D_SOD-323, symbol Diode:1N5819WS
- added D53, D55, D56: Barrel_Jack_Switch, A_HDJ_Library:DC_Jack_DC007B_30V_10A, symbol Diode:ESD9B5.0ST5G
- added D57: 1K/1%, A_HDJ_Library:R_0402_1005Metric, symbol Diode:1N5819WS
- added J90: 2004850740, CON_2004850740, symbol 200485-0740:2004850740
- added J91: HDMI_A_1.4, Connector_Video:HDMI_A_Molex_208658-1001_Horizontal, symbol Connector:HDMI_A_1.4
- added L79: 1.5uH, symbol Device:L
- added Q29: AO3407, Package_TO_SOT_SMD:SOT-23, symbol Transistor_FET:2N7002
- added Q30, Q31, Q32: HM7533HBPR, Package_TO_SOT_SMD:SOT-89-3, symbol Transistor_FET:2N7002
- added R179, R189, R192, R193, R82: 21.5K/1%, A_HDJ_Library:R_0402_1005Metric, symbol Device:R
- added R180, R186: 0R/1%, A_HDJ_Library:R_0402_1005Metric, symbol Device:R
- added R181, R182, R183, R184, R187, R188, R190, R191: 56K/1%, A_HDJ_Library:R_0402_1005Metric, symbol Device:R
- added R185: 2.2K/1%, A_HDJ_Library:R_0402_1005Metric, symbol Device:R
- added R80: 15k/1%, A_HDJ_Library:R_0402_1005Metric, symbol Device:R
- added R84: 8R/1%, A_HDJ_Library:R_0402_1005Metric, symbol Device:R
- added U87: STLD40DPUR, STLD40DPUR:SON_DPUR_STM, symbol STLD40DPUR:STLD40DPUR
- added U96, U99: ADV7611, Package_QFP:LQFP-64-1EP_10x10mm_P0.5mm_EP5x5mm, symbol Interface_HDMI:ADV7611
- added U97, U98: D3V3XA4B10LP, Package_DFN_QFN:Diodes_UDFN-10_1x2.5mm_P0.5mm, symbol Power_Protection:D3V3XA4B10LP
- added Y81, Y82: Crystal_GND24, A_HDJ_Library:Crystal_SMD_3225-4Pin_3.2x2.5mm, symbol Device:Crystal_GND24
- R104: value 1K/1% -> 470R/1%; DF_Comment 贴片电阻0402-1K-1% -> 贴片电阻0402-470R-1%
Connections:
- net DDC_SDA is gone; now on net DDC_SCL: D46.2 (A2), D51.2 (A2), Q25.3 (D), Q27.3 (D), R177.2, R207.2
- net +1V8: now also U96.14 (CVDD), U96.2 (CVDD), U96.24 (DVDD), U96.40 (DVDD), U96.52 (DVDD), U96.57 (PVDD), U96.60 (DVDD), U99.14 (CVDD), U99.2 (CVDD), U99.24 (DVDD), U99.40 (DVDD), U99.52 (DVDD), U99.57 (PVDD), U99.60 (DVDD)
- net +3V3: now also J83.31, J83.4, R104.1, C99.2, J90.31, J90.4, L79.1, Q29.1 (G), Q30.1 (G), Q31.1 (G), R179.1, R82.1, U87.1 (VI), U96.11 (TVDD), U96.23 (DVDDIO), U96.34 (DVDDIO), U96.44 (DVDDIO), U96.5 (TVDD), U96.55 (INT1), U96.56 (~{RESET}), U96.8 (TVDD), U99.11 (TVDD), U99.23 (DVDDIO), U99.34 (DVDDIO), U99.44 (DVDDIO), U99.5 (TVDD), U99.55 (INT1), U99.56 (~{RESET}), U99.8 (TVDD); no longer J83.2, J83.3, J83.33, J83.34, J83.5, J83.6
- net +5V: now also D57.2 (A), J91.18 (+5V), U96.64 (RXA_5V), U99.64 (RXA_5V)
- net 5V_HDMI_VCC: now also D57.1 (K), R189.1, R192.1
- net DDC_SCL: now also D56.2 (A2), J91.15 (SCL), J91.16 (SDA), Q31.3 (D), R192.2, U96.62 (DDCA_SCL), U96.63 (DDCA_SDA), U99.62 (DDCA_SCL), U99.63 (DDCA_SDA)
- net DDIB_SCL: now also U99.53 (SCL)
- net DDIB_SDA: now also U99.54 (SDA)
- net GND: now also J83.29, J83.3, J83.36, C101.1, C99.1, D53.1 (A1), D55.1 (A1), D56.1 (A1), J90.29, J90.3, J90.36, J90.G1, J90.G2, J90.P1, J90.P2, J90.P3, J90.P4, J91.11 (CKS), J91.17 (GND), J91.2 (D2S), J91.5 (D1S), J91.8 (D0S), J91.SH, Q32.2 (S), R180.2, R186.2, R80.2, R84.2, U87.3 (GND), U87.9 (PGND), U96.65 (GND), U97.3 (VSS), U97.8 (VSS), U98.3 (VSS), U98.8 (VSS), U99.65 (GND), Y82.2 (G), Y82.4 (G); no longer J83.10, J83.13, J83.16, J83.19, J83.22, J83.25, J83.30, J83.7, R104.1
- net HPD: now also D55.2 (A2), J91.19 (HPD/HEAC-), R185.2, U96.1 (HPA_A/INT2), U99.1 (HPA_A/INT2)
- net LED_SCB+: now also J83.2; no longer J83.39, J83.40
- net LED_SCB-: now also J83.1; no longer J83.31, J83.32
- net LED_SCT+: now also C101.2, D1.1 (K), J90.2, U87.6 (V0)
- net LED_SCT-: now also J90.1, R84.1, U87.4 (FB)
- net SL_BRI: now also U87.7 (EN)
- net TCP0_SCL: now also U96.53 (SCL)
- net TCP0_SDA: now also U96.54 (SDA)
- net TMDS_CK+: now also U96.3 (RXA_C-); no longer C126.2, R197.1, U90.4, U90.7 (NC)
- net TMDS_CK-: now also U96.4 (RXA_C+); no longer C127.2, R196.1, U90.5, U90.6 (NC)
- net TMDS_D0+: now also U96.13 (RXA_2+); no longer C124.2, R199.1, U90.1, U90.10 (NC)
- net TMDS_D0-: now also U96.7 (RXA_0+); no longer C125.2, R198.1, U90.2, U90.9 (NC)
- net TMDS_D1+: now also U96.12 (RXA_2-); no longer C122.2, R203.1, U89.4, U89.7 (NC)
- net TMDS_D1-: now also U96.6 (RXA_0-); no longer C123.2, R202.1, U89.5, U89.6 (NC)
- net TMDS_D2+: now also U96.9 (RXA_1-); no longer C90.2, R206.1, U89.1, U89.10 (NC)
- net TMDS_D2-: now also U96.10 (RXA_1+); no longer C121.2, R205.1, U89.2, U89.9 (NC)
- net ~{PWR_LED}/~{PSON}: now also R193.1
- net DDIB_INT: now reaches J24.9
- net TCP0_INT: now reaches J84.6
- net DBUG_HPD: now reaches R104.2
- net DBUG_HPD: now also Q29.2 (S)
- net B19: now reaches J83.8
- net B19: now also U99.19 (P19)
- net B20: now reaches J83.9
- net B20: now also U99.18 (P20)
- net B15: now reaches J83.20
- net B15: now also U99.26 (P15)
- net B12: now reaches J83.17
- net B12: now also U99.29 (P12)
- net B9: now reaches J83.14
- net B9: now also U99.32 (P9)
- net B22: now reaches J83.11
- net B22: now also U99.16 (P22)
- net B0: now reaches J83.21
- net B0: now also U99.43 (P0)
- net B13: now reaches J83.18
- net B13: now also U99.28 (P13)
- net B10: now reaches J83.15
- net B10: now also U99.31 (P10)
- net B23: now reaches J83.12
- net B23: now also U99.15 (P23)
- net B2: now reaches J83.23
- net B2: now also U99.41 (P2)
- net B3: now reaches J83.24
- net B3: now also U99.39 (P3)
- net B5: now reaches J83.26
- net B5: now also U99.37 (P5)
- net B6: now reaches J83.27
- net B6: now also U99.36 (P6)
- net B7: now reaches J83.28
- net B7: now also U99.35 (P7)
- new net: Q32.3 (D), R181.2, R182.2, R183.2, R184.2, R186.1, R187.2, R188.2, R190.2, R191.2
- new net: Q29.3 (D), R180.1, R185.1
- new net: D1.2 (A), L79.2, U87.8 (SW)
- new net: D53.2 (A2), Q30.3 (D), R189.2
- new net: Q32.1 (G), R193.2
- new net: R80.1, U87.2 (RSET)
- new net: J90.30, U96.25 (LLC)
- new net: J90.34, U96.45 (DE)
- new net: J90.32, U96.46 (HS)
- new net: J90.33, U96.47 (VS/FIELD/ALSB)
- new net: J83.30, U99.25 (LLC)
- new net: J83.32, U99.46 (HS)
- new net: J83.33, U99.47 (VS/FIELD/ALSB)
- new net: J83.34, U99.45 (DE)
- new net: U99.58 (XTALP), Y82.1
- new net: U99.59 (XTALN), Y82.3
- new net: Y81.2 (G), Y81.4 (G)
- new net B1: J83.22, U99.42 (P1)
- new net B11: J83.16, U99.30 (P11)
- new net B14: J83.19, U99.27 (P14)
- new net B16: J83.5, U99.22 (P16)
- new net B17: J83.6, U99.21 (P17)
- new net B18: J83.7, U99.20 (P18)
- new net B21: J83.10, U99.17 (P21)
- new net B4: J83.25, U99.38 (P4)
- new net B8: J83.13, U99.33 (P8)
- new net DBUG_CK+: C144.2, J91.12 (CK-), R182.1, U98.4, U98.7 (NC)
- new net DBUG_CK-: C145.2, J91.10 (CK+), R181.1, U98.5, U98.6 (NC)
- new net DBUG_D0+: C141.2, J91.7 (D0+), R184.1, U98.1, U98.10 (NC)
- new net DBUG_D0-: C142.2, J91.9 (D0-), R183.1, U98.2, U98.9 (NC)
- new net DBUG_D1+: C130.2, J91.4 (D1+), R188.1, U97.4, U97.7 (NC)
- new net DBUG_D1-: C140.2, J91.6 (D1-), R187.1, U97.5, U97.6 (NC)
- new net DBUG_D2+: C128.2, J91.1 (D2+), R191.1, U97.1, U97.10 (NC)
- new net DBUG_D2-: C129.2, J91.3 (D2-), R190.1, U97.2, U97.9 (NC)
- new net DBUG_SCL: Q30.2 (S), R179.2
- new net DBUG_SDA: Q31.2 (S), R82.2
- new net DBUG_TX0+: C128.1
- new net DBUG_TX0-: C129.1
- new net DBUG_TX1+: C130.1
- new net DBUG_TX1-: C140.1
- new net DBUG_TX2+: C141.1
- new net DBUG_TX2-: C142.1
- new net DBUG_TX3+: C144.1
- new net DBUG_TX3-: C145.1
- new net DDIB_CK+: C126.2, R197.1, U90.4, U90.7 (NC), U99.3 (RXA_C-)
- new net DDIB_CK-: C127.2, R196.1, U90.5, U90.6 (NC), U99.4 (RXA_C+)
- new net DDIB_D0+: C124.2, R199.1, U90.1, U90.10 (NC), U99.13 (RXA_2+)
- new net DDIB_D0-: C125.2, R198.1, U90.2, U90.9 (NC), U99.7 (RXA_0+)
- new net DDIB_D1+: C122.2, R203.1, U89.4, U89.7 (NC), U99.12 (RXA_2-)
- new net DDIB_D1-: C123.2, R202.1, U89.5, U89.6 (NC), U99.6 (RXA_0-)
- new net DDIB_D2+: C90.2, R206.1, U89.1, U89.10 (NC), U99.9 (RXA_1-)
- new net DDIB_D2-: C121.2, R205.1, U89.2, U89.9 (NC), U99.10 (RXA_1+)
- new net P0: J90.21, U96.43 (P0)
- new net P1: J90.22, U96.42 (P1)
- new net P10: J90.15, U96.31 (P10)
- new net P11: J90.16, U96.30 (P11)
- new net P12: J90.17, U96.29 (P12)
- new net P13: J90.18, U96.28 (P13)
- new net P14: J90.19, U96.27 (P14)
- new net P15: J90.20, U96.26 (P15)
- new net P16: J90.5, U96.22 (P16)
- new net P17: J90.6, U96.21 (P17)
- new net P18: J90.7, U96.20 (P18)
- new net P19: J90.8, U96.19 (P19)
- new net P2: J90.23, U96.41 (P2)
- new net P20: J90.9, U96.18 (P20)
- new net P21: J90.10, U96.17 (P21)
- new net P22: J90.11, U96.16 (P22)
- new net P23: J90.12, U96.15 (P23)
- new net P3: J90.24, U96.39 (P3)
- new net P4: J90.25, U96.38 (P4)
- new net P5: J90.26, U96.37 (P5)
- new net P6: J90.27, U96.36 (P6)
- new net P7: J90.28, U96.35 (P7)
- new net P8: J90.13, U96.33 (P8)
- new net P9: J90.14, U96.32 (P9)
- no-connect marks 68 -> 26
Other:
- note added: "ADV7611 Outputs B->G->R 7->0 where B0 is #0 and R7 is #23"
- note added: "Screen Inputs R->G->B 0->7 where R0 is #0 and B7 is #23"
- note removed: "ADV7613 OBSOLETE TO BE REPLACED"
- moved on the sheet: C110, C111, C112, C113, C114, C115, C116, C117, C121, C122, C123, C124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

Commit message: Switched HDMI DBUG and TCP0 back, added I2C Protection circuits, and a lot more random changes/updates/progress
Parts:
- removed D44, D46: Barrel_Jack_Switch, A_HDJ_Library:DC_Jack_DC007B_30V_10A, symbol Diode:ESD9B5.0ST5G
Connections:
- net DDC_SCL: no longer D49.2 (A2), D51.2 (A2), D56.2 (A2), J91.15 (SCL), J91.16 (SDA), Q12.3 (D), Q25.3 (D), Q27.3 (D), Q31.3 (D), R177.2, R192.2, R204.2, R207.2, U96.63 (DDCA_SDA), U99.62 (DDCA_SCL), U99.63 (DDCA_SDA)
- net DDIB_SCL: no longer U99.53 (SCL)
- net DDIB_SDA: no longer U99.54 (SDA)
- net GND: now also Y81.2 (G), Y81.4 (G)
- net HPD: no longer D50.2 (A2), D55.2 (A2), J91.19 (HPD/HEAC-), R185.2, R200.2, U99.1 (HPA_A/INT2)
- net TCP0_SCL: no longer U96.53 (SCL)
- net TCP0_SDA: no longer U96.54 (SDA)
- net DDC1_SCL: now reaches D53.2 (A2), Q30.3 (D), R189.2
- net DDC1_SCL: now also J91.15 (SCL)
- net at U96.58 (XTALP): now also Y81.1
- net at U96.59 (XTALN): now also Y81.3
- new net DDC1_SDA: D56.2 (A2), J91.16 (SDA), Q31.3 (D), R192.2
- new net DDC2_SCL: D49.2 (A2), Q12.3 (D), R204.2, U99.62 (DDCA_SCL)
- new net DDC2_SDA: D51.2 (A2), Q27.3 (D), R207.2, U99.63 (DDCA_SDA)
- new net DDC_SDA: Q25.3 (D), R177.2, U96.63 (DDCA_SDA)
- new net DDIB_ADV_SCL: U99.53 (SCL)
- new net DDIB_ADV_SDA: U99.54 (SDA)
- new net HPD1: D55.2 (A2), J91.19 (HPD/HEAC-), R185.2
- new net HPD2: D50.2 (A2), R200.2, U99.1 (HPA_A/INT2)
- new net TCP0_ADV_SCL: U96.53 (SCL)
- new net TCP0_ADV_SDA: U96.54 (SDA)
Other:
- moved on the sheet: U91, U92, Y81

Commit message: Partial wiring of power path and top screen
Parts:
- J91: LCSC Part (none) -> C916313
Changed lines of the file:
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@@
+			)
+		)
+		(property "LCSC Part" "C916313"
+			(at 447.04 424.18 0)
+			(hide yes)
+			(show_name no)
+			(do_not_autoplace no)
+			(effects
+				(font
+					(size 1.27 1.27)
+				)
 			)
 		)

Commit message: Rewired M.2 M key to fit new location. removed Fan_Temp as the design will move to a passive heatsink.
Parts:
- added R100, R101: 10K/1%, A_HDJ_Library:R_0402_1005Metric, symbol Device:R
Connections:
- net +3V3: now also R100.1, R101.1; no longer J83.31, J90.31
- new net RPi_LCD_EN: J83.31, J90.31, R100.2, R101.2
