File: Motherboard/Motherboard.kicad_pcb (KiCad board)
At the start: 4 copper layers, 110 x 85 mm, 346 parts, among them J1 BM09B-NSHSS-TBT_LF__SN_, J15 Bus_M.2_Socket_M, J16 Bus_M.2_Socket_E, J17 BM10B-NSHSS-TBT_LF__SN_, J19 BM04B-NSHSS-TBT_LF__SN_, J20 BM04B-NSHSS-TBT_LF__SN_, J24 200485-0710, J25 BM12B-NSHSS-TBT_LF__SN_, J4 USB3_A_Stacked, J78 Speaker_L, J79 Speaker_R, J80 USB_C_Receptacle_USB2.0_16P, J83 2004850740, J84 FFC2A33-08-T-R, J85 JST_XHP2_Battery1, J86 JST_XHP2_Battery2, J87 JST_XHP2_Battery3, J88 JST_XHP2_Battery4, J89 JST_XHP2_Battery5, J90 2004850740, J91 HDMI_A_1.4, M1 Fan_4pin, Q11 AO3407, Q12 HM7533HBPR, Q23 AO3407, Q24 HM7533HBPR, Q25 HM7533HBPR, Q26 HM7533HBPR, Q27 HM7533HBPR, Q28 HM7533HBPR, Q29 AO3407, Q30 HM7533HBPR, Q31 HM7533HBPR, Q32 HM7533HBPR, Q78 CSD17303Q5, Q79 CSD17303Q5, Q80 2N7002, Q81 2N7002, SW78 SW_Push, SW79 SW_Push, U10 ULC0524P, U11 ULC0524P, U14 CH224K, U15 SY8253ADC, U16 SY8253ADC, U3 ULC0524P, U78 RP2040, U79 BQ25798, U80 PCM5102A, U81 TPS61088RHLR, U82 BQ27441DRZT-G1A, U83 CP2615-xx-xM, U84 PAM8403D, U85 ADS1015IDGS, U86 TPS62131, U87 STLD40DPUR, U89 D3V3XA4B10LP, U9 ULC0524P, U90 D3V3XA4B10LP, U91 D3V3XA4B10LP, U92 D3V3XA4B10LP, U95 W25Q128JVS, U96 ADV7611, U97 D3V3XA4B10LP, U98 D3V3XA4B10LP, U99 ADV7611, Y81 Crystal_GND24, Y82 Crystal_GND24

Commit message: HDMI-TCP0 Screen wired!
Parts:
- C88, R102: moved to B.Cu
- moved R102 53.2 mm to (204.6, 68.1)
- moved J84 15.3 mm to (203.4, 68.0)
- moved C111 14.8 mm to (164.1, 79.9)
- moved C101 14.8 mm to (163.4, 73.5)
- moved C110 14.8 mm to (164.1, 78.9)
- moved C112 14.8 mm to (166.5, 82.1)
- moved C113 14.8 mm to (166.5, 83.1)
- moved C114 14.8 mm to (165.4, 77.2)
- moved C115 14.8 mm to (165.4, 78.2)
- moved C116 14.8 mm to (168.6, 84.4)
- moved C117 14.8 mm to (168.6, 85.4)
- moved C99 14.8 mm to (172.3, 76.1)
- moved D1 14.8 mm to (165.4, 74.6)
- moved J90 14.8 mm to (154.9, 69.0)
- moved Q23 14.8 mm to (157.9, 91.4)
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Connections:
- A2 pad 124: /LattePanda Module/DDIB_INT -> /HDMI-LVDS/DDIB_INT
- A2 pad 126: /LattePanda Module/TCP0_INT -> /HDMI-LVDS/TCP0_INT
Routing:
- net /HDMI-LVDS/TCP0_SCL: track 0.04 -> 83.4 mm, vias 0 -> 2
- net /HDMI-LVDS/TCP0_SDA: track 0.03 -> 76.9 mm, vias 0 -> 2
- net /HDMI-LVDS/TCP0_INT: track 0.00 -> 46.3 mm, vias 0 -> 1
- net /HDMI-LVDS/TCP0_TX3+: track 15.6 -> 30.6 mm
- net /HDMI-LVDS/TCP0_TX1+: track 18.1 -> 33.0 mm
- net /HDMI-LVDS/TCP0_TX2+: track 19.4 -> 34.4 mm
- net /HDMI-LVDS/TCP0_TX2-: track 19.4 -> 34.4 mm
- net /HDMI-LVDS/TCP0_TX0+: track 19.8 -> 34.6 mm
- net /HDMI-LVDS/TCP0_TX3-: track 15.6 -> 30.5 mm
- net /HDMI-LVDS/TCP0_TX1-: track 18.0 -> 32.9 mm
- net /HDMI-LVDS/TCP0_TX0-: track 19.8 -> 34.6 mm
- net +1V8: track 91.4 -> 94.6 mm
- net +3V3: track 113.1 -> 115.0 mm, vias 19 -> 21
- net Net-(J84-Pad7): track 0.00 -> 1.29 mm, vias 0 -> 1
- net GND: track 63.7 -> 64.2 mm, vias 61 -> 63
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Other:
- board size 110 x 85 mm -> 150 x 85 mm

Commit message: Routed (Mostly) M.2 M/E Key
Parts:
- C49, C50, C89, C91, C98, D9, H8, J15, L3, R3, R30, R33, R34, R35, R99, U86: moved to B.Cu
- C88, U82: moved to F.Cu
- moved C84 186.4 mm to (242.1, 131.1)
- moved D26 186.4 mm to (239.3, 138.7)
- moved R68 186.4 mm to (235.7, 135.1)
- moved R69 186.4 mm to (235.7, 137.1)
- moved R72 186.4 mm to (235.7, 139.1)
- moved TP11 186.4 mm to (238.9, 131.9)
- moved TP12 186.4 mm to (238.9, 135.4)
- moved C157 156.2 mm to (219.6, 114.8), turned to -90 degrees
- moved C156 155.3 mm to (217.3, 115.5)
- moved C158 153.4 mm to (219.7, 108.7), turned to -90 degrees
- moved R10 153.1 mm to (216.1, 117.2), turned to 90 degrees
- moved C154 151.7 mm to (217.6, 106.1)
- moved C151 149.7 mm to (211.1, 113.3), turned to -90 degrees
- moved C150 149.1 mm to (209.5, 113.3), turned to -90 degrees
- moved C155 148.6 mm to (213.1, 105.4), turned to 90 degrees
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Connections:
- net Net-(A2-USB2_P7+) renamed /LattePanda Module/Audio_D+
- net Net-(A2-USB2_P7-) renamed /LattePanda Module/Audio_D-
- net Net-(D23-A) renamed /PSU/9VIn
Routing:
- net +3V3: track 115.0 -> 264.5 mm, vias 21 -> 44
- net GND: track 64.2 -> 154.3 mm, vias 63 -> 98
- net /HDMI-LVDS/DDIB_SCL: track 0.00 -> 47.9 mm, vias 0 -> 3
- net /~{PLT_RST}: track 0.00 -> 46.6 mm, vias 0 -> 4
- net /HDMI-LVDS/DDIB_SDA: track 0.00 -> 46.4 mm, vias 0 -> 3
- net /LattePanda Module/HSIO_3_RX+: track 0.00 -> 44.7 mm, vias 0 -> 1
- net /LattePanda Module/HSIO_3_RX-: track 0.00 -> 44.7 mm, vias 0 -> 1
- net /LattePanda Module/HSIO_3_TX+: track 0.00 -> 43.7 mm, vias 0 -> 1
- net /LattePanda Module/HSIO_3_TX-: track 0.00 -> 43.7 mm, vias 0 -> 1
- net /LattePanda Module/SUSCLK_WIFI: track 0.00 -> 43.2 mm, vias 0 -> 1
- net /LattePanda Module/REFCLK3-: track 0.00 -> 42.1 mm, vias 0 -> 3
- net /LattePanda Module/REFCLK3+: track 0.00 -> 42.1 mm, vias 0 -> 3
- net /LattePanda Module/HSIO_2_RX-: track 0.00 -> 37.5 mm, vias 0 -> 2
- net /LattePanda Module/HSIO_2_RX+: track 0.00 -> 37.5 mm, vias 0 -> 2
- net /LattePanda Module/USB_2_P7+: track 0.00 -> 36.5 mm, vias 0 -> 1
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
Commit message: Wired Battery_RAW input
Parts:
- removed JP79: SolderJumper_3_Open, Jumper:SolderJumper-3_P1.3mm_Bridged2Bar12_RoundedPad1.0x1.5mm_NumberLabels
- removed R171: 0R/1%, A_HDJ_Library:R_0402_1005Metric
- added D29: SS54, A_HDJ_Library:D_SMA, B.Cu at (189.6, 140.8)
- added D30: SS54, A_HDJ_Library:D_SMA, B.Cu at (189.6, 137.2)
- C137, D28, D47, R174, R177, R91, R93, U82: moved to B.Cu
- H8, J15: moved to F.Cu
- moved J1 194.4 mm to (246.0, 152.7), turned to 180 degrees
- moved J17 191.8 mm to (247.5, 111.0), turned to 90 degrees
- moved R52 130.2 mm to (202.0, 153.5), turned to 90 degrees
- moved Q81 125.5 mm to (211.2, 154.4), turned to 90 degrees
- moved R47 125.2 mm to (200.6, 153.5), turned to 90 degrees
- moved R49 125.2 mm to (204.6, 153.5), turned to 90 degrees
- moved U82 124.6 mm to (165.2, 132.5), turned to 180 degrees
- moved R46 118.5 mm to (200.9, 155.2)
- moved D22 116.3 mm to (206.8, 153.7), turned to 90 degrees
- moved J86 106.8 mm to (164.6, 138.8)
- moved J89 105.4 mm to (164.6, 145.6)
- moved J15 99.4 mm to (281.9, 137.4), turned to -90 degrees
- moved J87 98.3 mm to (173.1, 145.6)
- moved R89 95.0 mm to (215.0, 56.5), turned to 180 degrees
- moved C137 94.9 mm to (166.2, 135.0)
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Connections:
- net Net-(D28-A) renamed /PSU/B_RAW
- R46 pad 1: Net-(JP79-C) -> /LattePanda Module/SLS_S3
Routing:
- net /LattePanda Module/HSIO_2_RX-: track 37.5 -> 0.00 mm, vias 2 -> 0
- net /LattePanda Module/HSIO_2_RX+: track 37.5 -> 0.00 mm, vias 2 -> 0
- net GND: track 154.3 -> 121.2 mm, vias 98 -> 23
- net /M.2 E&M Key/CON_PCIE_TX_1-: track 32.4 -> 0.00 mm
- net /M.2 E&M Key/CON_PCIE_TX_1+: track 32.4 -> 0.00 mm
- net /LattePanda Module/SUSCLK_WIFI: track 43.2 -> 19.5 mm, vias 1 -> 2
- net +3V3: track 264.5 -> 241.1 mm, vias 44 -> 42
- net +5V: track 26.0 -> 3.68 mm, vias 3 -> 1
- net Net-(U96-VS/FIELD/ALSB): track 17.8 -> 0.00 mm
- net /~{PLT_RST}: track 46.6 -> 30.2 mm, vias 4 -> 1
- net /PSU/B_RAW: track 0.00 -> 15.7 mm
- net /PSU/BAT+: track 0.00 -> 7.30 mm, vias 0 -> 3
- net /~{WAKE}: track 35.7 -> 29.0 mm
- net /LattePanda Module/HSIO_3_TX-: track 43.7 -> 49.3 mm
- net /LattePanda Module/HSIO_3_TX+: track 43.7 -> 49.3 mm
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
Commit message: Rewired M.2 M key to fit new location. removed Fan_Temp as the design will move to a passive heatsink.
Parts:
- removed C84: 100nF/50V, A_HDJ_Library:C_0402_1005Metric
- removed D26: 1N5819WS, A_HDJ_Library:D_SOD-323
- removed M1: Fan_4pin, A_HDJ_Library:JST_PH_B4B-PH-K_1x04_P2.00mm_Vertical
- removed R64: 4.7K/1%, Resistor_SMD:R_0402_1005Metric
- removed R66: 21.5K/1%, Resistor_SMD:R_0402_1005Metric
- removed R68: 21.5K/1%, A_HDJ_Library:R_0402_1005Metric
- removed R69: 100R/1%, A_HDJ_Library:R_0402_1005Metric
- removed R72: 4.7K/1%, A_HDJ_Library:R_0402_1005Metric
- removed TP11, TP12: TestPoint, A_HDJ_Library:TestPoint_Pad_D1.5mm
- added R100: 10K/1%, A_HDJ_Library:R_0402_1005Metric, B.Cu at (148.8, 65.7)
- added R101: 10K/1%, A_HDJ_Library:R_0402_1005Metric, F.Cu at (161.7, 105.9)
- C51, C52, C53, C54, R27: moved to B.Cu
- C91, D9, R30: moved to F.Cu
- moved Q30 168.6 mm to (299.8, 71.8)
- moved Q31 168.6 mm to (299.8, 77.9)
- moved Q32 168.6 mm to (299.8, 84.1)
- moved U97 168.6 mm to (297.9, 89.2)
- moved U98 168.6 mm to (300.9, 89.2)
- moved C143 166.0 mm to (231.7, 49.9)
- moved D9 157.6 mm to (286.3, 146.2), turned to 180 degrees
- moved C52 156.3 mm to (269.9, 132.8), turned to -90 degrees
- moved D57 156.2 mm to (308.8, 69.7)
- moved R104 156.2 mm to (308.8, 73.7)
- moved R179 156.2 mm to (308.8, 75.7)
- moved R180 156.2 mm to (308.8, 77.7)
- moved R181 156.2 mm to (308.8, 79.7)
- moved R182 156.2 mm to (308.8, 81.6)
- moved R190 156.2 mm to (314.6, 69.7)
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Connections:
- J83 pad 31: +3V3 -> /HDMI-LVDS/RPi_LCD_EN
- J90 pad 31: +3V3 -> /HDMI-LVDS/RPi_LCD_EN
- U78 pad 31: unconnected-(U78-GPIO20-Pad31) -> /HDMI-LVDS/RPi_LCD_EN
- U86 pad 13: VDC -> /PSU/PWR_EN
Routing:
- net /~{WAKE}: track 29.0 -> 126.4 mm, vias 1 -> 3
- net /~{PLT_RST}: track 30.2 -> 126.4 mm, vias 1 -> 5
- net /LattePanda Module/REFCLK0-: track 0.00 -> 87.0 mm, vias 0 -> 1
- net /LattePanda Module/REFCLK0+: track 0.00 -> 87.0 mm, vias 0 -> 1
- net /LattePanda Module/HSIO_2_TX-: track 0.00 -> 82.3 mm
- net /LattePanda Module/HSIO_2_TX+: track 0.00 -> 82.3 mm
- net /LattePanda Module/SUSCLK_WIFI: track 19.5 -> 99.2 mm, vias 2 -> 3
- net /LattePanda Module/HSIO_2_RX-: track 0.00 -> 73.1 mm, vias 0 -> 1
- net /LattePanda Module/HSIO_2_RX+: track 0.00 -> 73.1 mm, vias 0 -> 1
- net +3V3: track 241.1 -> 286.0 mm, vias 42 -> 49
- net /HDMI-LVDS/RPi_LCD_EN: track 0.00 -> 24.4 mm, vias 0 -> 1
- net GND: track 121.2 -> 136.5 mm, vias 23 -> 77
- net Net-(D9-K): track 0.00 -> 12.4 mm
- net Net-(J15-SUSCLK): track 0.00 -> 6.78 mm
- net /PSU/PWR_EN: track 0.00 -> 4.31 mm, vias 0 -> 2
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Other:
- board text added: "VVV - USBC-PD needs to be flipped to the other side because of the heatsink"
