File: Motherboard/USB2.0&USB3.0.kicad_sch (KiCad schematic)
At the start: 21 parts, among them J4 USB3_A_Stacked, J81 USB_A, J82 USB3_A, J92 USB3_A, U3 ULC0524P, U5 ULC0524P, U9 ULC0524P

Commit message: Many, Many fixes and changes. Mostly Schematic-related.
Parts:
- removed unit 1 of J4
- J4: now not fitted; now left out of the parts list
Connections:
- net CON_USB3_SSTX_N: now also J82.8 (SSTX-)
- net CON_USB3_SSTX_P: now also J82.9 (SSTX+)
- net CON_USB4_SSTX_N: now also J92.8 (SSTX-); no longer J4.17 (SSTX2-)
- net CON_USB4_SSTX_P: now also J92.9 (SSTX+); no longer J4.18 (SSTX2+)
- net GND: now also J82.4 (GND), J82.7 (DRAIN), J82.SH (SHIELD), J92.4 (GND), J92.7 (DRAIN), J92.SH (SHIELD); no longer J4.13 (GND2), J4.16 (DRAIN2), J4.19 (SHIELD)
- net USB3_SSRX_N: now also J82.5 (SSRX-)
- net USB3_SSRX_P: now also J82.6 (SSRX+)
- net USB4_SSRX_N: now also J92.5 (SSRX-); no longer J4.14 (SSRX2-)
- net USB4_SSRX_P: now also J92.6 (SSRX+); no longer J4.15 (SSRX2+)
- net USB_2_P1+: now also J92.3 (D+); no longer J4.12 (D2+)
- net USB_2_P1-: now also J92.2 (D-); no longer J4.11 (D2-)
- net USB_2_P2+: now also J82.3 (D+)
- net USB_2_P2-: now also J82.2 (D-)
- net at J4.10 (VBUS2): no longer F6.2
- net at J82.1 (VBUS): now also F4.2
- net at J92.1 (VBUS): now also F6.2
- new net: J4.13 (GND2), J4.16 (DRAIN2), J4.19 (SHIELD)
Other:
- moved on the sheet: J82, J92
Changed lines of the file:
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@@
 	)
 	(junction
+		(at 361.95 207.01)
+		(diameter 0)
+		(color 0 0 0 0)
+	)
+	(junction
 		(at 339.09 236.22)
 		(diameter 0)
@@
 	)
 	(junction
-		(at 269.24 226.06)
+		(at 405.13 285.75)
 		(diameter 0)
 		(color 0 0 0 0)
 	)
 	(junction
-		(at 335.28 257.81)
+		(at 269.24 226.06)
 		(diameter 0)
 		(color 0 0 0 0)
 	)
 	(junction
-		(at 294.64 236.22)
+		(at 335.28 257.81)
 		(diameter 0)
 		(color 0 0 0 0)
 	)
 	(junction
-		(at 307.34 134.62)
+		(at 294.64 236.22)
 		(diameter 0)
 		(color 0 0 0 0)
 	)
 	(junction
-		(at 361.95 207.01)
+		(at 307.34 134.62)
 		(diameter 0)
 		(color 0 0 0 0)
@@
 	(wire
 		(pts
-			(xy 359.41 207.01) (xy 361.95 207.01)
+			(xy 407.67 285.75) (xy 405.13 285.75)
+		)
+		(stroke
+			(width 0)
+			(type default)
+		)
+	)
+	(wire
+		(pts
+			(xy 359.41 207.01) (xy 364.49 207.01)
 		)
 		(stroke
@@
 	(wire
 		(pts
-			(xy 361.95 207.01) (xy 364.49 207.01)
-		)
-		(stroke
-			(width 0)
-			(type default)
-		)
-	)
-	(wire
-		(pts
 			(xy 339.09 231.14) (xy 339.09 236.22)
 		)
@@
 	(wire
 		(pts
-			(xy 361.95 285.75) (xy 364.49 285.75)
+			(xy 405.13 285.75) (xy 402.59 285.75)
 		)
 		(stroke
@@
 	(wire
 		(pts
-			(xy 359.41 285.75) (xy 361.95 285.75)
+			(xy 359.41 285.75) (xy 364.49 285.75)
 		)
 		(stroke
@@
 	(symbol
 		(lib_id "Connector:USB3_A_Stacked")
-		(at 359.41 267.97 0)
+		(at 402.59 267.97 0)
 		(mirror y)
 		(unit 2)
 		(body_style 1)
 		(exclude_from_sim no)
-		(in_bom yes)
-		(on_board yes)
-		(in_pos_files yes)
-		(dnp no)
+		(in_bom no)
+		(on_board no)
+		(in_pos_files no)
+		(dnp yes)
 		(fields_autoplaced yes)
 		(property "Reference" "J4"
-			(at 370.84 267.335 0)
+			(at 414.02 267.335 0)
 			(show_name no)
 			(do_not_autoplace no)
@@
 		)
 		(property "Value" "USB3_A_Stacked"
-			(at 370.84 269.875 0)
+			(at 414.02 269.875 0)
 			(show_name no)
 			(do_not_autoplace no)
@@
 		)
 		(property "Footprint" "A_HDJ_Library:USB3_A_Molex_48406-0001_Horizontal_Stacked"
-			(at 355.6 265.43 0)
+			(at 398.78 265.43 0)
 			(hide yes)
 			(show_name no)
@@
 		)
 		(property "Datasheet" ""
-			(at 355.6 265.43 0)
+			(at 398.78 265.43 0)
 			(hide yes)
 			(show_name no)
@@
 		)
 		(property "Description" ""
-			(at 359.41 267.97 0)
+			(at 402.59 267.97 0)
 			(hide yes)
 			(show_name no)
@@
 		)
 		(property "SCH_Show_Footprint" ""
-			(at 359.41 267.97 0)
+			(at 402.59 267.97 0)
 			(hide yes)
 			(show_name no)
@@
 		)
 		(property "Sim.Device" ""
-			(at 359.41 267.97 0)
+			(at 402.59 267.97 0)
 			(hide yes)
 			(show_name no)
@@
 		)
 		(property "Sim.Pins" ""
-			(at 359.41 267.97 0)
+			(at 402.59 267.97 0)
 			(hide yes)
 			(show_name no)
@@
 		)
 		(property "Sim.Type" ""
-			(at 359.41 267.97 0)
+			(at 402.59 267.97 0)
 			(hide yes)
 			(show_name no)
@@
 		)
 		(property "Buy_Link" "https://item.szlcsc.com/3132965.html"
-			(at 685.8 538.48 0)
+			(at 728.98 538.48 0)
 			(hide yes)
 			(show_name no)
@@
 		)
 		(property "DF_Comment" "双层USB3.0 A母座_USB-303WSD-BRY"
-			(at 685.8 538.48 0)
+			(at 728.98 538.48 0)
 			(hide yes)
 			(show_name no)
@@
 		)
 		(property "LCSC Part" "C2895028"
-			(at 685.8 538.48 0)
+			(at 728.98 538.48 0)
 			(hide yes)
 			(show_name no)
@@
 	(symbol
 		(lib_id "Connector:USB3_A")
-		(at 402.59 189.23 0)
+		(at 359.41 189.23 0)
 		(mirror y)
 		(unit 1)
@@
 		(fields_autoplaced yes)
 		(property "Reference" "J82"
-			(at 414.02 188.5949 0)
+			(at 370.84 188.5949 0)
 			(show_name no)
 			(do_not_autoplace no)
@@
 		)
 		(property "Value" "USB3_A"
-			(at 414.02 191.1349 0)
+			(at 370.84 191.1349 0)
 			(show_name no)
 			(do_not_autoplace no)
@@
 		)
 		(property "Footprint" "Connector_USB:USB3_A_Molex_48393-001"
-			(at 398.78 186.69 0)
+			(at 355.6 186.69 0)
 			(hide yes)
 			(show_name no)
@@
 		)
 		(property "Datasheet" ""
-			(at 398.78 186.69 0)
+			(at 355.6 186.69 0)
 			(hide yes)
 			(show_name no)
@@
 		)
 		(property "Description" "USB 3.0 A connector"
-			(at 402.59 189.23 0)
+			(at 359.41 189.23 0)
 			(hide yes)
 			(show_name no)
@@
 	)
 	(symbol
-		(lib_id "Connector:USB3_A_Stacked")
-		(at 359.41 189.23 0)
-		(mirror y)
-		(unit 1)
-		(body_style 1)
-		(exclude_from_sim no)
-		(in_bom yes)
-		(on_board yes)
-		(in_pos_files yes)
-		(dnp no)
-		(fields_autoplaced yes)
-		(property "Reference" "J4"
-			(at 370.84 188.595 0)
-			(show_name no)
-			(do_not_autoplace no)
-			(effects
-				(font
-					(size 1.27 1.27)
-				)
-				(justify right)
-			)
-		)
-		(property "Value" "USB3_A_Stacked"
-			(at 370.84 191.135 0)
-			(show_name no)
-			(do_not_autoplace no)
-			(effects
-				(font
-					(size 1.27 1.27)
-				)
-				(justify right)
-			)
-		)
-		(property "Footprint" "A_HDJ_Library:USB3_A_Molex_48406-0001_Horizontal_Stacked"
-			(at 355.6 186.69 0)
-			(hide yes)
-			(show_name no)
-			(do_not_autoplace no)
-			(effects
-				(font
-					(size 1.27 1.27)
-				)
-			)
-		)
-		(property "Datasheet" ""
-			(at 355.6 186.69 0)
-			(hide yes)
-			(show_name no)
-			(do_not_autoplace no)
-			(effects
-				(font
-					(size 1.27 1.27)
-				)
-			)
-		)
-		(property "Description" ""
-			(at 359.41 189.23 0)
-			(hide yes)
-			(show_name no)
-			(do_not_autoplace no)
-			(effects
-				(font
-					(size 1.27 1.27)
-				)
-			)
-		)
-		(property "SCH_Show_Footprint" ""
-			(at 359.41 189.23 0)
-			(hide yes)
-			(show_name no)
-			(do_not_autoplace no)
-			(effects
-				(font
-					(size 1.27 1.27)
-				)
-			)
-		)
-		(property "Sim.Device" ""
-			(at 359.41 189.23 0)
-			(hide yes)
-			(show_name no)
-			(do_not_autoplace no)
-			(effects
-				(font
-					(size 1.27 1.27)
-				)
-			)
-		)
-		(property "Sim.Pins" ""
-			(at 359.41 189.23 0)
-			(hide yes)
-			(show_name no)
-			(do_not_autoplace no)
-			(effects
-				(font
-					(size 1.27 1.27)
-				)
-			)
-		)
-		(property "Sim.Type" ""
-			(at 359.41 189.23 0)
-			(hide yes)
-			(show_name no)
-			(do_not_autoplace no)
-			(effects
-				(font
-					(size 1.27 1.27)
-				)
-			)
-		)
-		(property "Buy_Link" "https://item.szlcsc.com/3132965.html"
-			(at 685.8 381 0)
-			(hide yes)
-			(show_name no)
-			(do_not_autoplace no)
-			(effects
-				(font
-					(size 1.27 1.27)
-				)
-			)
-		)
-		(property "DF_Comment" "双层USB3.0 A母座_USB-303WSD-BRY"
-			(at 685.8 381 0)
-			(hide yes)
-			(show_name no)
-			(do_not_autoplace no)
-			(effects
-				(font
-					(size 1.27 1.27)
-				)
-			)
-		)
-		(property "LCSC Part" "C2895028"
-			(at 685.8 459.74 0)
-			(hide yes)
-			(show_name no)
-			(do_not_autoplace no)
-			(effects
-				(font
-					(size 1.27 1.27)
-				)
-			)
-		)
-		(pin "3"
-		)
-		(pin "15"
-		)
-		(pin "2"
-		)
-		(pin "12"
-		)
-		(pin "13"
-		)
-		(pin "9"
-		)
-		(pin "17"
-		)
-		(pin "6"
-		)
-		(pin "14"
-		)
-		(pin "11"
-		)
-		(pin "10"
-		)
-		(pin "1"
-		)
-		(pin "5"
-		)
-		(pin "7"
-		)
-		(pin "8"
-		)
-		(pin "16"
-		)
-		(pin "4"
-		)
-		(pin "19"
-		)
-		(pin "18"
-		)
-		(instances
-			(project "Motherboard"
-				(path "/2a6d114a-7fd7-4207-b5f7-4ea9c34f36aa/f9aa04f2-8362-4e9f-9e54-e2b1a8ec9b0a"
-					(reference "J4")
-					(unit 1)
-				)
-			)
-		)
-	)
-	(symbol
 		(lib_id "Device:Fuse")
 		(at 342.9 257.81 90)
@@
 	(symbol
 		(lib_id "Connector:USB3_A")
-		(at 402.59 267.97 0)
+		(at 359.41 267.97 0)
 		(mirror y)
 		(unit 1)
@@
 		(fields_autoplaced yes)
 		(property "Reference" "J92"
-			(at 414.02 267.3349 0)
+			(at 370.84 267.3349 0)
 			(show_name no)
 			(do_not_autoplace no)
@@
 		)
 		(property "Value" "USB3_A"
-			(at 414.02 269.8749 0)
+			(at 370.84 269.8749 0)
 			(show_name no)
 			(do_not_autoplace no)
@@
 		)
 		(property "Footprint" "Connector_USB:USB3_A_Molex_48393-001"
-			(at 398.78 265.43 0)
+			(at 355.6 265.43 0)
 			(hide yes)
 			(show_name no)
@@
 		)
 		(property "Datasheet" ""
-			(at 398.78 265.43 0)
+			(at 355.6 265.43 0)
 			(hide yes)
 			(show_name no)
@@
 		)
 		(property "Description" "USB 3.0 A connector"
-			(at 402.59 267.97 0)
+			(at 359.41 267.97 0)
 			(hide yes)
 			(show_name no)

Commit message: Quick Save: Many things are being changed/updated/fixed.
Parts:
- added J93: USB_A, Connector_USB:USB_A_Molex_48037-2200_Horizontal, symbol Connector:USB_A
Changed lines of the file:
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@@
+	)
+	(symbol
+		(lib_id "Connector:USB_A")
+		(at 382.27 105.41 0)
+		(mirror y)
+		(unit 1)
+		(body_style 1)
+		(exclude_from_sim no)
+		(in_bom yes)
+		(on_board yes)
+		(in_pos_files yes)
+		(dnp no)
+		(fields_autoplaced yes)
+		(property "Reference" "J93"
+			(at 388.62 104.1399 0)
+			(show_name no)
+			(do_not_autoplace no)
+			(effects
+				(font
+					(size 1.27 1.27)
+				)
+				(justify right)
+			)
+		)
+		(property "Value" "USB_A"
+			(at 388.62 106.6799 0)
+			(show_name no)
+			(do_not_autoplace no)
+			(effects
+				(font
+					(size 1.27 1.27)
+				)
+				(justify right)
+			)
+		)
+		(property "Footprint" "Connector_USB:USB_A_Molex_48037-2200_Horizontal"
+			(at 378.46 106.68 0)
+			(hide yes)
+			(show_name no)
+			(do_not_autoplace no)
+			(effects
+				(font
+					(size 1.27 1.27)
+				)
+			)
+		)
+		(property "Datasheet" ""
+			(at 378.46 106.68 0)
+			(hide yes)
+			(show_name no)
+			(do_not_autoplace no)
+			(effects
+				(font
+					(size 1.27 1.27)
+				)
+			)
+		)
+		(property "Description" "USB Type A connector"
+			(at 382.27 105.41 0)
+			(hide yes)
+			(show_name no)
+			(do_not_autoplace no)
+			(effects
+				(font
+					(size 1.27 1.27)
+				)
+			)
+		)
+		(pin "4"
+		)
+		(pin "2"
+		)
+		(pin "3"
+		)
+		(pin "1"
+		)
+		(pin "SH"
+		)
+		(instances
+			(project "Motherboard"
+				(path "/2a6d114a-7fd7-4207-b5f7-4ea9c34f36aa/f9aa04f2-8362-4e9f-9e54-e2b1a8ec9b0a"
+					(reference "J93")
+					(unit 1)
+				)
+			)
+		)
 	)
 	(symbol

Commit message: Quick Save
Parts:
- removed J81: USB_A, symbol Connector:USB_A
Connections:
- net GND: now also J93.4 (GND), J93.SH (Shield)
- net USB_2_P3+: now also J93.3 (D+)
- net USB_2_P3-: now also J93.2 (D-)
- net at F3.2: now also J93.1 (VBUS)
Other:
- moved on the sheet: J93
Changed lines of the file:
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@@
 	)
 	(junction
-		(at 361.95 115.57)
-		(diameter 0)
-		(color 0 0 0 0)
-	)
-	(junction
 		(at 405.13 285.75)
 		(diameter 0)
@@
 	)
 	(junction
+		(at 361.95 115.57)
+		(diameter 0)
+		(color 0 0 0 0)
+	)
+	(junction
 		(at 294.64 226.06)
 		(diameter 0)
@@
 	)
 	(symbol
-		(lib_id "Connector:USB_A")
-		(at 359.41 105.41 0)
-		(mirror y)
-		(unit 1)
-		(body_style 1)
-		(exclude_from_sim no)
-		(in_bom yes)
-		(on_board yes)
-		(in_pos_files yes)
-		(dnp no)
-		(fields_autoplaced yes)
-		(property "Reference" "J81"
-			(at 365.76 104.1399 0)
-			(show_name no)
-			(do_not_autoplace no)
-			(effects
-				(font
-					(size 1.27 1.27)
-				)
-				(justify right)
-			)
-		)
-		(property "Value" "USB_A"
-			(at 365.76 106.6799 0)
-			(show_name no)
-			(do_not_autoplace no)
-			(effects
-				(font
-					(size 1.27 1.27)
-				)
-				(justify right)
-			)
-		)
-		(property "Footprint" ""
-			(at 355.6 106.68 0)
-			(hide yes)
-			(show_name no)
-			(do_not_autoplace no)
-			(effects
-				(font
-					(size 1.27 1.27)
-				)
-			)
-		)
-		(property "Datasheet" ""
-			(at 355.6 106.68 0)
-			(hide yes)
-			(show_name no)
-			(do_not_autoplace no)
-			(effects
-				(font
-					(size 1.27 1.27)
-				)
-			)
-		)
-		(property "Description" "USB Type A connector"
-			(at 359.41 105.41 0)
-			(hide yes)
-			(show_name no)
-			(do_not_autoplace no)
-			(effects
-				(font
-					(size 1.27 1.27)
-				)
-			)
-		)
-		(pin "2"
-		)
-		(pin "SH"
-		)
-		(pin "1"
-		)
-		(pin "3"
-		)
-		(pin "4"
-		)
-		(instances
-			(project "Motherboard"
-				(path "/2a6d114a-7fd7-4207-b5f7-4ea9c34f36aa/f9aa04f2-8362-4e9f-9e54-e2b1a8ec9b0a"
-					(reference "J81")
-					(unit 1)
-				)
-			)
-		)
-	)
-	(symbol
 		(lib_id "Power_Protection:D3V3XA4B10LP")
 		(at 320.04 127 0)
@@
 	(symbol
 		(lib_id "Connector:USB_A")
-		(at 382.27 105.41 0)
+		(at 359.41 105.41 0)
 		(mirror y)
 		(unit 1)
@@
 		(fields_autoplaced yes)
 		(property "Reference" "J93"
-			(at 388.62 104.1399 0)
+			(at 365.76 104.1399 0)
 			(show_name no)
 			(do_not_autoplace no)
@@
 		)
 		(property "Value" "USB_A"
-			(at 388.62 106.6799 0)
+			(at 365.76 106.6799 0)
 			(show_name no)
 			(do_not_autoplace no)
@@
 		)
 		(property "Footprint" "Connector_USB:USB_A_Molex_48037-2200_Horizontal"
-			(at 378.46 106.68 0)
+			(at 355.6 106.68 0)
 			(hide yes)
 			(show_name no)
@@
 		)
 		(property "Datasheet" ""
-			(at 378.46 106.68 0)
+			(at 355.6 106.68 0)
 			(hide yes)
 			(show_name no)
@@
 		)
 		(property "Description" "USB Type A connector"
-			(at 382.27 105.41 0)
+			(at 359.41 105.41 0)
 			(hide yes)
 			(show_name no)

Commit message: Completed routing of 9V and 3.3V of PSU
Parts:
- C62, F3, J93: now not fitted; now left out of the parts list
Changed lines of the file:
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@@
 		(unit 1)
 		(body_style 1)
-		(exclude_from_sim no)
-		(in_bom yes)
-		(on_board yes)
-		(in_pos_files yes)
-		(dnp no)
+		(exclude_from_sim yes)
+		(in_bom no)
+		(on_board no)
+		(in_pos_files no)
+		(dnp yes)
 		(fields_autoplaced yes)
 		(property "Reference" "#PWR0173"
@@
 		(unit 1)
 		(body_style 1)
-		(exclude_from_sim no)
-		(in_bom yes)
-		(on_board yes)
-		(in_pos_files yes)
-		(dnp no)
+		(exclude_from_sim yes)
+		(in_bom no)
+		(on_board no)
+		(in_pos_files no)
+		(dnp yes)
 		(property "Reference" "C62"
 			(at 320.04 91.44 90)
@@
 		(unit 1)
 		(body_style 1)
-		(exclude_from_sim no)
-		(in_bom yes)
-		(on_board yes)
-		(in_pos_files yes)
-		(dnp no)
+		(exclude_from_sim yes)
+		(in_bom no)
+		(on_board no)
+		(in_pos_files no)
+		(dnp yes)
 		(fields_autoplaced yes)
 		(property "Reference" "#PWR0169"
@@
 		(unit 1)
 		(body_style 1)
-		(exclude_from_sim no)
-		(in_bom yes)
-		(on_board yes)
-		(in_pos_files yes)
-		(dnp no)
+		(exclude_from_sim yes)
+		(in_bom no)
+		(on_board no)
+		(in_pos_files no)
+		(dnp yes)
 		(fields_autoplaced yes)
 		(property "Reference" "#PWR0166"
@@
 		(unit 1)
 		(body_style 1)
-		(exclude_from_sim no)
-		(in_bom yes)
-		(on_board yes)
-		(in_pos_files yes)
-		(dnp no)
+		(exclude_from_sim yes)
+		(in_bom no)
+		(on_board no)
+		(in_pos_files no)
+		(dnp yes)
 		(property "Reference" "F3"
 			(at 336.55 102.87 90)
@@
 		(unit 1)
 		(body_style 1)
-		(exclude_from_sim no)
-		(in_bom yes)
-		(on_board yes)
-		(in_pos_files yes)
-		(dnp no)
+		(exclude_from_sim yes)
+		(in_bom no)
+		(on_board no)
+		(in_pos_files no)
+		(dnp yes)
 		(fields_autoplaced yes)
 		(property "Reference" "J93"
