File: Motherboard/LattePanda Module.kicad_sch (KiCad schematic)
At the start: 92 parts, among them IC78 PCM2704CDBR, IC79 TS3DV621RUAR, J3 Conn_01x03_Pin, J5 SM03B-SRSS-TB, J78 Speaker_L, J79 Speaker_R, SW78 SW_Push, SW79 SW_Push, SW80 SW_Push, SW81 SW_Push, SW82 SW_Nidec_CAS-120A1, U10 ULC0524P, U11 ULC0524P, U12 ULC0524P, U78 RP2040, U84 PAM8403D, U88 RP2354B, U95 W25Q128JVS, Y1 ABM8-272-T3, Y2 ABM8-272-T3, Y78 Crystal

Commit message: Swapped Volume and Brightness sliders for easier wiring.
Parts:
- C3, C4: value 15p -> 15pF
- L5: footprint A_HDJ_Library:L_Sunlord_SWPA4020S -> Inductor_SMD:L_0603_1608Metric
Connections:
- net DDIB_TOUCH_SCL: now also U12.5, U12.6 (NC)
- net DDIB_TOUCH_SDA: now also U12.4, U12.7 (NC)
- net I2C2_SCL: no longer U12.2, U12.9 (NC)
- net I2C2_SDA: no longer U12.1, U12.10 (NC)
- net I2C3_SCL: no longer U12.5, U12.6 (NC)
- net I2C3_SDA: no longer U12.4, U12.7 (NC)
- net TCP0_TOUCH_SCL: now also U12.2, U12.9 (NC)
- net TCP0_TOUCH_SDA: now also U12.1, U12.10 (NC)
- net SL_BRI: no longer names the net of U88.56 (GPIO45/ADC5)
Changed lines of the file:
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@@
 		)
 	)
-	(label "I2C3_SCL"
-		(at 478.79 344.17 180)
-		(effects
-			(font
-				(size 1.27 1.27)
-			)
-			(justify right bottom)
-		)
-	)
 	(label "I2C4_SDA"
 		(at 406.4 300.99 0)
@@
 		)
 	)
-	(label "I2C2_SCL"
-		(at 414.02 344.17 0)
-		(effects
-			(font
-				(size 1.27 1.27)
-			)
-			(justify left bottom)
-		)
-	)
 	(label "DDI_TX3-"
 		(at 270.51 226.06 180)
@@
 		)
 	)
-	(label "I2C3_SDA"
-		(at 478.79 334.01 180)
-		(effects
-			(font
-				(size 1.27 1.27)
-			)
-			(justify right bottom)
-		)
-	)
 	(label "I2C2_SDA"
 		(at 360.68 300.99 0)
@@
 		)
 	)
-	(label "I2C2_SDA"
-		(at 414.02 334.01 0)
-		(effects
-			(font
-				(size 1.27 1.27)
-			)
-			(justify left bottom)
-		)
-	)
 	(label "DDI_TX1+"
 		(at 177.8 271.78 0)
@@
 		)
 	)
+	(hierarchical_label "DDIB_TOUCH_SDA"
+		(shape bidirectional)
+		(at 478.79 334.01 0)
+		(effects
+			(font
+				(size 1.27 1.27)
+			)
+			(justify left)
+		)
+	)
 	(hierarchical_label "RPI_BAT_SDA"
 		(shape bidirectional)
@@
 		)
 	)
-	(hierarchical_label "SL_BRI"
-		(shape output)
-		(at 459.74 219.71 180)
-		(effects
-			(font
-				(size 1.27 1.27)
-			)
-			(justify right)
-		)
-	)
 	(hierarchical_label "LED_WiFi_R"
 		(shape output)
@@
 		)
 	)
+	(hierarchical_label "DDIB_TOUCH_SCL"
+		(shape input)
+		(at 478.79 344.17 0)
+		(effects
+			(font
+				(size 1.27 1.27)
+			)
+			(justify left)
+		)
+	)
 	(hierarchical_label "Row3"
 		(shape input)
@@
 		)
 	)
+	(hierarchical_label "TCP0_TOUCH_SCL"
+		(shape input)
+		(at 414.02 344.17 180)
+		(effects
+			(font
+				(size 1.27 1.27)
+			)
+			(justify right)
+		)
+	)
 	(hierarchical_label "TCP0_TX3-"
 		(shape output)
@@
 		)
 	)
+	(hierarchical_label "TCP0_TOUCH_SDA"
+		(shape bidirectional)
+		(at 414.02 334.01 180)
+		(effects
+			(font
+				(size 1.27 1.27)
+			)
+			(justify right)
+		)
+	)
 	(hierarchical_label "HSIO_1_TX-"
 		(shape output)
@@
 			)
 		)
-		(property "Value" "15p"
+		(property "Value" "15pF"
 			(at 452.501 176.403 0)
 			(show_name no)
@@
 			)
 		)
-		(property "Value" "15p"
+		(property "Value" "15pF"
 			(at 446.659 191.897 0)
 			(show_name no)
@@
 			)
 		)
-		(property "Footprint" "A_HDJ_Library:L_Sunlord_SWPA4020S"
+		(property "Footprint" "Inductor_SMD:L_0603_1608Metric"
 			(at 518.16 113.03 0)
 			(hide yes)
