File: Motherboard/M.2 E&M Key.kicad_sch (KiCad schematic)
At the start: 25 parts, among them J15 Bus_M.2_Socket_M, J16 Bus_M.2_Socket_E

Commit message: Motherboard Complete (aside from parts-BOM associations)
Connections:
- net RPi_WiFi_M2E: now reaches J16.6 (~{LED_1})
- no-connect marks 51 -> 50
Changed lines of the file:
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@@
 	(text "To be grounded for SATA, No Connect for PCIe"
 		(exclude_from_sim no)
-		(at 252.73 194.31 0)
+		(at 251.46 189.23 0)
 		(effects
 			(font
@@
 	)
 	(no_connect
-		(at 454.66 190.5)
-	)
-	(no_connect
 		(at 200.66 156.21)
 	)
@@
 		)
 	)
+	(hierarchical_label "RPi_WiFi_M2E"
+		(shape output)
+		(at 454.66 190.5 0)
+		(effects
+			(font
+				(size 1.27 1.27)
+			)
+			(justify left)
+		)
+	)

Commit message: Created updated BOM for PCBWay on all CTRL daughterboards. These boards have likely hit their final* version
*Ive said "Finished Version" many times in this project. I'm confident now, but no guarantees.
Parts:
- C49, C50, C55, C56: DF_Comment 贴片电容0402-10UF-10V-X5R_GRM155R61A106ME44D -> (none); MPN (none) -> any/open; Manufacturer (none) -> any/open; Specifications (For Resistors/Capacitors) (none) -> 220nF 0402 Ceramic 20% 50V X5R
- C51, C53, C57, C59: DF_Comment 贴片电容0402-10UF-10V-X5R_GRM155R61A106ME44D -> (none); MPN (none) -> any/open; Manufacturer (none) -> any/open; Specifications (For Resistors/Capacitors) (none) -> 10uF 0402 Ceramic 20% 10V X5R
- C52, C54, C58, C60: DF_Comment 贴片电容0402-10UF-10V-X5R_GRM155R61A106ME44D -> (none); MPN (none) -> any/open; Manufacturer (none) -> any/open; Specifications (For Resistors/Capacitors) (none) -> 100nF 0402 Ceramic 20% 50V X5R
- D9: MPN (none) -> XL-1608UGC-04
- H7, H8: MPN (none) -> SMTWEM225STR
- J15: MPN (none) -> APCI0107-P001A; Manufacturer (none) -> Lian Xin Technology
- J16: MPN (none) -> APCI0108-P001A; Manufacturer (none) -> Lian Xin Technology
- R27, R29, R30, R32, R33, R34, R35: DF_Comment 贴片电阻0402-10K-1% -> (none)

Commit message: Motherboard Complete.
Parts:
- D9: Specifications (For Resistors/Capacitors) (none) -> N/A
- H7, H8: LCSC Part C5301801 -> (none); Specifications (For Resistors/Capacitors) (none) -> N/A
- J15: LCSC Part C7498140 -> (none); Specifications (For Resistors/Capacitors) (none) -> N/A
- J16: LCSC Part C7498141 -> (none); Specifications (For Resistors/Capacitors) (none) -> N/A
- R27, R29, R32, R33: MPN (none) -> any/open; Specifications (For Resistors/Capacitors) (none) -> 0R 1% 0402
- R30: MPN (none) -> any/open; Specifications (For Resistors/Capacitors) (none) -> 2.2k 1% 63mW 0402
- R34, R35: MPN (none) -> any/open; Specifications (For Resistors/Capacitors) (none) -> 10k 1% 63mW 0402
- TP2: MPN (none) -> N/A; Specifications (For Resistors/Capacitors) (none) -> N/A

Commit message: Majorly reworked Display system, condensed and fixed BOM, and many other schematic and design cleanups. \Programs folder was also cleaned up.
Everything is still a work in progress, many things are now unfinished, especially the PCB.
Parts:
- C49, C50, C55, C56: value 220nF/50V -> 220nF; footprint A_HDJ_Library:C_0402_1005Metric -> Capacitor_SMD:C_0402_1005Metric; MPN any/open -> GRM155R61H224ME01D
- C51, C53, C57, C59: value 10uF/10V -> 10uF; footprint A_HDJ_Library:C_0402_1005Metric -> Capacitor_SMD:C_0402_1005Metric; Field-1 (none) -> G; MPN any/open -> GMC04X5R106M10NT
- C52, C54, C58, C60: value 100nF/50V -> 100nF; footprint A_HDJ_Library:C_0402_1005Metric -> Capacitor_SMD:C_0402_1005Metric; Field-1 (none) -> N; MPN any/open -> TCC0402X5R104M500AT
- R27, R29, R32, R33: footprint A_HDJ_Library:R_0402_1005Metric -> Resistor_SMD:R_0402_1005Metric; MPN any/open -> CQ02WGF0000TCE
- R30: value 2.2K/1% -> 2.2k/1%; footprint A_HDJ_Library:R_0402_1005Metric -> Resistor_SMD:R_0402_1005Metric; MPN any/open -> NQ02WGF2201TCE
- R34, R35: value 10K/1% -> 10k/1%; footprint A_HDJ_Library:R_0402_1005Metric -> Resistor_SMD:R_0402_1005Metric; MPN any/open -> MCR01MZPF1002
Changed lines of the file:
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@@
 			)
 		)
-		(property "Footprint" "A_HDJ_Library:R_0402_1005Metric"
+		(property "Footprint" "Resistor_SMD:R_0402_1005Metric"
 			(at 189.738 116.84 90)
 			(hide yes)
@@
 			)
 		)
-		(property "MPN" "any/open"
+		(property "MPN" "CQ02WGF0000TCE"
 			(at 187.96 116.84 0)
 			(hide yes)
@@
 			)
 		)
-		(property "Value" "10K/1%"
+		(property "Value" "10k/1%"
 			(at 476.25 144.78 0)
 			(show_name no)
@@
 			)
 		)
-		(property "Footprint" "A_HDJ_Library:R_0402_1005Metric"
+		(property "Footprint" "Resistor_SMD:R_0402_1005Metric"
 			(at 473.202 146.05 90)
 			(hide yes)
@@
 			)
 		)
-		(property "MPN" "any/open"
+		(property "MPN" "MCR01MZPF1002"
 			(at 474.98 146.05 0)
 			(hide yes)
@@
 			)
 		)
-		(property "Value" "10uF/10V"
+		(property "Value" "10uF"
 			(at 441.96 95.25 90)
 			(show_name no)
@@
 			)
 		)
-		(property "Footprint" "A_HDJ_Library:C_0402_1005Metric"
+		(property "Footprint" "Capacitor_SMD:C_0402_1005Metric"
 			(at 431.8 97.4852 0)
 			(hide yes)
@@
 			)
 		)
-		(property "Field-1" ""
+		(property "Field-1" "G"
 			(at 339.09 -339.09 0)
 			(hide yes)
@@
 			)
 		)
-		(property "MPN" "any/open"
+		(property "MPN" "GMC04X5R106M10NT"
 			(at 435.61 96.52 90)
 			(hide yes)
@@
 			)
 		)
-		(property "Value" "2.2K/1%"
+		(property "Value" "2.2k/1%"
 			(at 273.05 168.91 0)
 			(show_name no)
@@
 			)
 		)
-		(property "Footprint" "A_HDJ_Library:R_0402_1005Metric"
+		(property "Footprint" "Resistor_SMD:R_0402_1005Metric"
 			(at 265.938 167.64 90)
 			(hide yes)
@@
 			)
 		)
-		(property "MPN" "any/open"
+		(property "MPN" "NQ02WGF2201TCE"
 			(at 264.16 167.64 0)
 			(hide yes)
@@
 			)
 		)
-		(property "Value" "100nF/50V"
+		(property "Value" "100nF"
 			(at 441.96 114.3 90)
 			(show_name no)
@@
 			)
 		)
-		(property "Footprint" "A_HDJ_Library:C_0402_1005Metric"
+		(property "Footprint" "Capacitor_SMD:C_0402_1005Metric"
 			(at 431.8 116.5352 0)
 			(hide yes)
@@
 			)
 		)
-		(property "Field-1" ""
+		(property "Field-1" "N"
 			(at 320.04 -320.04 0)
 			(hide yes)
@@
 			)
 		)
-		(property "MPN" "any/open"
+		(property "MPN" "TCC0402X5R104M500AT"
 			(at 435.61 115.57 90)
 			(hide yes)
@@
 			)
 		)
-		(property "Value" "220nF/50V"
+		(property "Value" "220nF"
 			(at 167.64 137.16 90)
 			(show_name no)
@@
 			)
 		)
-		(property "Footprint" "A_HDJ_Library:C_0402_1005Metric"
+		(property "Footprint" "Capacitor_SMD:C_0402_1005Metric"
 			(at 166.37 138.43 0)
 			(hide yes)
@@
 			)
 		)
-		(property "MPN" "any/open"
+		(property "MPN" "GRM155R61H224ME01D"
 			(at 166.37 138.43 90)
 			(hide yes)
@@
 			)
 		)
-		(property "Value" "10uF/10V"
+		(property "Value" "10uF"
 			(at 238.76 106.68 90)
 			(show_name no)
@@
 			)
 		)
-		(property "Footprint" "A_HDJ_Library:C_0402_1005Metric"
+		(property "Footprint" "Capacitor_SMD:C_0402_1005Metric"
 			(at 228.6 108.9152 0)
 			(hide yes)
@@
 			)
 		)
-		(property "Field-1" ""
+		(property "Field-1" "G"
 			(at 124.46 -124.46 0)
 			(hide yes)
@@
 			)
 		)
-		(property "MPN" "any/open"
+		(property "MPN" "GMC04X5R106M10NT"
 			(at 232.41 107.95 90)
 			(hide yes)
@@
 			)
 		)
-		(property "Value" "100nF/50V"
+		(property "Value" "100nF"
 			(at 238.76 100.33 90)
 			(show_name no)
@@
 			)
 		)
-		(property "Footprint" "A_HDJ_Library:C_0402_1005Metric"
+		(property "Footprint" "Capacitor_SMD:C_0402_1005Metric"
 			(at 228.6 102.5652 0)
 			(hide yes)
@@
 			)
 		)
-		(property "Field-1" ""
+		(property "Field-1" "N"
 			(at 130.81 -130.81 0)
 			(hide yes)
@@
 			)
 		)
-		(property "MPN" "any/open"
+		(property "MPN" "TCC0402X5R104M500AT"
 			(at 232.41 101.6 90)
 			(hide yes)
@@
 			)
 		)
-		(property "Footprint" "A_HDJ_Library:R_0402_1005Metric"
+		(property "Footprint" "Resistor_SMD:R_0402_1005Metric"
 			(at 469.9 199.898 90)
 			(hide yes)
@@
 			)
 		)
-		(property "MPN" "any/open"
+		(property "MPN" "CQ02WGF0000TCE"
 			(at 469.9 198.12 90)
 			(hide yes)
@@
 			)
 		)
-		(property "Value" "220nF/50V"
+		(property "Value" "220nF"
 			(at 167.64 134.62 90)
 			(show_name no)
@@
 			)
 		)
-		(property "Footprint" "A_HDJ_Library:C_0402_1005Metric"
+		(property "Footprint" "Capacitor_SMD:C_0402_1005Metric"
 			(at 166.37 135.89 0)
 			(hide yes)
@@
 			)
 		)
-		(property "MPN" "any/open"
+		(property "MPN" "GRM155R61H224ME01D"
 			(at 166.37 135.89 90)
 			(hide yes)
@@
 			)
 		)
-		(property "Value" "10uF/10V"
+		(property "Value" "10uF"
 			(at 441.96 107.95 90)
 			(show_name no)
@@
 			)
 		)
-		(property "Footprint" "A_HDJ_Library:C_0402_1005Metric"
+		(property "Footprint" "Capacitor_SMD:C_0402_1005Metric"
 			(at 431.8 110.1852 0)
 			(hide yes)
@@
 			)
 		)
-		(property "Field-1" ""
+		(property "Field-1" "G"
 			(at 326.39 -326.39 0)
 			(hide yes)
@@
 			)
 		)
-		(property "MPN" "any/open"
+		(property "MPN" "GMC04X5R106M10NT"
 			(at 435.61 109.22 90)
 			(hide yes)
@@
 			)
 		)
-		(property "Value" "220nF/50V"
+		(property "Value" "220nF"
 			(at 370.84 138.43 90)
 			(show_name no)
@@
 			)
 		)
-		(property "Footprint" "A_HDJ_Library:C_0402_1005Metric"
+		(property "Footprint" "Capacitor_SMD:C_0402_1005Metric"
 			(at 369.57 139.7 0)
 			(hide yes)
@@
 			)
 		)
-		(property "MPN" "any/open"
+		(property "MPN" "GRM155R61H224ME01D"
 			(at 369.57 139.7 90)
 			(hide yes)
@@
 			)
 		)
-		(property "Value" "100nF/50V"
+		(property "Value" "100nF"
 			(at 238.76 113.03 90)
 			(show_name no)
@@
 			)
 		)
-		(property "Footprint" "A_HDJ_Library:C_0402_1005Metric"
+		(property "Footprint" "Capacitor_SMD:C_0402_1005Metric"
 			(at 228.6 115.2652 0)
 			(hide yes)
@@
 			)
 		)
-		(property "Field-1" ""
+		(property "Field-1" "N"
 			(at 118.11 -118.11 0)
 			(hide yes)
@@
 			)
 		)
-		(property "MPN" "any/open"
+		(property "MPN" "TCC0402X5R104M500AT"
 			(at 232.41 114.3 90)
 			(hide yes)
@@
 			)
 		)
-		(property "Footprint" "A_HDJ_Library:R_0402_1005Metric"
+		(property "Footprint" "Resistor_SMD:R_0402_1005Metric"
 			(at 395.478 114.3 90)
 			(hide yes)
@@
 			)
 		)
-		(property "MPN" "any/open"
+		(property "MPN" "CQ02WGF0000TCE"
 			(at 393.7 114.3 0)
 			(hide yes)
@@
 			)
 		)
-		(property "Value" "220nF/50V"
+		(property "Value" "220nF"
 			(at 370.84 135.89 90)
 			(show_name no)
@@
 			)
 		)
-		(property "Footprint" "A_HDJ_Library:C_0402_1005Metric"
+		(property "Footprint" "Capacitor_SMD:C_0402_1005Metric"
 			(at 369.57 137.16 0)
 			(hide yes)
@@
 			)
 		)
-		(property "MPN" "any/open"
+		(property "MPN" "GRM155R61H224ME01D"
 			(at 369.57 137.16 90)
 			(hide yes)
@@
 			)
 		)
-		(property "Value" "10uF/10V"
+		(property "Value" "10uF"
 			(at 238.76 93.98 90)
 			(show_name no)
@@
 			)
 		)
-		(property "Footprint" "A_HDJ_Library:C_0402_1005Metric"
+		(property "Footprint" "Capacitor_SMD:C_0402_1005Metric"
 			(at 228.6 96.2152 0)
 			(hide yes)
@@
 			)
 		)
-		(property "Field-1" ""
+		(property "Field-1" "G"
 			(at 137.16 -137.16 0)
 			(hide yes)
@@
 			)
 		)
-		(property "MPN" "any/open"
+		(property "MPN" "GMC04X5R106M10NT"
 			(at 232.41 95.25 90)
 			(hide yes)
@@
 			)
 		)
-		(property "Footprint" "A_HDJ_Library:R_0402_1005Metric"
+		(property "Footprint" "Resistor_SMD:R_0402_1005Metric"
 			(at 261.62 198.628 90)
 			(hide yes)
@@
 			)
 		)
-		(property "MPN" "any/open"
+		(property "MPN" "CQ02WGF0000TCE"
 			(at 261.62 196.85 90)
 			(hide yes)
@@
 			)
 		)
-		(property "Value" "10K/1%"
+		(property "Value" "10k/1%"
 			(at 469.9 147.32 0)
 			(show_name no)
@@
 			)
 		)
-		(property "Footprint" "A_HDJ_Library:R_0402_1005Metric"
+		(property "Footprint" "Resistor_SMD:R_0402_1005Metric"
 			(at 472.948 146.05 90)
 			(hide yes)
@@
 			)
 		)
-		(property "MPN" "any/open"
+		(property "MPN" "MCR01MZPF1002"
 			(at 471.17 146.05 0)
 			(hide yes)
@@
 			)
 		)
-		(property "Value" "100nF/50V"
+		(property "Value" "100nF"
 			(at 441.96 101.6 90)
 			(show_name no)
@@
 			)
 		)
-		(property "Footprint" "A_HDJ_Library:C_0402_1005Metric"
+		(property "Footprint" "Capacitor_SMD:C_0402_1005Metric"
 			(at 431.8 103.8352 0)
 			(hide yes)
@@
 			)
 		)
-		(property "Field-1" ""
+		(property "Field-1" "N"
 			(at 332.74 -332.74 0)
 			(hide yes)
@@
 			)
 		)
-		(property "MPN" "any/open"
+		(property "MPN" "TCC0402X5R104M500AT"
 			(at 435.61 102.87 90)
 			(hide yes)

Commit message: General Readme update
Parts:
- J15: value Bus_M.2_Socket_M -> M.2 Socket M; footprint A_HDJ_Library:PCIe_M.2_Connectors_P=0.5mm_H=4.2mm_KeyM -> MDT420M03001:MDT420M03001
- J16: value Bus_M.2_Socket_E -> M.2 Socket E; footprint A_HDJ_Library:PCIe_M.2_Connectors_P=0.5mm_H=4.2mm_KeyE -> MDT420E03001:MDT420E03001
Changed lines of the file:
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@@
 			)
 		)
-		(property "Value" "Bus_M.2_Socket_E"
+		(property "Value" "M.2 Socket E"
 			(at 431.4541 121.92 0)
 			(show_name no)
@@
 			)
 		)
-		(property "Footprint" "A_HDJ_Library:PCIe_M.2_Connectors_P=0.5mm_H=4.2mm_KeyE"
+		(property "Footprint" "MDT420E03001:MDT420E03001"
 			(at 429.26 143.51 0)
 			(hide yes)
@@
 			)
 		)
-		(property "Value" "Bus_M.2_Socket_M"
+		(property "Value" "M.2 Socket M"
 			(at 228.2541 120.65 0)
 			(show_name no)
@@
 			)
 		)
-		(property "Footprint" "A_HDJ_Library:PCIe_M.2_Connectors_P=0.5mm_H=4.2mm_KeyM"
+		(property "Footprint" "MDT420M03001:MDT420M03001"
 			(at 226.06 142.24 0)
 			(hide yes)

Commit message: Repository push for Project Deadline :o
Parts:
- C49, C50, C55, C56: SCH_Show_Footprint C0402 -> (none)
- C51, C53, C57, C59: Field-1 G -> (none); SCH_Show_Footprint C0402 -> (none)
- C52, C54, C58, C60: Field-1 N -> (none); SCH_Show_Footprint C0402 -> (none)
- D9: SCH_Show_Footprint LED0603 -> (none)
- H7, H8: DF_Comment 贴片螺母柱M2XC4X2.5+C2.7X1.5 -> (none)
- J15: Buy_Link https://item.szlcsc.com/8568582.html -> (none); DF_Comment M.2连接器KEY-M_H4.2mm-67P_APCI0107-P001A -> (none)
- J16: Buy_Link https://item.szlcsc.com/8568583.html -> (none); DF_Comment M.2连接器KEY-E_H4.2mm-67P_APCI0108-P001A -> (none)
- TP2: MPN N/A -> (none)
