File: Motherboard/fan_temp.kicad_sch (KiCad schematic)
At the start: 23 parts, among them M1 Fan_4pin, M2 Fan_4pin

Commit message: Rewired M.2 M key to fit new location. removed Fan_Temp as the design will move to a passive heatsink.
Parts:
- C84, D26, M1, R68, R69, R72: now not fitted; now left out of the parts list
- TP11, TP12: now not fitted
Changed lines of the file:
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@@
 		(body_style 1)
 		(exclude_from_sim no)
-		(in_bom yes)
-		(on_board yes)
+		(in_bom no)
+		(on_board no)
 		(in_pos_files yes)
-		(dnp no)
+		(dnp yes)
 		(property "Reference" "R69"
 			(at 327.66 166.37 90)
@@
 		(exclude_from_sim no)
 		(in_bom no)
-		(on_board yes)
+		(on_board no)
 		(in_pos_files yes)
 		(dnp yes)
@@
 		(body_style 1)
 		(exclude_from_sim no)
-		(in_bom yes)
-		(on_board yes)
+		(in_bom no)
+		(on_board no)
 		(in_pos_files yes)
-		(dnp no)
+		(dnp yes)
 		(property "Reference" "C84"
 			(at 344.17 148.59 0)
@@
 		(body_style 1)
 		(exclude_from_sim no)
-		(in_bom yes)
-		(on_board yes)
+		(in_bom no)
+		(on_board no)
 		(in_pos_files yes)
-		(dnp no)
+		(dnp yes)
 		(fields_autoplaced yes)
 		(property "Reference" "#PWR0113"
@@
 		(exclude_from_sim no)
 		(in_bom no)
-		(on_board yes)
+		(on_board no)
 		(in_pos_files yes)
-		(dnp no)
+		(dnp yes)
 		(property "Reference" "TP12"
 			(at 295.148 169.672 0)
@@
 		(body_style 1)
 		(exclude_from_sim no)
-		(in_bom yes)
-		(on_board yes)
+		(in_bom no)
+		(on_board no)
 		(in_pos_files yes)
-		(dnp no)
+		(dnp yes)
 		(fields_autoplaced yes)
 		(property "Reference" "#PWR0117"
@@
 		(body_style 1)
 		(exclude_from_sim no)
-		(in_bom yes)
-		(on_board yes)
+		(in_bom no)
+		(on_board no)
 		(in_pos_files yes)
-		(dnp no)
+		(dnp yes)
 		(fields_autoplaced yes)
 		(property "Reference" "#PWR0114"
@@
 		(body_style 1)
 		(exclude_from_sim no)
-		(in_bom yes)
-		(on_board yes)
+		(in_bom no)
+		(on_board no)
 		(in_pos_files yes)
-		(dnp no)
+		(dnp yes)
 		(fields_autoplaced yes)
 		(property "Reference" "#PWR0110"
@@
 		(body_style 1)
 		(exclude_from_sim no)
-		(in_bom yes)
-		(on_board yes)
+		(in_bom no)
+		(on_board no)
 		(in_pos_files yes)
-		(dnp no)
+		(dnp yes)
 		(fields_autoplaced yes)
 		(property "Reference" "#PWR0116"
@@
 		(exclude_from_sim no)
 		(in_bom no)
-		(on_board yes)
+		(on_board no)
 		(in_pos_files yes)
 		(dnp yes)
@@
 		(body_style 1)
 		(exclude_from_sim no)
-		(in_bom yes)
-		(on_board yes)
+		(in_bom no)
+		(on_board no)
 		(in_pos_files yes)
-		(dnp no)
+		(dnp yes)
 		(fields_autoplaced yes)
 		(property "Reference" "#PWR0118"
@@
 		(body_style 1)
 		(exclude_from_sim no)
-		(in_bom yes)
-		(on_board yes)
+		(in_bom no)
+		(on_board no)
 		(in_pos_files yes)
-		(dnp no)
+		(dnp yes)
 		(fields_autoplaced yes)
 		(property "Reference" "M1"
@@
 		(body_style 1)
 		(exclude_from_sim no)
-		(in_bom yes)
-		(on_board yes)
+		(in_bom no)
+		(on_board no)
 		(in_pos_files yes)
-		(dnp no)
+		(dnp yes)
 		(fields_autoplaced yes)
 		(property "Reference" "#PWR0111"
@@
 		(body_style 1)
 		(exclude_from_sim no)
-		(in_bom yes)
-		(on_board yes)
+		(in_bom no)
+		(on_board no)
 		(in_pos_files yes)
-		(dnp no)
+		(dnp yes)
 		(property "Reference" "R68"
 			(at 326.39 161.29 90)
@@
 		(body_style 1)
 		(exclude_from_sim no)
-		(in_bom yes)
-		(on_board yes)
+		(in_bom no)
+		(on_board no)
 		(in_pos_files yes)
-		(dnp no)
+		(dnp yes)
 		(fields_autoplaced yes)
 		(property "Reference" "#PWR0112"
@@
 		(body_style 1)
 		(exclude_from_sim no)
-		(in_bom yes)
-		(on_board yes)
+		(in_bom no)
+		(on_board no)
 		(in_pos_files yes)
-		(dnp no)
+		(dnp yes)
 		(fields_autoplaced yes)
 		(property "Reference" "#PWR0108"
@@
 		(body_style 1)
 		(exclude_from_sim no)
-		(in_bom yes)
-		(on_board yes)
+		(in_bom no)
+		(on_board no)
 		(in_pos_files yes)
-		(dnp no)
+		(dnp yes)
 		(fields_autoplaced yes)
 		(property "Reference" "D26"
@@
 		(body_style 1)
 		(exclude_from_sim no)
-		(in_bom yes)
-		(on_board yes)
+		(in_bom no)
+		(on_board no)
 		(in_pos_files yes)
-		(dnp no)
+		(dnp yes)
 		(fields_autoplaced yes)
 		(property "Reference" "#PWR0109"
@@
 		(body_style 1)
 		(exclude_from_sim no)
-		(in_bom yes)
-		(on_board yes)
+		(in_bom no)
+		(on_board no)
 		(in_pos_files yes)
-		(dnp no)
+		(dnp yes)
 		(property "Reference" "R72"
 			(at 354.33 153.67 0)
@@
 		(exclude_from_sim no)
 		(in_bom no)
-		(on_board yes)
+		(on_board no)
 		(in_pos_files yes)
-		(dnp no)
+		(dnp yes)
 		(property "Reference" "TP11"
 			(at 311.15 154.686 0)
@@
 		(body_style 1)
 		(exclude_from_sim no)
-		(in_bom yes)
-		(on_board yes)
+		(in_bom no)
+		(on_board no)
 		(in_pos_files yes)
-		(dnp no)
+		(dnp yes)
 		(fields_autoplaced yes)
 		(property "Reference" "#PWR0115"

Commit message: Motherboard Complete.
Parts:
- M1: LCSC Part C131334 -> (none)

Commit message: Repository push for Project Deadline :o
Parts:
- C84: value 100nF/50V -> 100nF; footprint A_HDJ_Library:C_0402_1005Metric -> Capacitor_SMD:C_0402_1005Metric; DF_Comment 贴片电容0402-10UF-10V-X5R_GRM155R61A106ME44D -> (none); MPN (none) -> TCC0402X5R104M500AT; SCH_Show_Footprint C0402 -> (none); Specifications (For Resistors/Capacitors) (none) -> 100nF 0402 Ceramic 20% 50V X5R; now fitted; now in the parts list
- C85: SCH_Show_Footprint C0402 -> (none)
- D26: MPN (none) -> 1N5819WS; SCH_Show_Footprint SOD-323 -> (none); Specifications (For Resistors/Capacitors) (none) -> N/A; now fitted; now in the parts list
- D27: SCH_Show_Footprint SOD-323 -> (none)
- M1: DF_Comment JST B4B-PH-K-S(LF)(SN) -> (none); now fitted; now in the parts list
- R68: footprint A_HDJ_Library:R_0402_1005Metric -> Resistor_SMD:R_0402_1005Metric; DF_Comment 贴片电阻0402-10K-1% -> (none); MPN (none) -> 0402WGF2152TCE; Specifications (For Resistors/Capacitors) (none) -> 21.5k 1% 63mW 0402; now fitted; now in the parts list
- R69: footprint A_HDJ_Library:R_0402_1005Metric -> Resistor_SMD:R_0402_1005Metric; DF_Comment 贴片电阻0402-10K-1% -> (none); MPN (none) -> AC0402FR-07100RL; Specifications (For Resistors/Capacitors) (none) -> 100R 1% 63mW 0402; now fitted; now in the parts list
- R72: footprint A_HDJ_Library:R_0402_1005Metric -> Resistor_SMD:R_0402_1005Metric; DF_Comment 贴片电阻0402-10K-1% -> (none); MPN (none) -> CQ02WGF4701TCE; Specifications (For Resistors/Capacitors) (none) -> 4.7k 1% 63mW 0402; now fitted; now in the parts list
- TP11, TP12: Specifications (For Resistors/Capacitors) (none) -> N/A; now fitted; now in the parts list
