File: Motherboard/GPIO.kicad_sch (KiCad schematic)
At the start: 12 parts, among them J19 BM04B-NSHSS-TBT_LF__SN_, J20 BM04B-NSHSS-TBT_LF__SN_, J50 5034801400, J51 5034801400, J52 503480-0800

Commit message: Routed RP2354B, USB ports, rewired HDMI lanes to be cleaner, and many other fixes and improvements.
Connections:
- net at R133.2: now also J52.4; no longer J52.3
- net at R132.2: now also J52.2; no longer J52.5
- net at R131.2: now also J52.1; no longer J52.6
- net at R130.2: now also J52.5; no longer J52.2
- net at R84.2: now also J52.6; no longer J52.1
- net at R119.2: now also J52.3; no longer J52.4
Other:
- moved on the sheet: R119, R130, R131, R132, R133, R84
Changed lines of the file:
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@@
 	(wire
 		(pts
-			(xy 326.39 302.26) (xy 314.96 302.26)
+			(xy 314.96 289.56) (xy 326.39 289.56)
 		)
 		(stroke
@@
 	(wire
 		(pts
-			(xy 314.96 294.64) (xy 326.39 294.64)
+			(xy 314.96 297.18) (xy 326.39 297.18)
 		)
 		(stroke
@@
 	(wire
 		(pts
-			(xy 295.91 214.63) (xy 309.88 214.63)
+			(xy 325.12 302.26) (xy 326.39 302.26)
 		)
 		(stroke
@@
 	(wire
 		(pts
-			(xy 295.91 241.3) (xy 295.91 243.84)
+			(xy 325.12 294.64) (xy 326.39 294.64)
 		)
 		(stroke
@@
 	(wire
 		(pts
-			(xy 325.12 297.18) (xy 326.39 297.18)
+			(xy 295.91 214.63) (xy 309.88 214.63)
 		)
 		(stroke
@@
 	(wire
 		(pts
-			(xy 295.91 191.77) (xy 295.91 189.23)
+			(xy 295.91 241.3) (xy 295.91 243.84)
 		)
 		(stroke
@@
 	(wire
 		(pts
-			(xy 317.5 289.56) (xy 298.45 289.56)
+			(xy 295.91 191.77) (xy 295.91 189.23)
 		)
 		(stroke
@@
 	(wire
 		(pts
-			(xy 326.39 289.56) (xy 325.12 289.56)
+			(xy 317.5 302.26) (xy 298.45 302.26)
 		)
 		(stroke
@@
 	(wire
 		(pts
-			(xy 298.45 294.64) (xy 307.34 294.64)
+			(xy 298.45 297.18) (xy 307.34 297.18)
 		)
 		(stroke
@@
 	(wire
 		(pts
-			(xy 307.34 302.26) (xy 298.45 302.26)
+			(xy 307.34 289.56) (xy 298.45 289.56)
 		)
 		(stroke
@@
 	(wire
 		(pts
-			(xy 326.39 292.1) (xy 306.07 292.1)
+			(xy 326.39 299.72) (xy 306.07 299.72)
 		)
 		(stroke
@@
 	(wire
 		(pts
-			(xy 317.5 297.18) (xy 298.45 297.18)
+			(xy 317.5 294.64) (xy 298.45 294.64)
 		)
 		(stroke
@@
 	(wire
 		(pts
-			(xy 326.39 299.72) (xy 306.07 299.72)
+			(xy 326.39 292.1) (xy 306.07 292.1)
 		)
 		(stroke
@@
 	(hierarchical_label "LED_PWR_B"
 		(shape input)
-		(at 326.39 302.26 0)
+		(at 326.39 289.56 0)
 		(effects
 			(font
@@
 	(hierarchical_label "LED_WiFi_G"
 		(shape input)
-		(at 326.39 292.1 0)
+		(at 326.39 299.72 0)
 		(effects
 			(font
@@
 	(hierarchical_label "LED_WiFi_R"
 		(shape input)
-		(at 326.39 289.56 0)
+		(at 326.39 302.26 0)
 		(effects
 			(font
@@
 	(hierarchical_label "LED_PWR_R"
 		(shape input)
-		(at 326.39 297.18 0)
+		(at 326.39 294.64 0)
 		(effects
 			(font
@@
 	(hierarchical_label "LED_PWR_G"
 		(shape input)
-		(at 326.39 299.72 0)
+		(at 326.39 292.1 0)
 		(effects
 			(font
@@
 	(hierarchical_label "LED_WiFi_B"
 		(shape input)
-		(at 326.39 294.64 0)
+		(at 326.39 297.18 0)
 		(effects
 			(font
@@
 	(symbol
 		(lib_id "Device:R")
-		(at 311.15 294.64 270)
+		(at 311.15 297.18 270)
 		(unit 1)
 		(body_style 1)
@@
 		(dnp no)
 		(property "Reference" "R133"
-			(at 311.15 290.576 90)
+			(at 311.15 293.116 90)
 			(show_name no)
 			(do_not_autoplace no)
@@
 		)
 		(property "Value" "47R/1%"
-			(at 311.15 292.354 90)
+			(at 311.15 294.894 90)
 			(show_name no)
 			(do_not_autoplace no)
@@
 		)
 		(property "Footprint" "Resistor_SMD:R_0402_1005Metric"
-			(at 311.15 292.862 90)
+			(at 311.15 295.402 90)
 			(hide yes)
 			(show_name no)
@@
 		)
 		(property "Datasheet" ""
-			(at 311.15 294.64 0)
+			(at 311.15 297.18 0)
 			(hide yes)
 			(show_name no)
@@
 		)
 		(property "Description" "Resistor"
-			(at 311.15 294.64 0)
+			(at 311.15 297.18 0)
 			(hide yes)
 			(show_name no)
@@
 	(symbol
 		(lib_id "Device:R")
-		(at 302.26 299.72 270)
+		(at 302.26 292.1 270)
 		(unit 1)
 		(body_style 1)
@@
 		(dnp no)
 		(property "Reference" "R132"
-			(at 302.26 295.656 90)
+			(at 302.26 288.036 90)
 			(show_name no)
 			(do_not_autoplace no)
@@
 		)
 		(property "Value" "47R/1%"
-			(at 302.26 297.434 90)
+			(at 302.26 289.814 90)
 			(show_name no)
 			(do_not_autoplace no)
@@
 		)
 		(property "Footprint" "Resistor_SMD:R_0402_1005Metric"
-			(at 302.26 297.942 90)
+			(at 302.26 290.322 90)
 			(hide yes)
 			(show_name no)
@@
 		)
 		(property "Datasheet" ""
-			(at 302.26 299.72 0)
+			(at 302.26 292.1 0)
 			(hide yes)
 			(show_name no)
@@
 		)
 		(property "Description" "Resistor"
-			(at 302.26 299.72 0)
+			(at 302.26 292.1 0)
 			(hide yes)
 			(show_name no)
@@
 	(symbol
 		(lib_id "Device:R")
-		(at 311.15 302.26 270)
+		(at 311.15 289.56 270)
 		(unit 1)
 		(body_style 1)
@@
 		(dnp no)
 		(property "Reference" "R131"
-			(at 311.15 298.196 90)
+			(at 311.15 285.496 90)
 			(show_name no)
 			(do_not_autoplace no)
@@
 		)
 		(property "Value" "47R/1%"
-			(at 311.15 299.974 90)
+			(at 311.15 287.274 90)
 			(show_name no)
 			(do_not_autoplace no)
@@
 		)
 		(property "Footprint" "Resistor_SMD:R_0402_1005Metric"
-			(at 311.15 300.482 90)
+			(at 311.15 287.782 90)
 			(hide yes)
 			(show_name no)
@@
 		)
 		(property "Datasheet" ""
-			(at 311.15 302.26 0)
+			(at 311.15 289.56 0)
 			(hide yes)
 			(show_name no)
@@
 		)
 		(property "Description" "Resistor"
-			(at 311.15 302.26 0)
+			(at 311.15 289.56 0)
 			(hide yes)
 			(show_name no)
@@
 	(symbol
 		(lib_id "Device:R")
-		(at 302.26 292.1 270)
+		(at 302.26 299.72 270)
 		(unit 1)
 		(body_style 1)
@@
 		(dnp no)
 		(property "Reference" "R130"
-			(at 302.26 288.036 90)
+			(at 302.26 295.656 90)
 			(show_name no)
 			(do_not_autoplace no)
@@
 		)
 		(property "Value" "47R/1%"
-			(at 302.26 289.814 90)
+			(at 302.26 297.434 90)
 			(show_name no)
 			(do_not_autoplace no)
@@
 		)
 		(property "Footprint" "Resistor_SMD:R_0402_1005Metric"
-			(at 302.26 290.322 90)
+			(at 302.26 297.942 90)
 			(hide yes)
 			(show_name no)
@@
 		)
 		(property "Datasheet" ""
-			(at 302.26 292.1 0)
+			(at 302.26 299.72 0)
 			(hide yes)
 			(show_name no)
@@
 		)
 		(property "Description" "Resistor"
-			(at 302.26 292.1 0)
+			(at 302.26 299.72 0)
 			(hide yes)
 			(show_name no)
@@
 	(symbol
 		(lib_id "Device:R")
-		(at 321.31 289.56 270)
+		(at 321.31 302.26 270)
 		(unit 1)
 		(body_style 1)
@@
 		(dnp no)
 		(property "Reference" "R84"
-			(at 321.31 285.496 90)
+			(at 321.31 298.196 90)
 			(show_name no)
 			(do_not_autoplace no)
@@
 		)
 		(property "Value" "150R/1%"
-			(at 321.31 287.274 90)
+			(at 321.31 299.974 90)
 			(show_name no)
 			(do_not_autoplace no)
@@
 		)
 		(property "Footprint" "Resistor_SMD:R_0402_1005Metric"
-			(at 321.31 287.782 90)
+			(at 321.31 300.482 90)
 			(hide yes)
 			(show_name no)
@@
 		)
 		(property "Datasheet" ""
-			(at 321.31 289.56 0)
+			(at 321.31 302.26 0)
 			(hide yes)
 			(show_name no)
@@
 		)
 		(property "Description" "Resistor"
-			(at 321.31 289.56 0)
+			(at 321.31 302.26 0)
 			(hide yes)
 			(show_name no)
@@
 	(symbol
 		(lib_id "Device:R")
-		(at 321.31 297.18 270)
+		(at 321.31 294.64 270)
 		(unit 1)
 		(body_style 1)
@@
 		(dnp no)
 		(property "Reference" "R119"
-			(at 321.31 293.116 90)
+			(at 321.31 290.576 90)
 			(show_name no)
 			(do_not_autoplace no)
@@
 		)
 		(property "Value" "150R/1%"
-			(at 321.31 294.894 90)
+			(at 321.31 292.354 90)
 			(show_name no)
 			(do_not_autoplace no)
@@
 		)
 		(property "Footprint" "Resistor_SMD:R_0402_1005Metric"
-			(at 321.31 295.402 90)
+			(at 321.31 292.862 90)
 			(hide yes)
 			(show_name no)
@@
 		)
 		(property "Datasheet" ""
-			(at 321.31 297.18 0)
+			(at 321.31 294.64 0)
 			(hide yes)
 			(show_name no)
@@
 		)
 		(property "Description" "Resistor"
-			(at 321.31 297.18 0)
-			(hide yes)
-			(show_name no)
+			(at 321.31 294.64 0)
+			(hide yes)
+			(show_name no)

Commit message: Created updated BOM for PCBWay on all CTRL daughterboards. These boards have likely hit their final* version
*Ive said "Finished Version" many times in this project. I'm confident now, but no guarantees.
Parts:
- D33: DF_Comment 双向静电保护二极管_ESD5V0B03-1006_DFN1006 -> (none); LCSC Part C521894 -> (none); MPN (none) -> ESD5V0B03-1006
- J50, J51: MPN (none) -> 5034801400
- J52: MPN (none) -> 5034800800; Manufacturer_Part_Number 503480-0800 -> (none)
Other:
- note removed: "Update these to use top facing connectors"

Commit message: Routed 1V8, 3V3 and 9V voltage regulators
Connections:
- net +1V8: now also J51.2; no longer J50.6
- net +3V3: now also J50.6; no longer J51.2
- net SL_BRI: now also J51.1; no longer J50.7
- net SL_VOL: now also J50.7; no longer J51.1
Changed lines of the file:
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@@
 	(wire
 		(pts
-			(xy 314.96 289.56) (xy 326.39 289.56)
+			(xy 295.91 276.86) (xy 307.34 276.86)
 		)
 		(stroke
@@
 	(wire
 		(pts
-			(xy 314.96 297.18) (xy 326.39 297.18)
+			(xy 314.96 289.56) (xy 326.39 289.56)
 		)
 		(stroke
@@
 	(wire
 		(pts
-			(xy 295.91 276.86) (xy 307.34 276.86)
+			(xy 314.96 297.18) (xy 326.39 297.18)
 		)
 		(stroke
@@
 	(wire
 		(pts
-			(xy 325.12 302.26) (xy 326.39 302.26)
+			(xy 295.91 214.63) (xy 307.34 214.63)
 		)
 		(stroke
@@
 	(wire
 		(pts
-			(xy 325.12 294.64) (xy 326.39 294.64)
+			(xy 325.12 302.26) (xy 326.39 302.26)
 		)
 		(stroke
@@
 	(wire
 		(pts
-			(xy 295.91 214.63) (xy 309.88 214.63)
+			(xy 325.12 294.64) (xy 326.39 294.64)
 		)
 		(stroke
@@
 	(hierarchical_label "SL_VOL"
 		(shape output)
-		(at 295.91 279.4 0)
+		(at 295.91 212.09 0)
 		(effects
 			(font
@@
 	(hierarchical_label "SL_BRI"
 		(shape output)
-		(at 295.91 212.09 0)
+		(at 295.91 279.4 0)
 		(effects
 			(font
@@
 	(symbol
 		(lib_id "power:+1V8")
-		(at 309.88 214.63 270)
+		(at 307.34 276.86 270)
 		(unit 1)
 		(body_style 1)
@@
 		(fields_autoplaced yes)
 		(property "Reference" "#PWR0145"
-			(at 306.07 214.63 0)
+			(at 303.53 276.86 0)
 			(hide yes)
 			(show_name no)
@@
 		)
 		(property "Value" "+1V8"
-			(at 313.69 214.6299 90)
+			(at 311.15 276.8599 90)
 			(show_name no)
 			(do_not_autoplace no)
@@
 		)
 		(property "Footprint" ""
-			(at 309.88 214.63 0)
+			(at 307.34 276.86 0)
 			(hide yes)
 			(show_name no)
@@
 		)
 		(property "Datasheet" ""
-			(at 309.88 214.63 0)
+			(at 307.34 276.86 0)
 			(hide yes)
 			(show_name no)
@@
 		)
 		(property "Description" "Power symbol creates a global label with name \"+1V8\""
-			(at 309.88 214.63 0)
+			(at 307.34 276.86 0)
 			(hide yes)
 			(show_name no)
@@
 	(symbol
 		(lib_id "power:+3V3")
-		(at 307.34 276.86 270)
+		(at 307.34 214.63 270)
 		(mirror x)
 		(unit 1)
@@
 		(fields_autoplaced yes)
 		(property "Reference" "#PWR026"
-			(at 303.53 276.86 0)
+			(at 303.53 214.63 0)
 			(hide yes)
 			(show_name no)
@@
 		)
 		(property "Value" "+3V3"
-			(at 311.15 276.8599 90)
+			(at 311.15 214.6299 90)
 			(show_name no)
 			(do_not_autoplace no)
@@
 		)
 		(property "Footprint" ""
-			(at 307.34 276.86 0)
+			(at 307.34 214.63 0)
 			(hide yes)
 			(show_name no)
@@
 		)
 		(property "Datasheet" ""
-			(at 307.34 276.86 0)
+			(at 307.34 214.63 0)
 			(hide yes)
 			(show_name no)
@@
 		)
 		(property "Description" "Power symbol creates a global label with name \"+3V3\""
-			(at 307.34 276.86 0)
+			(at 307.34 214.63 0)
 			(hide yes)
 			(show_name no)

Commit message: Motherboard Complete.
Parts:
- D33, J50, J51: Specifications (For Resistors/Capacitors) (none) -> N/A
- J19, J20: Manufacturer_Name JST (JAPAN SOLDERLESS TERMINALS) -> (none); Manufacturer_Part_Number BM04B-NSHSS-TBT(LF)(SN) -> (none); Mouser Part Number 306-4BNSHSSTBTL -> (none); Mouser Price/Stock https://www.mouser.co.uk/ProductDetail/JST-Commercial/BM04B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 -> (none)
- J52: LCSC Part C596711 -> (none); Manufacturer_Name Molex -> (none); Mouser Price/Stock https://www.mouser.co.uk/ProductDetail/Molex/503480-0800?qs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 -> (none); Specifications (For Resistors/Capacitors) (none) -> N/A
- R119, R84: MPN (none) -> any/open; Specifications (For Resistors/Capacitors) (none) -> 150R 1% 63mW 0402
- R130, R131, R132, R133: MPN (none) -> any/open; Specifications (For Resistors/Capacitors) (none) -> 47R 1% 63mW 0402

Commit message: Majorly reworked Display system, condensed and fixed BOM, and many other schematic and design cleanups. \Programs folder was also cleaned up.
Everything is still a work in progress, many things are now unfinished, especially the PCB.
Parts:
- R119, R84: MPN any/open -> 0402WGF1500TCE
- R130, R131, R132, R133: MPN any/open -> AC0402FR-0747RL
Changed lines of the file:
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@@
 	)
 	(symbol
+		(lib_id "power:+1V8")
+		(at 307.34 276.86 270)
+		(unit 1)
+		(body_style 1)
+		(exclude_from_sim no)
+		(in_bom yes)
+		(on_board yes)
+		(in_pos_files yes)
+		(dnp no)
+		(fields_autoplaced yes)
+		(property "Reference" "#PWR0131"
+			(at 303.53 276.86 0)
+			(hide yes)
+			(show_name no)
+			(do_not_autoplace no)
+			(effects
+				(font
+					(size 1.27 1.27)
+				)
+			)
+		)
+		(property "Value" "+1V8"
+			(at 311.15 276.8599 90)
+			(show_name no)
+			(do_not_autoplace no)
+			(effects
+				(font
+					(size 1.27 1.27)
+				)
+				(justify left)
+			)
+		)
+		(property "Footprint" ""
+			(at 307.34 276.86 0)
+			(hide yes)
+			(show_name no)
+			(do_not_autoplace no)
+			(effects
+				(font
+					(size 1.27 1.27)
+				)
+			)
+		)
+		(property "Datasheet" ""
+			(at 307.34 276.86 0)
+			(hide yes)
+			(show_name no)
+			(do_not_autoplace no)
+			(effects
+				(font
+					(size 1.27 1.27)
+				)
+			)
+		)
+		(property "Description" "Power symbol creates a global label with name \"+1V8\""
+			(at 307.34 276.86 0)
+			(hide yes)
+			(show_name no)
+			(do_not_autoplace no)
+			(effects
+				(font
+					(size 1.27 1.27)
+				)
+			)
+		)
+		(pin "1"
+		)
+		(instances
+			(project "Motherboard"
+				(path "/2a6d114a-7fd7-4207-b5f7-4ea9c34f36aa/f7e36582-0575-4ab7-aed9-3fad0f8951d3"
+					(reference "#PWR0131")
+					(unit 1)
+				)
+			)
+		)
+	)
+	(symbol
 		(lib_id "power:GND")
 		(at 298.45 304.8 90)
@@
 			)
 		)
-		(property "MPN" "any/open"
+		(property "MPN" "AC0402FR-0747RL"
 			(at 311.15 297.18 90)
 			(hide yes)
@@
 			)
 		)
-		(property "MPN" "any/open"
+		(property "MPN" "AC0402FR-0747RL"
 			(at 302.26 292.1 90)
 			(hide yes)
@@
 			)
 		)
-		(property "MPN" "any/open"
+		(property "MPN" "AC0402FR-0747RL"
 			(at 311.15 289.56 90)
 			(hide yes)
@@
 			)
 		)
-		(property "MPN" "any/open"
+		(property "MPN" "AC0402FR-0747RL"
 			(at 302.26 299.72 90)
 			(hide yes)
@@
 			)
 		)
-		(property "MPN" "any/open"
+		(property "MPN" "0402WGF1500TCE"
 			(at 321.31 302.26 90)
 			(hide yes)
@@
 	)
 	(symbol
-		(lib_id "power:+1V8")
-		(at 307.34 276.86 270)
-		(unit 1)
-		(body_style 1)
-		(exclude_from_sim no)
-		(in_bom yes)
-		(on_board yes)
-		(in_pos_files yes)
-		(dnp no)
-		(fields_autoplaced yes)
-		(property "Reference" "#PWR0145"
-			(at 303.53 276.86 0)
-			(hide yes)
-			(show_name no)
-			(do_not_autoplace no)
-			(effects
-				(font
-					(size 1.27 1.27)
-				)
-			)
-		)
-		(property "Value" "+1V8"
-			(at 311.15 276.8599 90)
-			(show_name no)
-			(do_not_autoplace no)
-			(effects
-				(font
-					(size 1.27 1.27)
-				)
-				(justify left)
-			)
-		)
-		(property "Footprint" ""
-			(at 307.34 276.86 0)
-			(hide yes)
-			(show_name no)
-			(do_not_autoplace no)
-			(effects
-				(font
-					(size 1.27 1.27)
-				)
-			)
-		)
-		(property "Datasheet" ""
-			(at 307.34 276.86 0)
-			(hide yes)
-			(show_name no)
-			(do_not_autoplace no)
-			(effects
-				(font
-					(size 1.27 1.27)
-				)
-			)
-		)
-		(property "Description" "Power symbol creates a global label with name \"+1V8\""
-			(at 307.34 276.86 0)
-			(hide yes)
-			(show_name no)
-			(do_not_autoplace no)
-			(effects
-				(font
-					(size 1.27 1.27)
-				)
-			)
-		)
-		(pin "1"
-		)
-		(instances
-			(project "Motherboard"
-				(path "/2a6d114a-7fd7-4207-b5f7-4ea9c34f36aa/f7e36582-0575-4ab7-aed9-3fad0f8951d3"
-					(reference "#PWR0145")
-					(unit 1)
-				)
-			)
-		)
-	)
-	(symbol
 		(lib_id "Diode:ESD9B5.0ST5G")
 		(at 300.99 311.15 270)
@@
 			)
 		)
-		(property "MPN" "any/open"
+		(property "MPN" "0402WGF1500TCE"
 			(at 321.31 294.64 90)
 			(hide yes)

Commit message: General Readme update
Connections:
- net +1V8 is gone; now on net +3V3: J51.2
Changed lines of the file:
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@@
-	)
-	(symbol
-		(lib_id "power:+1V8")
-		(at 307.34 276.86 270)
-		(unit 1)
-		(body_style 1)
-		(exclude_from_sim no)
-		(in_bom yes)
-		(on_board yes)
-		(in_pos_files yes)
-		(dnp no)
-		(fields_autoplaced yes)
-		(property "Reference" "#PWR0131"
-			(at 303.53 276.86 0)
-			(hide yes)
-			(show_name no)
-			(do_not_autoplace no)
-			(effects
-				(font
-					(size 1.27 1.27)
-				)
-			)
-		)
-		(property "Value" "+1V8"
-			(at 311.15 276.8599 90)
-			(show_name no)
-			(do_not_autoplace no)
-			(effects
-				(font
-					(size 1.27 1.27)
-				)
-				(justify left)
-			)
-		)
-		(property "Footprint" ""
-			(at 307.34 276.86 0)
-			(hide yes)
-			(show_name no)
-			(do_not_autoplace no)
-			(effects
-				(font
-					(size 1.27 1.27)
-				)
-			)
-		)
-		(property "Datasheet" ""
-			(at 307.34 276.86 0)
-			(hide yes)
-			(show_name no)
-			(do_not_autoplace no)
-			(effects
-				(font
-					(size 1.27 1.27)
-				)
-			)
-		)
-		(property "Description" "Power symbol creates a global label with name \"+1V8\""
-			(at 307.34 276.86 0)
-			(hide yes)
-			(show_name no)
-			(do_not_autoplace no)
-			(effects
-				(font
-					(size 1.27 1.27)
-				)
-			)
-		)
-		(pin "1"
-		)
-		(instances
-			(project "Motherboard"
-				(path "/2a6d114a-7fd7-4207-b5f7-4ea9c34f36aa/f7e36582-0575-4ab7-aed9-3fad0f8951d3"
-					(reference "#PWR0131")
-					(unit 1)
-				)
-			)
-		)
 	)
 	(symbol
@@
 					(unit 1)
 				)
+			)
+		)
+	)
+	(symbol
+		(lib_id "power:+3V3")
+		(at 307.34 276.86 270)
+		(mirror x)
+		(unit 1)
+		(body_style 1)
+		(exclude_from_sim no)
+		(in_bom yes)
+		(on_board yes)
+		(in_pos_files yes)
+		(dnp no)
+		(fields_autoplaced yes)
+		(property "Reference" "#PWR039"
+			(at 303.53 276.86 0)
+			(hide yes)
+			(show_name no)
+			(do_not_autoplace no)
+			(effects
+				(font
+					(size 1.27 1.27)
+				)
+			)
+		)
+		(property "Value" "+3V3"
+			(at 311.15 276.8599 90)
+			(show_name no)
+			(do_not_autoplace no)
+			(effects
+				(font
+					(size 1.27 1.27)
+				)
+				(justify left)
+			)
+		)
+		(property "Footprint" ""
+			(at 307.34 276.86 0)
+			(hide yes)
+			(show_name no)
+			(do_not_autoplace no)
+			(effects
+				(font
+					(size 1.27 1.27)
+				)
+			)
+		)
+		(property "Datasheet" ""
+			(at 307.34 276.86 0)
+			(hide yes)
+			(show_name no)
+			(do_not_autoplace no)
+			(effects
+				(font
+					(size 1.27 1.27)
+				)
+			)
+		)
+		(property "Description" "Power symbol creates a global label with name \"+3V3\""
+			(at 307.34 276.86 0)
+			(hide yes)
+			(show_name no)
+			(do_not_autoplace no)
+			(effects
+				(font
+					(size 1.27 1.27)
+				)
+			)
+		)
+		(pin "1"
+		)
+		(instances
+			(project "Motherboard"
+				(path "/2a6d114a-7fd7-4207-b5f7-4ea9c34f36aa/f7e36582-0575-4ab7-aed9-3fad0f8951d3"
+					(reference "#PWR039")
+					(unit 1)
+				)

Commit message: Repository push for Project Deadline :o
Parts:
- D33: Buy_Link https://item.szlcsc.com/539388.html -> (none); SCH_Show_Footprint D0402 -> (none)
- J19, J20: Height 6 -> (none)
- J52: Height 1.87 -> (none)
