File: CTRL_PWR/_autosave-CTRL_PWR.kicad_pcb (KiCad board)
At the start: 2 copper layers, 34 x 17 mm, 9 parts, among them J1 BM09B-NSHSS-TBT_LF__SN_

Commit message: Corrected CTRL_PWR (+other WIP changes)
Connections:
- J1 pad 2: +3V3 -> GND
Changed lines of the file:
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@@
 			(size 0.6 1.7)
 			(layers "B.Cu" "B.Mask" "B.Paste")
-			(net "+3V3")
+			(net "GND")
 			(pinfunction "2_2")
 			(pintype "passive")
@@
 		)
 		(min_thickness 0.0254)
-		(fill
+		(fill yes
 			(island_removal_mode 1)
 		)
@@
 		)
 		(min_thickness 0.25)
-		(fill
+		(fill yes
 			(thermal_gap 0.5)
 			(thermal_bridge_width 0.5)
