File: CTRL_PWR/CTRL_PWR.kicad_sch (KiCad schematic)
At the start: 6 parts, among them J1 BM09B-NSHSS-TBT_LF__SN_

Commit message: Corrected CTRL_PWR (+other WIP changes)
Parts:
- removed D1: LED_PWR, LED_THT:LED_D5.0mm-4_RGB, symbol Device:LED_BGKR
- removed D2: LED_WIFI, LED_THT:LED_D5.0mm-4_RGB, symbol Device:LED_BGKR
- added D21: ESD5V0B03, A_HDJ_Library:D_0402_1005Metric, symbol Diode:ESD9B5.0ST5G
- added D3, D4: LED_RKGB, LED_THT:LED_D5.0mm-4_RGB, symbol Device:LED_RKGB
Connections:
- net +3V3 is gone; now on net GND: J1.2, S1.3 (NO_1), S1.4 (NO_2)
- net GND: now also D21.2 (A2), D3.2 (K), D4.2 (K)
- net at J1.7: now also D4.4 (BA)
- net at J1.8: now also D4.3 (GA)
- net at J1.9: now also D4.1 (RA)
- net at J1.1, S1.1 (COM_1), S1.2 (COM_2): now also D21.1 (A1)
- net at J1.5: now also D3.1 (RA)
- net at J1.4: now also D3.3 (GA)
- net at J1.3: now also D3.4 (BA)

Commit message: CTRL_PWR updated to use 8P FPC Connector
Parts:
- removed J1: BM09B-NSHSS-TBT_LF__SN_, BM09B-NSHSS-TBT_LF__SN_:BM09BNSHSSTBTLFSN, symbol BM09B-NSHSS-TBT_LF__SN_:BM09B-NSHSS-TBT_LF__SN_
- added J2: 503480-0800, 503480-0800:5034800800, symbol 503480-0800:503480-0800
- D21: LCSC Part (none) -> C521894
- D3, D4: LCSC Part (none) -> C2837020
- S1: Height 4.3 -> (none); LCSC Part (none) -> C2733654; Manufacturer_Name OMRON Electronics -> (none); Manufacturer_Part_Number B3S-1002 -> (none); Mouser Part Number 653-B3S-1002 -> (none); Mouser Price/Stock https://www.mouser.co.uk/ProductDetail/Omron-Electronics/B3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 -> (none)
Connections:
- net GND: now also J2.10, J2.7, J2.9
- net at D3.1 (RA): now also J2.4
- net at D3.3 (GA): now also J2.5
- net at D3.4 (BA): now also J2.6
- net at D4.1 (RA): now also J2.1
- net at D4.3 (GA): now also J2.2
- net at D4.4 (BA): now also J2.3
- net at D21.1 (A1), S1.1 (COM_1), S1.2 (COM_2): now also J2.8

Commit message: Updated CTRL_Z to use 3 pin FPC and ESD Protection.
Parts:
- J2: LCSC Part (none) -> C596711; Mouser Part Number 538-503480-0800 -> (none)
Changed lines of the file:
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@@
 			)
 		)
-		(property "Mouser Part Number" "538-503480-0800"
+		(property "LCSC Part" "C596711"
 			(at 43.18 572.39 0)
 			(hide yes)

Commit message: Added resistors to the LEDs on CTRL_PWR
Parts:
- added R1, R2: 180R, Resistor_SMD:R_0402_1005Metric, symbol Device:R
- added R3, R4, R5, R6: 47R, Resistor_SMD:R_0402_1005Metric, symbol Device:R
Connections:
- net at D3.1 (RA): now also R1.2; no longer J2.4
- net at J2.5: now also R3.1; no longer D3.3 (GA)
- net at D3.4 (BA): now also R4.2; no longer J2.6
- net at D4.1 (RA): now also R2.2; no longer J2.1
- net at D4.3 (GA): now also R5.2; no longer J2.2
- net at D4.4 (BA): now also R6.2; no longer J2.3
- new net: D3.3 (GA), R3.2
- new net: J2.6, R4.1
- new net: J2.1, R2.1
- new net: J2.3, R6.1
- new net: J2.4, R1.1
- new net: J2.2, R5.1

Commit message: Updated CTRLs to be one sided (saves a billion dollars somehow), added LCSC_Parts for BOM, and other fixes. (Part 1/2)
Parts:
- H1, H2: LCSC Part (none) -> N/A
Connections:
- net GND: now also J2.2; no longer J2.7
- net at R3.1: now also J2.4; no longer J2.5
- net at R4.1: now also J2.3; no longer J2.6
- net at D21.1 (A1), S1.1 (COM_1), S1.2 (COM_2): now also J2.1; no longer J2.8
- net at R2.1: now also J2.8; no longer J2.1
- net at R6.1: now also J2.6; no longer J2.3
- net at R1.1: now also J2.5; no longer J2.4
- net at R5.1: now also J2.7; no longer J2.2
Changed lines of the file:
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@@
 	(symbol
 		(lib_id "power:GND")
-		(at 24.13 77.47 270)
+		(at 24.13 92.71 270)
 		(unit 1)
 		(body_style 1)
@@
 		(fields_autoplaced yes)
 		(property "Reference" "#PWR03"
-			(at 17.78 77.47 0)
+			(at 17.78 92.71 0)
 			(hide yes)
 			(show_name no)
@@
 		)
 		(property "Value" "GND"
-			(at 20.32 77.4699 90)
+			(at 20.32 92.7099 90)
 			(show_name no)
 			(do_not_autoplace no)
@@
 		)
 		(property "Footprint" ""
-			(at 24.13 77.47 0)
+			(at 24.13 92.71 0)
 			(hide yes)
 			(show_name no)
@@
 		)
 		(property "Datasheet" ""
-			(at 24.13 77.47 0)
+			(at 24.13 92.71 0)
 			(hide yes)
 			(show_name no)
@@
 		)
 		(property "Description" "Power symbol creates a global label with name \"GND\" , ground"
-			(at 24.13 77.47 0)
+			(at 24.13 92.71 0)
 			(hide yes)
 			(show_name no)
@@
 			)
 		)
+		(property "LCSC Part" "N/A"
+			(at 72.39 135.89 0)
+			(hide yes)
+			(show_name no)
+			(do_not_autoplace no)
+			(effects
+				(font
+					(size 1.27 1.27)
+				)
+			)
+		)
 		(instances
 			(project "CTRL_PWR"
@@
 	(symbol
 		(lib_id "power:GND")
-		(at 24.13 80.01 270)
+		(at 24.13 95.25 270)
 		(unit 1)
 		(body_style 1)
@@
 		(fields_autoplaced yes)
 		(property "Reference" "#PWR04"
-			(at 17.78 80.01 0)
+			(at 17.78 95.25 0)
 			(hide yes)
 			(show_name no)
@@
 		)
 		(property "Value" "GND"
-			(at 20.32 80.0099 90)
+			(at 20.32 95.2499 90)
 			(show_name no)
 			(do_not_autoplace no)
@@
 		)
 		(property "Footprint" ""
-			(at 24.13 80.01 0)
+			(at 24.13 95.25 0)
 			(hide yes)
 			(show_name no)
@@
 		)
 		(property "Datasheet" ""
-			(at 24.13 80.01 0)
+			(at 24.13 95.25 0)
 			(hide yes)
 			(show_name no)
@@
 		)
 		(property "Description" "Power symbol creates a global label with name \"GND\" , ground"
-			(at 24.13 80.01 0)
+			(at 24.13 95.25 0)
 			(hide yes)
 			(show_name no)
@@
 	(symbol
 		(lib_id "503480-0800:503480-0800")
-		(at 24.13 77.47 0)
+		(at 24.13 95.25 0)
+		(mirror x)
 		(unit 1)
 		(body_style 1)
@@
 		(dnp no)
 		(property "Reference" "J2"
-			(at 35.56 102.87 0)
+			(at 35.56 69.85 0)
 			(show_name no)
 			(do_not_autoplace no)
@@
 		)
 		(property "Value" "503480-0800"
-			(at 35.56 100.33 0)
+			(at 35.56 72.39 0)
 			(show_name no)
 			(do_not_autoplace no)
@@
 		)
 		(property "Footprint" "503480-0800:5034800800"
-			(at 43.18 172.39 0)
+			(at 43.18 0.33 0)
 			(hide yes)
 			(show_name no)
@@
 		)
 		(property "Datasheet" "https://datasheet.datasheetarchive.com/originals/distributors/Datasheets_SAMA/dd73662b6fd345cd2d55f223314e3d3c.pdf"
-			(at 43.18 272.39 0)
+			(at 43.18 -99.67 0)
 			(hide yes)
 			(show_name no)
@@
 		)
 		(property "Description" "Easy-On BackFlip 0.5mm FPC Connector, 8P Molex 503480 Series 0.5mm Pitch 8 Way Right Angle SMT Male FPC Connector, Solder"
-			(at 24.13 77.47 0)
+			(at 24.13 95.25 0)
 			(hide yes)
 			(show_name no)
@@
 		)
 		(property "Height" "1.87"
-			(at 43.18 472.39 0)
+			(at 43.18 -299.67 0)
 			(hide yes)
 			(show_name no)
@@
 		)
 		(property "LCSC Part" "C596711"
-			(at 43.18 572.39 0)
+			(at 43.18 -399.67 0)
 			(hide yes)
 			(show_name no)
@@
 		)
 		(property "Mouser Price/Stock" "https://www.mouser.co.uk/ProductDetail/Molex/503480-0800?qs=bodV9ulq6Gz33SKuZL445g%3D%3D"
-			(at 43.18 672.39 0)
+			(at 43.18 -499.67 0)
 			(hide yes)
 			(show_name no)
@@
 		)
 		(property "Manufacturer_Name" "Molex"
-			(at 43.18 772.39 0)
+			(at 43.18 -599.67 0)
 			(hide yes)
 			(show_name no)
@@
 		)
 		(property "Manufacturer_Part_Number" "503480-0800"
-			(at 43.18 872.39 0)
+			(at 43.18 -699.67 0)
 			(hide yes)
 			(show_name no)
@@
 			(at 91.44 135.89 0)
 			(hide yes)
+			(show_name no)
+			(do_not_autoplace no)
+			(effects
+				(font
+					(size 1.27 1.27)
+				)
+			)
+		)
+		(property "LCSC Part" "N/A"
+			(at 91.44 135.89 0)
+			(hide yes)

Commit message: Completed routing of 9V and 3.3V of PSU
Parts:
- removed D21: ESD5V0B03, A_HDJ_Library:D_0402_1005Metric, symbol Diode:ESD9B5.0ST5G
- removed R1, R2: 180R, Resistor_SMD:R_0402_1005Metric, symbol Device:R
- removed R3, R4, R5, R6: 47R, Resistor_SMD:R_0402_1005Metric, symbol Device:R
Connections:
- net at J2.4: now also D3.3 (GA)
- net at D3.1 (RA): now also J2.5
- net at D3.4 (BA): now also J2.3
- net at D4.1 (RA): now also J2.8
- net at D4.3 (GA): now also J2.7
- net at D4.4 (BA): now also J2.6

Commit message: Created updated BOM for PCBWay on all CTRL daughterboards. These boards have likely hit their final* version
*Ive said "Finished Version" many times in this project. I'm confident now, but no guarantees.
Parts:
- D3, D4: MPN (none) -> TJ-L5FCMXHTCSLCRGB-A5; Manufacturer (none) -> TOGIALED
- J2: LCSC Part C596711 -> (none); MPN (none) -> 5034800800; Manufacturer (none) -> MOLEX
- S1: MPN (none) -> B3S-1002; Manufacturer (none) -> OMRON
